File: power_db_hat/power_db_hat.kicad_sch (KiCad schematic)
At the start: 12 parts, among them J1 GPIO, J2 BAT1, J3 BAT2, J4 PD_power, J5 24V_out, J6 12V_out, J7 Conn_01x20_Pin, U1 CAT24C256

Commit message: working on it
Parts:
- removed J1: GPIO, Connector_PinSocket_2.54mm:PinSocket_2x20_P2.54mm_Vertical, symbol Connector_Generic:Conn_02x20_Odd_Even
- added C16, C17, C18: 100nF, symbol Device:C
- added D3: 5V, symbol Device:LED
- added D4: 12V, symbol Device:LED
- added D5: 24V, symbol Device:LED
- added D6: 3V3, symbol Device:LED
- added D7: LED, symbol Device:LED
- added J1: Conn_01x04_Pin, symbol Connector:Conn_01x04_Pin
- added R13: DNP, symbol Device:R_US
- added R23, R24, R25, R26, R3, R4: 0, symbol Device:R_US
- added R27, R28, R29, R30, R31: R, symbol Device:R_US
Connections:
- net +3.3V is gone; now on net +3V3: J4.3 (Pin_3)
- net +12V: now also C18.2, D4.2 (A), R25.1
- net +3V3: now also D6.2 (A)
- net +5V: now also D3.2 (A), R3.2
- net GND: now also C16.1, C17.1, C18.1, R27.2, R28.2, R29.2, R30.2, R31.2
- net VBAT1+: now also R13.1, R26.2
- net VBAT2+: now also R23.2, R4.1; no longer J5.2 (Pin_2)
- net power/5V_OUT: now also C16.2, R3.1
- net power/VIN_12V: now also R26.1
- net power/VIN_24V: now also R23.1
- net power/VOUT_12V: now also R25.2
- net power/VOUT_24V: now also R24.2
- new net: D5.1 (K), R30.1
- new net: D4.1 (K), R29.1
- new net: D6.1 (K), R27.1
- new net: D3.1 (K), R28.1
- new net: D7.1 (K), R31.1
- new net +24V: C17.2, D5.2 (A), J5.2 (Pin_2), R24.1
- new net IND: D7.2 (A)
- new net power/BUCK_IN: R13.2, R4.2
Other:
- added sheet HAT_connections (HAT_connections.kicad_sch)
- sheet power ports: added BUCK_IN; removed none
- note added: "TODO check available components in lab"
- note added: "secondary IMU or extra I2C"

Commit message: update
Parts:
- removed C1: 100n, symbol Device:C_Small
- removed JP1: ID_WP, symbol Jumper:SolderJumper_2_Open
- removed R1, R2: 3.9k, symbol Device:R_Small
- removed U1: CAT24C256, symbol Memory_EEPROM:CAT24C256
- C1: renamed from C17; footprint (none) -> Capacitor_SMD:C_0805_2012Metric_Pad1.18x1.45mm_HandSolder
- C2: renamed from C18; footprint (none) -> Capacitor_SMD:C_0805_2012Metric_Pad1.18x1.45mm_HandSolder
- C4: renamed from C16; footprint (none) -> Capacitor_SMD:C_0805_2012Metric_Pad1.18x1.45mm_HandSolder
- D1: renamed from D6; footprint (none) -> LED_SMD:LED_0603_1608Metric_Pad1.05x0.95mm_HandSolder
- D2: renamed from D3; footprint (none) -> LED_SMD:LED_0603_1608Metric_Pad1.05x0.95mm_HandSolder
- D3: renamed from D4; footprint (none) -> LED_SMD:LED_0603_1608Metric_Pad1.05x0.95mm_HandSolder
- D4: renamed from D5; footprint (none) -> LED_SMD:LED_0603_1608Metric_Pad1.05x0.95mm_HandSolder
- D5: renamed from D7; footprint (none) -> LED_SMD:LED_0603_1608Metric_Pad1.05x0.95mm_HandSolder
- J4: renamed from J1; footprint (none) -> Connector_JST:JST_GH_SM04B-GHS-TB_1x04-1MP_P1.25mm_Horizontal
- R1: renamed from R23; footprint (none) -> Resistor_SMD:R_0603_1608Metric_Pad0.98x0.95mm_HandSolder
- R10: renamed from R27; footprint (none) -> Resistor_SMD:R_0603_1608Metric_Pad0.98x0.95mm_HandSolder
- R11: renamed from R28; footprint (none) -> Resistor_SMD:R_0603_1608Metric_Pad0.98x0.95mm_HandSolder
- R12: renamed from R29; footprint (none) -> Resistor_SMD:R_0603_1608Metric_Pad0.98x0.95mm_HandSolder
- R13: renamed from R30; footprint (none) -> Resistor_SMD:R_0603_1608Metric_Pad0.98x0.95mm_HandSolder
- R14: renamed from R31; footprint (none) -> Resistor_SMD:R_0603_1608Metric_Pad0.98x0.95mm_HandSolder
- R2: renamed from R26; footprint (none) -> Resistor_SMD:R_0603_1608Metric_Pad0.98x0.95mm_HandSolder
- R3: renamed from R24; footprint (none) -> Resistor_SMD:R_0603_1608Metric_Pad0.98x0.95mm_HandSolder
- R4: renamed from R25; footprint (none) -> Resistor_SMD:R_0603_1608Metric_Pad0.98x0.95mm_HandSolder
- R5: renamed from R4; footprint (none) -> Resistor_SMD:R_0603_1608Metric_Pad0.98x0.95mm_HandSolder
- R6: renamed from R3; footprint (none) -> Resistor_SMD:R_0603_1608Metric_Pad0.98x0.95mm_HandSolder
- R7: renamed from R13; footprint (none) -> Resistor_SMD:R_0603_1608Metric_Pad0.98x0.95mm_HandSolder
- renumbered J6 to J3, J4 to J6, J3 to J8
Connections:
- no-connect marks 3 -> 0
Other:
- note added: "TODO change footprints for 10A rated components"
- note removed: "ID_SD and ID_SC PINS: These pins are reserved for HAT ID EEPROM. At boot time this I2C interface will be interrogated to look for an EEPROM that identifes the attached board and allows automagic setup of the GPIOs (and optionally, Linux drivers). Bridging JP1 enables write protection. DO NOT USE these pins for anything other than attaching an I2C ID EEPROM. Leave unconnected if ID EEPROM not requ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"

Commit message: update
Parts:
- added D10: TVS_3V3, symbol Device:D_Zener
- added D11, D9: TVS_12V, symbol Device:D_Zener
- added D8: TVS_24V, symbol Device:D_Zener
- added F1: FUSE_10A, symbol Device:Fuse
- added F2: FUSE_5A, symbol Device:Fuse
- R7: value DNP -> 0
Connections:
- net +12V: now also R4.2, F2.2; no longer R4.1
- net +24V: now also R3.2, F1.2; no longer R3.1
- net +3V3: now also D10.1 (K)
- net +5V: now also R6.1; no longer R6.2
- net GND: now also D10.2 (A), D11.2 (A), D8.2 (A), D9.2 (A)
- net PD_VIN: now also D11.1 (K)
- net VBAT1+: now also R7.2; no longer R7.1
- net power/5V_OUT: now also R6.2; no longer R6.1
- net power/BUCK_IN: now also R7.1; no longer R7.2
- net power/VOUT_12V: now also R4.1; no longer R4.2
- net power/VOUT_24V: now also R3.1; no longer R3.2
- new net: D8.1 (K), F1.1
- new net: D9.1 (K), F2.1
Other:
- note added: "26A rated jumpers"
- note added: "DNP"
- note added: "TODO secondary IMU or extra I2C"
- note added: "verify with current estimate"
- note removed: "TODO change footprints for 10A rated components"
- note removed: "secondary IMU or extra I2C"
- moved on the sheet: C1, C2, C4, D1, D2, D3, D4, D5, J4, J6, J7, R1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

Commit message: update
Parts:
- removed R5, R6, R7: 0, Resistor_SMD:R_0603_1608Metric_Pad0.98x0.95mm_HandSolder, symbol Device:R_US
- added D14, D17, D18, D19, D20, D21, D22, D23, D24, D25, D26, D27, D28, D29, D30, D31, D32, D33, D34, D35, D36, D37, D38: TVS_3V3, Diode_SMD:D_0603_1608Metric_Pad1.05x0.95mm_HandSolder, symbol Device:D_Zener
- added D39, D40: TVS_13V, Diode_SMD:D_0603_1608Metric_Pad1.05x0.95mm_HandSolder, symbol Device:D_Zener
- added D41: TVS_26V, Diode_SMD:D_0603_1608Metric_Pad1.05x0.95mm_HandSolder, symbol Device:D_Zener
- added JP2, JP3, JP4: SolderJumper_2_Open, Jumper:SolderJumper-2_P1.3mm_Open_TrianglePad1.0x1.5mm, symbol Jumper:SolderJumper_2_Open
- added R42, R43, R44, R45, R46, R47, R48, R49, R50, R51, R52, R53, R54, R55, R56, R57, R58, R59, R60, R61, R62, R63, R64: 33, Resistor_SMD:R_0603_1608Metric_Pad0.98x0.95mm_HandSolder, symbol Device:R_US
- D10: footprint (none) -> Diode_SMD:D_0603_1608Metric_Pad1.05x0.95mm_HandSolder
- D11, D9: value TVS_12V -> TVS_13V; footprint (none) -> Diode_SMD:D_0603_1608Metric_Pad1.05x0.95mm_HandSolder
- D8: value TVS_24V -> TVS_26V; footprint (none) -> Diode_SMD:D_0603_1608Metric_Pad1.05x0.95mm_HandSolder
- F1, F2: footprint (none) -> Fuse:Fuse_2512_6332Metric_Pad1.52x3.35mm_HandSolder
- J2, J8: footprint Connector_AMASS:AMASS_XT60PW-M_1x02_P7.20mm_Horizontal -> CONN_AMASS_3D_FIXED:AMASS_XT60PW-M_1x02_P7.20mm_Horizontal
- J3, J5: footprint Connector_AMASS:AMASS_XT60PW-F_1x02_P7.20mm_Horizontal -> CONN_AMASS_3D_FIXED:AMASS_XT60PW-F_1x02_P7.20mm_Horizontal
- J4: footprint Connector_JST:JST_GH_SM04B-GHS-TB_1x04-1MP_P1.25mm_Horizontal -> Connector_JST:JST_SH_SM04B-SRSS-TB_1x04-1MP_P1.00mm_Horizontal
Connections:
- net +3V3: now also R62.1
- net +5V: now also JP4.2 (B)
- net GND: now also J4.1 (Pin_1), D14.2 (A), D17.2 (A), D18.2 (A), D19.2 (A), D20.2 (A), D21.2 (A), D22.2 (A), D23.2 (A), D24.2 (A), D25.2 (A), D26.2 (A), D27.2 (A), D28.2 (A), D29.2 (A), D30.2 (A), D31.2 (A), D32.2 (A), D33.2 (A), D34.2 (A), D35.2 (A), D36.2 (A), D37.2 (A), D38.2 (A), D39.2 (A), D40.2 (A), D41.2 (A)
- net INT_HLD: now also R58.1; no longer J7.4 (Pin_4)
- net INT_RST: now also R59.1; no longer J7.3 (Pin_3)
- net INT_SLCTA: now also R61.1; no longer J7.1 (Pin_1)
- net INT_SLCTB: now also R57.1; no longer J7.5 (Pin_5)
- net IVC_SW_1: now also R43.1; no longer J7.19 (Pin_19)
- net IVC_SW_1_SOL: now also R44.1, R45.1; no longer J7.17 (Pin_17), J7.18 (Pin_18)
- net IVC_SW_2: now also R42.1; no longer J7.20 (Pin_20)
- net SPI_CS1: now also R47.1; no longer J7.15 (Pin_15)
- net SPI_CS2: now also R46.1; no longer J7.16 (Pin_16)
- net SPI_CS3: now also R50.1; no longer J7.12 (Pin_12)
- net SPI_CS4: now also R49.1; no longer J7.13 (Pin_13)
- net SPI_MISO: now also R51.1; no longer J7.11 (Pin_11)
- net SPI_MOSI: now also R54.1; no longer J7.8 (Pin_8)
- net SPI_SCLK: now also R48.1; no longer J7.14 (Pin_14)
- net STRT1: now also R53.1; no longer J7.9 (Pin_9)
- net STRT2: now also R52.1; no longer J7.10 (Pin_10)
- net VBAT1+: now also D39.1 (K), D40.1 (K), JP3.2 (B)
- net VBAT2+: now also D41.1 (K), JP2.2 (B)
- net power/5V_OUT: now also JP4.1 (A)
- net power/BUCK_IN: now also JP2.1 (A), JP3.1 (A)
- net ~{DRDY1}: now also R56.1; no longer J7.6 (Pin_6)
- net ~{DRDY2}: now also R55.1; no longer J7.7 (Pin_7)
- net ~{SYS_RESET}: now also R60.1; no longer J7.2 (Pin_2)
- net at J4.2 (Pin_2): now also D36.1 (K), R62.2
- net at J4.3 (Pin_3): now also D37.1 (K), R63.2
- net at J4.4 (Pin_4): now also D38.1 (K), R64.2
- new net: D27.1 (K), J7.12 (Pin_12), R50.2
- new net: D30.1 (K), J7.15 (Pin_15), R47.2
- new net: D22.1 (K), J7.7 (Pin_7), R55.2
- new net: D32.1 (K), J7.17 (Pin_17), R45.2
- new net: D35.1 (K), J7.20 (Pin_20), R42.2
- new net: D34.1 (K), J7.19 (Pin_19), R43.2
- new net: D23.1 (K), J7.8 (Pin_8), R54.2
- new net: D29.1 (K), J7.14 (Pin_14), R48.2
- new net: D31.1 (K), J7.16 (Pin_16), R46.2
- new net: D20.1 (K), J7.5 (Pin_5), R57.2
- new net: D14.1 (K), J7.1 (Pin_1), R61.2
- new net: D25.1 (K), J7.10 (Pin_10), R52.2
- new net: D26.1 (K), J7.11 (Pin_11), R51.2
- new net: D28.1 (K), J7.13 (Pin_13), R49.2
- new net: D33.1 (K), J7.18 (Pin_18), R44.2
- new net: D17.1 (K), J7.2 (Pin_2), R60.2
- new net: D18.1 (K), J7.3 (Pin_3), R59.2
- new net: D19.1 (K), J7.4 (Pin_4), R58.2
- new net: D21.1 (K), J7.6 (Pin_6), R56.2
- new net: D24.1 (K), J7.9 (Pin_9), R53.2
- new net EXT_SCL: R64.1
- new net EXT_SDA: R63.1
Other:
- note added: "Extra I2C for secondary IMU (qwIIC cable support)"
- note added: "TODO footprint for DF19-20P connector connector needs ground connection for shield"
- note removed: "DNP"
- note removed: "TODO secondary IMU or extra I2C"
- moved on the sheet: D11, J2, J4, J7

Commit message: lol
Other:
- added sheet servos+gpio (servos+gpio.kicad_sch)
- moved on the sheet: C1, C2, C4, D1, D2, D3, D4, D5, JP2, JP3, JP4, R1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
