File: power_db_hat/power_db_hat.kicad_pcb (KiCad board)
At the start: 2 copper layers, 65 x 56 mm, 11 parts, among them J1 GPIO, J2 BAT1, J3 BAT2, J4 PD_power, J5 24V_out, J6 12V_out, J7 Conn_01x20_Pin

Commit message: update
Parts:
- added C1: 100nF, Capacitor_SMD:C_0805_2012Metric_Pad1.18x1.45mm_HandSolder, F.Cu at (194.6, 113.5)
- added C10: 100nF, Capacitor_SMD:C_0805_2012Metric_Pad1.18x1.45mm_HandSolder, F.Cu at (221.6, 102.5)
- added C11: 4.7nF, Capacitor_SMD:C_0603_1608Metric_Pad1.08x0.95mm_HandSolder, F.Cu at (199.6, 107.5)
- added C12: 100nF, Capacitor_SMD:C_0805_2012Metric_Pad1.18x1.45mm_HandSolder, F.Cu at (206.6, 98.5)
- added C13: 47pF, Capacitor_SMD:C_0603_1608Metric_Pad1.08x0.95mm_HandSolder, F.Cu at (213.6, 91.5)
- added C14: 100nF, Capacitor_SMD:C_0805_2012Metric_Pad1.18x1.45mm_HandSolder, F.Cu at (206.6, 81.5)
- added C15: 47uF, Capacitor_SMD:C_0603_1608Metric_Pad1.08x0.95mm_HandSolder, F.Cu at (199.6, 110.5)
- added C16: 47uF, Capacitor_SMD:C_0603_1608Metric_Pad1.08x0.95mm_HandSolder, F.Cu at (199.6, 113.5)
- added C17: 47uF, Capacitor_SMD:C_0603_1608Metric_Pad1.08x0.95mm_HandSolder, F.Cu at (194.6, 107.5)
- added C18: 100nF, Capacitor_SMD:C_0805_2012Metric_Pad1.18x1.45mm_HandSolder, F.Cu at (222.6, 111.5)
- added C2: 100nF, Capacitor_SMD:C_0805_2012Metric_Pad1.18x1.45mm_HandSolder, F.Cu at (194.6, 93.5)
- added C4: 100nF, Capacitor_SMD:C_0805_2012Metric_Pad1.18x1.45mm_HandSolder, F.Cu at (194.6, 110.5)
- added C5: 100nF, Capacitor_SMD:C_0805_2012Metric_Pad1.18x1.45mm_HandSolder, F.Cu at (198.6, 85.5)
- added C6: 2.2uF, Capacitor_SMD:C_0603_1608Metric_Pad1.08x0.95mm_HandSolder, F.Cu at (194.6, 98.5)
- added C7: 2.2uF, Capacitor_SMD:C_0603_1608Metric_Pad1.08x0.95mm_HandSolder, F.Cu at (199.6, 95.5)
- added C8: 2.2uF, Capacitor_SMD:C_0603_1608Metric_Pad1.08x0.95mm_HandSolder, F.Cu at (199.6, 98.5)
- added C9: 2.2uF, Capacitor_SMD:C_0603_1608Metric_Pad1.08x0.95mm_HandSolder, F.Cu at (199.6, 92.5)
- added D1: 3V3, LED_SMD:LED_0603_1608Metric_Pad1.05x0.95mm_HandSolder, F.Cu at (219.0, 64.5)
- added D2: 5V, LED_SMD:LED_0603_1608Metric_Pad1.05x0.95mm_HandSolder, F.Cu at (219.0, 67.1)
- added D3: 12V, LED_SMD:LED_0603_1608Metric_Pad1.05x0.95mm_HandSolder, F.Cu at (219.0, 69.7)
- added D4: 24V, LED_SMD:LED_0603_1608Metric_Pad1.05x0.95mm_HandSolder, F.Cu at (219.0, 72.3)
- added D5: LED, LED_SMD:LED_0603_1608Metric_Pad1.05x0.95mm_HandSolder, F.Cu at (219.0, 74.9)
- added D6: B560C, Diode_SMD:D_SMB-SMC_Universal_Handsoldering, F.Cu at (211.6, 86.5)
- added D7: 12V, Diode_SMD:D_SMA-SMB_Universal_Handsoldering, F.Cu at (218.6, 95.5)
- added J4: Conn_01x04_Pin, Connector_JST:JST_GH_SM04B-GHS-TB_1x04-1MP_P1.25mm_Horizontal, F.Cu at (160.0, 69.5)
- added Q1: PMOS, Package_TO_SOT_SMD:TO-252-3_TabPin2, F.Cu at (230.6, 103.5)
- added Q2: PMOS, Package_TO_SOT_SMD:TO-252-3_TabPin2, F.Cu at (231.6, 112.5)
- added R1: 0, Resistor_SMD:R_0603_1608Metric_Pad0.98x0.95mm_HandSolder, F.Cu at (222.6, 115.5)
- added R10: R, Resistor_SMD:R_0603_1608Metric_Pad0.98x0.95mm_HandSolder, F.Cu at (227.7, 72.0)
- added R11: R, Resistor_SMD:R_0603_1608Metric_Pad0.98x0.95mm_HandSolder, F.Cu at (232.1, 64.5)
- added R12: R, Resistor_SMD:R_0603_1608Metric_Pad0.98x0.95mm_HandSolder, F.Cu at (232.1, 67.0)
- added R13: R, Resistor_SMD:R_0603_1608Metric_Pad0.98x0.95mm_HandSolder, F.Cu at (232.1, 69.5)
- added R14: R, Resistor_SMD:R_0603_1608Metric_Pad0.98x0.95mm_HandSolder, F.Cu at (232.1, 72.0)
- added R15: 12k, Resistor_SMD:R_0603_1608Metric_Pad0.98x0.95mm_HandSolder, F.Cu at (222.6, 91.5)
- added R16: 3k, Resistor_SMD:R_0603_1608Metric_Pad0.98x0.95mm_HandSolder, F.Cu at (198.6, 88.5)
- added R17: 12k, Resistor_SMD:R_0603_1608Metric_Pad0.98x0.95mm_HandSolder, F.Cu at (225.6, 85.5)
- added R18: 100, Resistor_SMD:R_0603_1608Metric_Pad0.98x0.95mm_HandSolder, F.Cu at (220.6, 86.5)
- added R19: 442k, Resistor_SMD:R_0603_1608Metric_Pad0.98x0.95mm_HandSolder, F.Cu at (202.6, 104.5)
- added R2: 0, Resistor_SMD:R_0603_1608Metric_Pad0.98x0.95mm_HandSolder, F.Cu at (140.5, 85.4)
- added R20: 442k, Resistor_SMD:R_0603_1608Metric_Pad0.98x0.95mm_HandSolder, F.Cu at (207.6, 104.5)
- added R21: 75k, Resistor_SMD:R_0603_1608Metric_Pad0.98x0.95mm_HandSolder, F.Cu at (227.6, 92.5)
- added R22: 442k, Resistor_SMD:R_0603_1608Metric_Pad0.98x0.95mm_HandSolder, F.Cu at (206.6, 101.5)
- added R23: 16.9k, Resistor_SMD:R_0603_1608Metric_Pad0.98x0.95mm_HandSolder, F.Cu at (206.6, 107.5)
- added R24: 2.2k, Resistor_SMD:R_0603_1608Metric_Pad0.98x0.95mm_HandSolder, F.Cu at (226.6, 95.5)
- added R25: 68k, Resistor_SMD:R_0603_1608Metric_Pad0.98x0.95mm_HandSolder, F.Cu at (231.6, 96.5)
- added R26: 10k, Resistor_SMD:R_0603_1608Metric_Pad0.98x0.95mm_HandSolder, F.Cu at (216.6, 104.5)
- added R27: 4.7k, Resistor_SMD:R_0603_1608Metric_Pad0.98x0.95mm_HandSolder, F.Cu at (217.6, 114.5)
- added R28: 100, Resistor_SMD:R_0603_1608Metric_Pad0.98x0.95mm_HandSolder, F.Cu at (221.6, 99.5)
- added R29: 200k, Resistor_SMD:R_0603_1608Metric_Pad0.98x0.95mm_HandSolder, F.Cu at (215.6, 109.5)
- added R3: 0, Resistor_SMD:R_0603_1608Metric_Pad0.98x0.95mm_HandSolder, F.Cu at (209.6, 110.5)
- added R30: 53.6k, Resistor_SMD:R_0603_1608Metric_Pad0.98x0.95mm_HandSolder, F.Cu at (197.6, 102.5)
- added R31: 10.2k, Resistor_SMD:R_0603_1608Metric_Pad0.98x0.95mm_HandSolder, F.Cu at (211.6, 99.5)
- added R4: 0, Resistor_SMD:R_0603_1608Metric_Pad0.98x0.95mm_HandSolder, F.Cu at (225.6, 88.5)
- added R5: 0, Resistor_SMD:R_0603_1608Metric_Pad0.98x0.95mm_HandSolder, F.Cu at (204.6, 112.5)
- added R6: 0, Resistor_SMD:R_0603_1608Metric_Pad0.98x0.95mm_HandSolder, F.Cu at (191.6, 80.5)
- added R7: DNP, Resistor_SMD:R_0603_1608Metric_Pad0.98x0.95mm_HandSolder, F.Cu at (126.5, 85.5)
- added U2: TL431DBZ, Package_TO_SOT_SMD:SOT-23, F.Cu at (198.6, 81.5)
- added U3: TPS54560BDDA, Package_SO:Texas_R-PDSO-G8_EP2.95x4.9mm_Mask2.4x3.1mm_ThermalVias, F.Cu at (206.6, 93.5)
- added U4: TL431DBZ, Package_TO_SOT_SMD:SOT-23, F.Cu at (216.6, 100.5)
- moved J2 21.0 mm to (126.6, 91.3)
- moved J8 21.0 mm to (147.6, 91.3)
- renumbered J6 to J3, J4 to J6, J3 to J8
Connections:
- net /GPIO12/PWM0 renamed /HAT_connections/GPIO12/PWM0
- net /GPIO13/PWM1 renamed /HAT_connections/GPIO13/PWM1
- net /GPIO14/TXD0 renamed /HAT_connections/GPIO14/TXD0
- net /GPIO15/RXD0 renamed /HAT_connections/GPIO15/RXD0
- net /GPIO16 renamed /HAT_connections/GPIO16
- net /GPIO17 renamed /HAT_connections/GPIO17
- net /GPIO18/PCM.CLK renamed /HAT_connections/GPIO18/PCM.CLK
- net /GPIO19/PCM.FS renamed /HAT_connections/GPIO19/PCM.FS
- net /GPIO20/PCM.DIN renamed /HAT_connections/GPIO20/PCM.DIN
- net /GPIO21/PCM.DOUT renamed /HAT_connections/GPIO21/PCM.DOUT
- net /GPIO22 renamed /HAT_connections/GPIO22
- net /GPIO25 renamed /HAT_connections/GPIO25
- net /GPIO26 renamed /HAT_connections/GPIO26
- net /GPIO27 renamed /HAT_connections/GPIO27
- net /GPIO2/SDA1 renamed /HAT_connections/GPIO2/SDA1
- net /GPIO3/SCL1 renamed /HAT_connections/GPIO3/SCL1
- net /GPIO4/GPCLK0 renamed /HAT_connections/GPIO4/GPCLK0
- net /GPIO5 renamed /HAT_connections/GPIO5
- net /GPIO6 renamed /HAT_connections/GPIO6
- net /ID_SCL renamed /HAT_connections/ID_SCL
- net /ID_SDA renamed /HAT_connections/ID_SDA
- J1 pad 16: /GPIO23 -> /SPI_CS3
- J1 pad 18: /GPIO24 -> /SPI_CS4
- J1 pad 19: /GPIO10/SPI0.MOSI -> /SPI_MOSI
- J1 pad 21: /GPIO9/SPI0.MISO -> /SPI_MISO
- J1 pad 23: /GPIO11/SPI0.SCLK -> /SPI_SCLK
- J1 pad 24: /GPIO8/SPI0.CE0 -> /SPI_CS1
- J1 pad 26: /GPIO7/SPI0.CE1 -> /SPI_CS2
- J2 pad 1: unconnected-(J2-Pin_1-Pad1) -> /VBAT1+
- J2 pad 2: unconnected-(J2-Pin_2-Pad2) -> /VBAT2+
- J3 pad 1: unconnected-(J6-Pin_1-Pad1) -> GND
- J3 pad 2: unconnected-(J6-Pin_2-Pad2) -> +12V
- J5 pad 1: unconnected-(J5-Pin_1-Pad1) -> GND
- J5 pad 2: unconnected-(J5-Pin_2-Pad2) -> +24V
- J6 pad 1: unconnected-(J4-Pin_1-Pad1) -> /PD_VIN
- J6 pad 2: unconnected-(J4-Pin_2-Pad2) -> GND
- J6 pad 3: unconnected-(J4-Pin_3-Pad3) -> +3V3
- J6 pad 4: unconnected-(J4-Pin_4-Pad4) -> GND
- J8 pad 1: unconnected-(J3-Pin_1-Pad1) -> GND
- J8 pad 2: unconnected-(J3-Pin_2-Pad2) -> /VBAT1+
Routing:
- net /VBAT1+: track 0.00 -> 13.8 mm
- added copper zone on F.Cu, net GND

Commit message: update
Parts:
- moved Q2 109.3 mm to (127.5, 79.0)
- moved Q1 88.6 mm to (145.4, 79.0)
Changed lines of the file:
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@@
 		(placed yes)
 		(layer "F.Cu")
-		(at 230.565 103.475)
+		(at 145.415 79.025)
 		(descr "TO-252/DPAK SMD package, http://www.infineon.com/cms/en/product/packages/PG-TO252/PG-TO252-3-1/")
 		(tags "DPAK TO-252 DPAK-3 TO-252-3 SOT-428")
@@
 		(placed yes)
 		(layer "F.Cu")
-		(at 231.565 112.475)
+		(at 127.54 79)
 		(descr "TO-252/DPAK SMD package, http://www.infineon.com/cms/en/product/packages/PG-TO252/PG-TO252-3-1/")
 		(tags "DPAK TO-252 DPAK-3 TO-252-3 SOT-428")
@@
 		)
 	)
-	(gr_arc
-		(start 100 46.5)
-		(mid 100.87868 44.37868)
+	(gr_line
+		(start 162 43.5)
 		(end 103 43.5)
 		(stroke
@@
 		(layer "Dwgs.User")
 	)
-	(gr_line
-		(start 100 47)
-		(end 100 46.5)
+	(gr_rect
+		(start 166 81.825)
+		(end 187 97.675)
 		(stroke
 			(width 0.1)
 			(type solid)
 		)
+		(fill no)
+		(locked yes)
 		(layer "Dwgs.User")
 	)
 	(gr_line
-		(start 100 63)
-		(end 100 81)
+		(start 165 47)
+		(end 165 46.5)
 		(stroke
 			(width 0.1)
@@
 		(layer "Dwgs.User")
 	)
-	(gr_line
-		(start 162 43.5)
-		(end 103 43.5)
+	(gr_rect
+		(start 169.9 64.45)
+		(end 187 77.55)
 		(stroke
 			(width 0.1)
 			(type solid)
 		)
+		(fill no)
+		(locked yes)
 		(layer "Dwgs.User")
 	)
 	(gr_arc
-		(start 162 43.5)
-		(mid 164.12132 44.37868)
-		(end 165 46.5)
+		(start 100 46.5)
+		(mid 100.87868 44.37868)
+		(end 103 43.5)
 		(stroke
 			(width 0.1)
@@
 	)
 	(gr_line
-		(start 165 47)
-		(end 165 46.5)
+		(start 100 63)
+		(end 100 81)
 		(stroke
 			(width 0.1)
@@
 		(layer "Dwgs.User")
 	)
-	(gr_rect
-		(start 166 81.825)
-		(end 187 97.675)
+	(gr_line
+		(start 100 47)
+		(end 100 46.5)
 		(stroke
 			(width 0.1)
 			(type solid)
 		)
-		(fill no)
-		(locked yes)
 		(layer "Dwgs.User")
 	)
@@
 		(layer "Dwgs.User")
 	)
-	(gr_rect
-		(start 169.9 64.45)
-		(end 187 77.55)
+	(gr_arc
+		(start 162 43.5)
+		(mid 164.12132 44.37868)
+		(end 165 46.5)
 		(stroke
 			(width 0.1)
 			(type solid)
 		)
-		(fill no)
-		(locked yes)
 		(layer "Dwgs.User")
 	)
-	(gr_line
-		(start 100 47)
-		(end 100 63)
+	(gr_arc
+		(start 162 44)
+		(mid 164.12132 44.87868)
+		(end 165 47)
 		(stroke
 			(width 0.1)
@@
 		(layer "Edge.Cuts")
 	)
-	(gr_arc
-		(start 100 47)
-		(mid 100.87868 44.87868)
-		(end 103 44)
+	(gr_line
+		(start 165 97)
+		(end 165 47)
 		(stroke
 			(width 0.1)
@@
 	)
 	(gr_line
-		(start 100 63)
-		(end 100 97)
+		(start 100 47)
+		(end 100 63)
 		(stroke
 			(width 0.1)
@@
 		(layer "Edge.Cuts")
 	)
-	(gr_line
-		(start 162 44)
-		(end 103 44)
+	(gr_arc
+		(start 165 97)
+		(mid 164.12132 99.12132)
+		(end 162 100)
 		(stroke
 			(width 0.1)
@@
 	)
 	(gr_arc
-		(start 162 44)
-		(mid 164.12132 44.87868)
-		(end 165 47)
+		(start 100 47)
+		(mid 100.87868 44.87868)
+		(end 103 44)
 		(stroke
 			(width 0.1)
@@
 		(layer "Edge.Cuts")
 	)
-	(gr_arc
-		(start 165 97)
-		(mid 164.12132 99.12132)
-		(end 162 100)
+	(gr_line
+		(start 100 63)
+		(end 100 97)
 		(stroke
 			(width 0.1)
@@
 	)
 	(gr_line
-		(start 165 97)
-		(end 165 47)
+		(start 162 44)
+		(end 103 44)
 		(stroke
 			(width 0.1)
@@
 		(layer "Edge.Cuts")
 	)
-	(gr_text "Extend PCB edge 0.5mm if using SMT header"
-		(at 103 42.5 0)
+	(gr_text "USB"
+		(at 177.724 71.552 0)
 		(layer "Dwgs.User")
 		(effects
 			(font
-				(size 1 1)
+				(size 2 2)
 				(thickness 0.15)
 			)
-			(justify left)
 		)
 	)
-	(gr_text "DISPLAY (OPTIONAL)"
-		(at 102.5 72 90)
+	(gr_text "RJ45"
+		(at 176.2 89.84 0)
 		(layer "Dwgs.User")
 		(effects
 			(font
-				(size 1 1)
+				(size 2 2)
 				(thickness 0.15)
 			)
 		)
 	)
-	(gr_text "RJ45"
-		(at 176.2 89.84 0)
+	(gr_text "DISPLAY (OPTIONAL)"
+		(at 102.5 72 90)
 		(layer "Dwgs.User")
 		(effects
 			(font
-				(size 2 2)
+				(size 1 1)
 				(thickness 0.15)
 			)
@@
 	)
 	(gr_text "USB"
-		(at 177.724 71.552 0)
+		(at 178.232 52.248 0)
 		(layer "Dwgs.User")
 		(effects
@@
 		)
 	)
-	(gr_text "USB"
-		(at 178.232 52.248 0)
+	(gr_text "Extend PCB edge 0.5mm if using SMT header"
+		(at 103 42.5 0)
 		(layer "Dwgs.User")
 		(effects
 			(font
-				(size 2 2)
+				(size 1 1)
 				(thickness 0.15)
 			)
+			(justify left)
 		)
 	)

Commit message: update
Parts:
- added C3: 100nF, Capacitor_SMD:C_0805_2012Metric_Pad1.18x1.45mm_HandSolder, F.Cu at (168.2, 128.6)
- added D10: TVS_3V3, Diode_SMD:D_0603_1608Metric_Pad1.05x0.95mm_HandSolder, B.Cu at (268.0, 146.3)
- added D11: TVS_13V, Diode_SMD:D_0603_1608Metric_Pad1.05x0.95mm_HandSolder, B.Cu at (268.0, 148.9)
- added D12: TVS_12V, Diode_SMD:D_0603_1608Metric_Pad1.05x0.95mm_HandSolder, B.Cu at (248.4, 157.9)
- added D13: TVS_12V, Diode_SMD:D_0603_1608Metric_Pad1.05x0.95mm_HandSolder, B.Cu at (248.4, 160.5)
- added D14: TVS_3V3, Diode_SMD:D_0603_1608Metric_Pad1.05x0.95mm_HandSolder, B.Cu at (268.0, 151.5)
- added D15: TVS_24V, Diode_SMD:D_0603_1608Metric_Pad1.05x0.95mm_HandSolder, B.Cu at (248.4, 163.0)
- added D16: TVS_24V, Diode_SMD:D_0603_1608Metric_Pad1.05x0.95mm_HandSolder, B.Cu at (248.4, 165.6)
- added D17: TVS_3V3, Diode_SMD:D_0603_1608Metric_Pad1.05x0.95mm_HandSolder, B.Cu at (268.0, 154.1)
- added D18: TVS_3V3, Diode_SMD:D_0603_1608Metric_Pad1.05x0.95mm_HandSolder, B.Cu at (268.0, 156.7)
- added D19: TVS_3V3, Diode_SMD:D_0603_1608Metric_Pad1.05x0.95mm_HandSolder, B.Cu at (263.6, 141.1)
- added D20: TVS_3V3, Diode_SMD:D_0603_1608Metric_Pad1.05x0.95mm_HandSolder, B.Cu at (263.6, 143.7)
- added D21: TVS_3V3, Diode_SMD:D_0603_1608Metric_Pad1.05x0.95mm_HandSolder, B.Cu at (263.6, 146.3)
- added D22: TVS_3V3, Diode_SMD:D_0603_1608Metric_Pad1.05x0.95mm_HandSolder, B.Cu at (263.6, 148.9)
- added D23: TVS_3V3, Diode_SMD:D_0603_1608Metric_Pad1.05x0.95mm_HandSolder, B.Cu at (263.6, 151.5)
- added D24: TVS_3V3, Diode_SMD:D_0603_1608Metric_Pad1.05x0.95mm_HandSolder, B.Cu at (263.6, 154.1)
- added D25: TVS_3V3, Diode_SMD:D_0603_1608Metric_Pad1.05x0.95mm_HandSolder, B.Cu at (263.6, 156.7)
- added D26: TVS_3V3, Diode_SMD:D_0603_1608Metric_Pad1.05x0.95mm_HandSolder, B.Cu at (259.2, 141.1)
- added D27: TVS_3V3, Diode_SMD:D_0603_1608Metric_Pad1.05x0.95mm_HandSolder, B.Cu at (259.2, 143.7)
- added D28: TVS_3V3, Diode_SMD:D_0603_1608Metric_Pad1.05x0.95mm_HandSolder, B.Cu at (259.2, 146.3)
- added D29: TVS_3V3, Diode_SMD:D_0603_1608Metric_Pad1.05x0.95mm_HandSolder, B.Cu at (259.2, 148.9)
- added D30: TVS_3V3, Diode_SMD:D_0603_1608Metric_Pad1.05x0.95mm_HandSolder, B.Cu at (259.2, 151.5)
- added D31: TVS_3V3, Diode_SMD:D_0603_1608Metric_Pad1.05x0.95mm_HandSolder, B.Cu at (259.2, 154.1)
- added D32: TVS_3V3, Diode_SMD:D_0603_1608Metric_Pad1.05x0.95mm_HandSolder, B.Cu at (259.2, 156.7)
- added D33: TVS_3V3, Diode_SMD:D_0603_1608Metric_Pad1.05x0.95mm_HandSolder, B.Cu at (254.8, 141.1)
- added D34: TVS_3V3, Diode_SMD:D_0603_1608Metric_Pad1.05x0.95mm_HandSolder, B.Cu at (254.8, 143.7)
- added D35: TVS_3V3, Diode_SMD:D_0603_1608Metric_Pad1.05x0.95mm_HandSolder, B.Cu at (254.8, 146.3)
- added D36: TVS_3V3, Diode_SMD:D_0603_1608Metric_Pad1.05x0.95mm_HandSolder, B.Cu at (254.8, 148.9)
- added D37: TVS_3V3, Diode_SMD:D_0603_1608Metric_Pad1.05x0.95mm_HandSolder, B.Cu at (254.8, 151.5)
- added D38: TVS_3V3, Diode_SMD:D_0603_1608Metric_Pad1.05x0.95mm_HandSolder, B.Cu at (254.8, 154.1)
- added D39: TVS_13V, Diode_SMD:D_0603_1608Metric_Pad1.05x0.95mm_HandSolder, F.Cu at (134.5, 85.5)
- added D40: TVS_13V, Diode_SMD:D_0603_1608Metric_Pad1.05x0.95mm_HandSolder, F.Cu at (123.5, 86.0)
- added D41: TVS_26V, Diode_SMD:D_0603_1608Metric_Pad1.05x0.95mm_HandSolder, F.Cu at (116.5, 86.0)
- added D8: TVS_26V, Diode_SMD:D_0603_1608Metric_Pad1.05x0.95mm_HandSolder, B.Cu at (268.0, 141.1)
- added D9: TVS_13V, Diode_SMD:D_0603_1608Metric_Pad1.05x0.95mm_HandSolder, B.Cu at (268.0, 143.7)
- added F1: FUSE_10A, Fuse:Fuse_2512_6332Metric_Pad1.52x3.35mm_HandSolder, F.Cu at (154.9, 137.3)
- added F2: FUSE_5A, Fuse:Fuse_2512_6332Metric_Pad1.52x3.35mm_HandSolder, F.Cu at (154.9, 142.2)
- added J10: Conn_01x04_Pin, Connector_JST:JST_GH_SM04B-GHS-TB_1x04-1MP_P1.25mm_Horizontal, F.Cu at (151.7, 95.7)
- added J9: Conn_01x04_Pin, Connector_JST:JST_GH_SM04B-GHS-TB_1x04-1MP_P1.25mm_Horizontal, F.Cu at (160.0, 86.0)
- added JP1: SolderJumper_2_Open, Jumper:SolderJumper-2_P1.3mm_Open_TrianglePad1.0x1.5mm, F.Cu at (176.0, 116.0)
- added JP2: SolderJumper_2_Open, Jumper:SolderJumper-2_P1.3mm_Open_TrianglePad1.0x1.5mm, F.Cu at (153.9, 125.1)
- added JP3: SolderJumper_2_Open, Jumper:SolderJumper-2_P1.3mm_Open_TrianglePad1.0x1.5mm, F.Cu at (153.9, 128.9)
- added JP4: SolderJumper_2_Open, Jumper:SolderJumper-2_P1.3mm_Open_TrianglePad1.0x1.5mm, F.Cu at (153.9, 132.8)
- added L1: 8.2uH, Inductors_custom:VSHB0754T_Molded_Power_Choke, F.Cu at (165.2, 146.4)
- added Q3: PMOS, Package_TO_SOT_SMD:TO-252-3_TabPin2, F.Cu at (125.4, 76.3)
- added Q4: PMOS, Package_TO_SOT_SMD:TO-252-3_TabPin2, F.Cu at (194.6, 73.4)
- added R32: 4.7k, Resistor_SMD:R_0603_1608Metric_Pad0.98x0.95mm_HandSolder, F.Cu at (163.6, 124.5)
- added R33: 10m, Resistor_SMD:R_2512_6332Metric_Pad1.40x3.35mm_HandSolder, B.Cu at (246.1, 147.2)
- added R34: 10m, Resistor_SMD:R_2512_6332Metric_Pad1.40x3.35mm_HandSolder, B.Cu at (246.1, 152.1)
- added R35: 4.7k, Resistor_SMD:R_0603_1608Metric_Pad0.98x0.95mm_HandSolder, F.Cu at (163.6, 127.0)
- added R36: 4.7k, Resistor_SMD:R_0603_1608Metric_Pad0.98x0.95mm_HandSolder, F.Cu at (163.6, 129.5)
- added R37: 4.7k, Resistor_SMD:R_0603_1608Metric_Pad0.98x0.95mm_HandSolder, F.Cu at (163.6, 132.1)
- added R38: 4.7k, Resistor_SMD:R_0603_1608Metric_Pad0.98x0.95mm_HandSolder, F.Cu at (163.6, 134.6)
- added R39: 4.7k, Resistor_SMD:R_0603_1608Metric_Pad0.98x0.95mm_HandSolder, F.Cu at (163.6, 137.1)
- added R40: 4.7k, Resistor_SMD:R_0603_1608Metric_Pad0.98x0.95mm_HandSolder, F.Cu at (163.6, 139.6)
- added R41: 4.7k, Resistor_SMD:R_0603_1608Metric_Pad0.98x0.95mm_HandSolder, F.Cu at (163.6, 142.1)
- added R42: 33, Resistor_SMD:R_0603_1608Metric_Pad0.98x0.95mm_HandSolder, F.Cu at (139.5, 124.5)
- added R43: 33, Resistor_SMD:R_0603_1608Metric_Pad0.98x0.95mm_HandSolder, F.Cu at (139.5, 127.0)
- added R44: 33, Resistor_SMD:R_0603_1608Metric_Pad0.98x0.95mm_HandSolder, F.Cu at (139.5, 129.5)
- added R45: 33, Resistor_SMD:R_0603_1608Metric_Pad0.98x0.95mm_HandSolder, F.Cu at (139.5, 132.1)
- added R46: 33, Resistor_SMD:R_0603_1608Metric_Pad0.98x0.95mm_HandSolder, F.Cu at (139.5, 134.6)
- added R47: 33, Resistor_SMD:R_0603_1608Metric_Pad0.98x0.95mm_HandSolder, F.Cu at (139.5, 137.1)
- added R48: 33, Resistor_SMD:R_0603_1608Metric_Pad0.98x0.95mm_HandSolder, F.Cu at (139.5, 139.6)
- added R49: 33, Resistor_SMD:R_0603_1608Metric_Pad0.98x0.95mm_HandSolder, F.Cu at (139.5, 142.1)
- added R50: 33, Resistor_SMD:R_0603_1608Metric_Pad0.98x0.95mm_HandSolder, F.Cu at (143.9, 124.5)
- added R51: 33, Resistor_SMD:R_0603_1608Metric_Pad0.98x0.95mm_HandSolder, F.Cu at (143.9, 127.0)
- added R52: 33, Resistor_SMD:R_0603_1608Metric_Pad0.98x0.95mm_HandSolder, F.Cu at (143.9, 129.5)
- added R53: 33, Resistor_SMD:R_0603_1608Metric_Pad0.98x0.95mm_HandSolder, F.Cu at (143.9, 132.1)
- added R54: 33, Resistor_SMD:R_0603_1608Metric_Pad0.98x0.95mm_HandSolder, F.Cu at (143.9, 134.6)
- added R55: 33, Resistor_SMD:R_0603_1608Metric_Pad0.98x0.95mm_HandSolder, F.Cu at (143.9, 137.1)
- added R56: 33, Resistor_SMD:R_0603_1608Metric_Pad0.98x0.95mm_HandSolder, F.Cu at (143.9, 139.6)
- added R57: 33, Resistor_SMD:R_0603_1608Metric_Pad0.98x0.95mm_HandSolder, F.Cu at (143.9, 142.1)
- added R58: 33, Resistor_SMD:R_0603_1608Metric_Pad0.98x0.95mm_HandSolder, F.Cu at (148.2, 124.5)
- added R59: 33, Resistor_SMD:R_0603_1608Metric_Pad0.98x0.95mm_HandSolder, F.Cu at (148.2, 127.0)
- added R60: 33, Resistor_SMD:R_0603_1608Metric_Pad0.98x0.95mm_HandSolder, F.Cu at (148.2, 129.5)
- added R61: 33, Resistor_SMD:R_0603_1608Metric_Pad0.98x0.95mm_HandSolder, F.Cu at (148.2, 132.1)
- added R62: 33, Resistor_SMD:R_0603_1608Metric_Pad0.98x0.95mm_HandSolder, F.Cu at (148.2, 134.6)
- added R63: 33, Resistor_SMD:R_0603_1608Metric_Pad0.98x0.95mm_HandSolder, F.Cu at (148.2, 137.1)
- added R64: 33, Resistor_SMD:R_0603_1608Metric_Pad0.98x0.95mm_HandSolder, F.Cu at (148.2, 139.6)
- added R8: 10m, Resistor_SMD:R_2512_6332Metric_Pad1.40x3.35mm_HandSolder, B.Cu at (246.1, 142.3)
- added U1: INA3221, Package_DFN_QFN:Texas_RGV0016A_VQFN-16-1EP_4x4mm_P0.65mm_EP2.1x2.1mm, B.Cu at (214.6, 87.2)
- D1, D2, D3, D4, D5, D6, D7, Q1, Q2, R10, R11, R12, R13, R14, R6, U2: moved to B.Cu
- J2, J8: footprint Connector_AMASS:AMASS_XT60PW-M_1x02_P7.20mm_Horizontal -> CONN_AMASS_3D_FIXED:AMASS_XT60PW-M_1x02_P7.20mm_Horizontal
- J3, J5: footprint Connector_AMASS:AMASS_XT60PW-F_1x02_P7.20mm_Horizontal -> CONN_AMASS_3D_FIXED:AMASS_XT60PW-F_1x02_P7.20mm_Horizontal
- J4: footprint Connector_JST:JST_GH_SM04B-GHS-TB_1x04-1MP_P1.25mm_Horizontal -> Connector_JST:JST_SH_SM04B-SRSS-TB_1x04-1MP_P1.00mm_Horizontal
- R19, R22: value 442k -> 309k
- R20: value 442k -> 53.6k
- R23: value 16.9k -> 14k
- R7: value DNP -> 0; moved to B.Cu
- moved R7 130.9 mm to (255.2, 109.6)
- moved R6 88.3 mm to (279.5, 89.1), turned to 180 degrees
- moved C2 68.0 mm to (163.5, 33.0)
- moved C6 68.0 mm to (163.5, 38.0)
- moved U2 63.8 mm to (262.3, 80.1), turned to 180 degrees
- moved C14 52.9 mm to (176.5, 38.0)
- moved C1 49.4 mm to (200.9, 64.5)
- moved C16 49.4 mm to (205.9, 64.5)
- moved R5 49.4 mm to (210.9, 63.5)
- moved C11 49.4 mm to (193.5, 58.5)
- moved C15 49.4 mm to (193.5, 61.5)
- moved C17 49.4 mm to (188.5, 58.5)
- moved C4 49.4 mm to (188.5, 61.5)
- moved R19 49.4 mm to (196.5, 55.5)
- moved R20 49.4 mm to (201.5, 55.5)
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Connections:
- C10 pad 1: /power/VOUT_12V -> /power/12V_SNS
- C15 pad 2: /power/5V_OUT -> /power/5V_SNS
- C16 pad 2: /power/5V_OUT -> /power/5V_SNS
- C17 pad 2: /power/5V_OUT -> /power/5V_SNS
- C18 pad 1: /power/VOUT_24V -> /power/24V_SNS
- D7 pad 2: /power/VIN_24V -> /power/24V_SWITCH
- J4 pad 1: unconnected-(J4-Pin_1-Pad1) -> GND
- J4 pad 2: unconnected-(J4-Pin_2-Pad2) -> Net-(D36-K)
- J4 pad 3: unconnected-(J4-Pin_3-Pad3) -> Net-(D37-K)
- J4 pad 4: unconnected-(J4-Pin_4-Pad4) -> Net-(D38-K)
- J7 pad 1: /INT_SLCTA -> Net-(D14-K)
- J7 pad 10: /STRT2 -> Net-(D25-K)
- J7 pad 11: /SPI_MISO -> Net-(D26-K)
- J7 pad 12: /SPI_CS3 -> Net-(D27-K)
- J7 pad 13: /SPI_CS4 -> Net-(D28-K)
- J7 pad 14: /SPI_SCLK -> Net-(D29-K)
- J7 pad 15: /SPI_CS1 -> Net-(D30-K)
- J7 pad 16: /SPI_CS2 -> Net-(D31-K)
- J7 pad 17: /IVC_SW_1_SOL -> Net-(D32-K)
- J7 pad 18: /IVC_SW_1_SOL -> Net-(D33-K)
- J7 pad 19: /IVC_SW_1 -> Net-(D34-K)
- J7 pad 2: /~{SYS_RESET} -> Net-(D17-K)
- J7 pad 20: /IVC_SW_2 -> Net-(D35-K)
- J7 pad 3: /INT_RST -> Net-(D18-K)
- J7 pad 4: /INT_HLD -> Net-(D19-K)
- J7 pad 5: /INT_SLCTB -> Net-(D20-K)
- J7 pad 6: /~{DRDY1} -> Net-(D21-K)
- J7 pad 7: /~{DRDY2} -> Net-(D22-K)
- J7 pad 8: /SPI_MOSI -> Net-(D23-K)
- J7 pad 9: /STRT1 -> Net-(D24-K)
- Q1 pad 1: /power/VOUT_12V -> /power/12V_SNS
- Q1 pad 3: /power/VIN_12V -> /power/12V_SWITCH
- Q2 pad 1: /power/VOUT_24V -> /power/24V_SNS
- Q2 pad 3: /power/VIN_24V -> /power/24V_SWITCH
- R15 pad 1: /power/VIN_12V -> /power/12V_SWITCH
- R17 pad 1: /power/VIN_12V -> /power/12V_SWITCH
- R21 pad 1: /power/VOUT_12V -> /power/12V_SNS
- R24 pad 1: /power/VIN_24V -> /power/24V_SWITCH
- R27 pad 1: /power/VIN_24V -> /power/24V_SWITCH
- R29 pad 1: /power/VOUT_24V -> /power/24V_SNS
- R3 pad 1: +24V -> /power/VOUT_24V
- R3 pad 2: /power/VOUT_24V -> +24V
- R30 pad 1: /power/5V_OUT -> /power/5V_SNS
- R4 pad 1: +12V -> /power/VOUT_12V
- R4 pad 2: /power/VOUT_12V -> +12V
- R6 pad 1: /power/5V_OUT -> +5V
- R6 pad 2: +5V -> /power/5V_OUT
- R7 pad 1: /VBAT1+ -> /power/BUCK_IN
- R7 pad 2: /power/BUCK_IN -> /VBAT1+
Routing:
- removed copper zone on F.Cu, net GND

Commit message: lol
Parts:
- removed Q4: PMOS, Package_TO_SOT_SMD:TO-252-3_TabPin2
- added D42: TVS_13V, Diode_SMD:D_0603_1608Metric_Pad1.05x0.95mm_HandSolder, F.Cu at (314.9, 85.8)
- added D43: TVS_26V, Diode_SMD:D_0603_1608Metric_Pad1.05x0.95mm_HandSolder, F.Cu at (314.9, 88.4)
- added D44: TVS_5V, Diode_SMD:D_0603_1608Metric_Pad1.05x0.95mm_HandSolder, F.Cu at (308.5, 77.6)
- added D45: TVS_3V3, Diode_SMD:D_0603_1608Metric_Pad1.05x0.95mm_HandSolder, F.Cu at (308.5, 80.2)
- added D46: TVS_3V3, Diode_SMD:D_0603_1608Metric_Pad1.05x0.95mm_HandSolder, F.Cu at (308.5, 82.8)
- added D47: TVS_5V, Diode_SMD:D_0603_1608Metric_Pad1.05x0.95mm_HandSolder, F.Cu at (308.5, 85.4)
- added D48: TVS_3V3, Diode_SMD:D_0603_1608Metric_Pad1.05x0.95mm_HandSolder, F.Cu at (308.5, 88.0)
- added D49: TVS_5V, Diode_SMD:D_0603_1608Metric_Pad1.05x0.95mm_HandSolder, F.Cu at (308.5, 90.5)
- added D50: TVS_3V3, Diode_SMD:D_0603_1608Metric_Pad1.05x0.95mm_HandSolder, F.Cu at (308.5, 93.1)
- added D51: TVS_5V, Diode_SMD:D_0603_1608Metric_Pad1.05x0.95mm_HandSolder, F.Cu at (308.5, 95.7)
- added Q5: PMOS, Package_TO_SOT_SMD:TO-252-3_TabPin2, F.Cu at (319.6, 80.5)
- D12, D13: value TVS_12V -> TVS_13V
- D15, D16: value TVS_24V -> TVS_26V
- R5, R7: value 0 -> 100k
- R6: value 0 -> 10k
Connections:
- D13 pad 1: /power/VIN_12V -> Net-(D13-K)
- D16 pad 2: GND -> Net-(D16-A)
- J10 pad 2: /power/VIN_24V -> Net-(D16-A)
- J9 pad 2: /power/VIN_12V -> Net-(D13-K)
- Q3 pad 1: /power/12V_SWITCH -> /power/24V_SWITCH
- Q3 pad 2: /power/VIN_12V -> Net-(Q3-G)
- Q3 pad 3: /power/VIN_12V -> /power/VIN_24V
- R5 pad 1: /VBAT2+ -> /power/VIN_12V
- R5 pad 2: /power/BUCK_IN -> Net-(D13-K)
- R6 pad 1: +5V -> Net-(D13-K)
- R6 pad 2: /power/5V_OUT -> Net-(Q5-G)
- R7 pad 1: /power/BUCK_IN -> /power/VIN_24V
- R7 pad 2: /VBAT1+ -> Net-(D16-A)
