File: power_db_hat/power_db_hat.kicad_pcb (KiCad board)
At the start: 4 copper layers, 65 x 56 mm, 136 parts, among them J1 Conn_01x02_Pin, J10 Screw_Terminal_01x02, J11 Conn_01x03_Pin, J12 Conn_01x03_Pin, J15 Screw_Terminal_01x02, J16 Screw_Terminal_01x02, J2 BAT2, J3 Screw_Terminal_01x02, J4 Screw_Terminal_01x02, J5 24V_out, J6 Conn_01x02_Pin, J7 Screw_Terminal_01x02, J8 BAT1, Q1 FDS6681Z, Q2 FDS6681Z, Q3 BC847, Q4 FDS6681Z, Q5 SIS468DN-T1-GE3, Q7 SIS468DN-T1-GE3, U1 INA3221, U2 LDD-700LS, U3 MAX17506ATP+T, U4 TL431DBZ, U5 MAX17506ATP+T, U6 LDD-700LS, U7 B2B pins, U8 DRV8212P, U9 DRV8212P

Commit message: exported files, working on BOM orders
Parts:
- moved TP2 0.10 mm to (109.0, 53.8)
- moved D1 0.10 mm to (106.2, 51.8)
- moved D2 0.10 mm to (106.2, 53.8)
- moved D3 0.10 mm to (106.2, 55.8)
- moved R10 0.10 mm to (102.4, 51.8)
- moved R11 0.10 mm to (102.4, 53.8)
- moved R12 0.10 mm to (102.4, 55.8)
- moved TP1 0.10 mm to (109.0, 51.8)
- moved TP3 0.10 mm to (109.0, 55.8)
Other:
- board text added: "12V"
- board text added: "3V3"
- board text added: "5V"
- board text added: "IND"
Changed lines of the file:
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@@
 		(grid_origin 100 100)
 		(pcbplotparams
-			(layerselection 0x00000000_00000000_00000000_000000a5)
+			(layerselection 0x00000000_00000000_55555555_5755f5ff)
 			(plot_on_all_layers_selection 0x00000000_00000000_00000000_00000000)
 			(disableapertmacros no)
 			(usegerberextensions yes)
-			(usegerberattributes no)
-			(usegerberadvancedattributes no)
-			(creategerberjobfile no)
+			(usegerberattributes yes)
+			(usegerberadvancedattributes yes)
+			(creategerberjobfile yes)
 			(dashed_line_dash_ratio 12)
 			(dashed_line_gap_ratio 3)
@@
 			(plotpadnumbers no)
 			(hidednponfab no)
-			(sketchdnponfab yes)
-			(crossoutdnponfab yes)
+			(sketchdnponfab no)
+			(crossoutdnponfab no)
 			(subtractmaskfromsilk no)
 			(outputformat 1)
 			(mirror no)
-			(drillshape 1)
+			(drillshape 0)
 			(scaleselection 1)
-			(outputdirectory "")
+			(outputdirectory "Fabrication outputs/NC Drill/")
 		)
 	)
@@
 	(footprint "TestPoint:TestPoint_Pad_D1.0mm"
 		(layer "F.Cu")
-		(at 109.0125 55.9 90)
+		(at 109.0125 55.8 90)
 		(descr "SMD pad as test Point, diameter 1.0mm")
 		(tags "test point SMD pad")
@@
 	(footprint "Resistor_SMD:R_0603_1608Metric_Pad0.98x0.95mm_HandSolder"
 		(layer "F.Cu")
-		(at 102.4125 53.9 180)
+		(at 102.4125 53.8 180)
 		(descr "Resistor SMD 0603 (1608 Metric), square (rectangular) end terminal, IPC-7351 nominal with elongated pad for handsoldering. (Body size source: IPC-SM-782 page 72, https://www.pcb-3d.com/wordpress/wp-content/uploads/ipc-sm-782a_amendment_1_and_2.pdf)")
 		(tags "resistor handsolder")
@@
 	(footprint "TestPoint:TestPoint_Pad_D1.0mm"
 		(layer "F.Cu")
-		(at 109.0125 51.9 90)
+		(at 109.0125 51.8 90)
 		(descr "SMD pad as test Point, diameter 1.0mm")
 		(tags "test point SMD pad")
@@
 	(footprint "Resistor_SMD:R_0603_1608Metric_Pad0.98x0.95mm_HandSolder"
 		(layer "F.Cu")
-		(at 102.4125 51.9 180)
+		(at 102.4125 51.8 180)
 		(descr "Resistor SMD 0603 (1608 Metric), square (rectangular) end terminal, IPC-7351 nominal with elongated pad for handsoldering. (Body size source: IPC-SM-782 page 72, https://www.pcb-3d.com/wordpress/wp-content/uploads/ipc-sm-782a_amendment_1_and_2.pdf)")
 		(tags "resistor handsolder")
@@
 	(footprint "TestPoint:TestPoint_Pad_D1.0mm"
 		(layer "F.Cu")
-		(at 109.0125 53.9 90)
+		(at 109 53.8 90)
 		(descr "SMD pad as test Point, diameter 1.0mm")
 		(tags "test point SMD pad")
@@
 	(footprint "Resistor_SMD:R_0603_1608Metric_Pad0.98x0.95mm_HandSolder"
 		(layer "F.Cu")
-		(at 102.4125 55.9 180)
+		(at 102.4125 55.8 180)
 		(descr "Resistor SMD 0603 (1608 Metric), square (rectangular) end terminal, IPC-7351 nominal with elongated pad for handsoldering. (Body size source: IPC-SM-782 page 72, https://www.pcb-3d.com/wordpress/wp-content/uploads/ipc-sm-782a_amendment_1_and_2.pdf)")
 		(tags "resistor handsolder")
@@
 	(footprint "LED_SMD:LED_0603_1608Metric_Pad1.05x0.95mm_HandSolder"
 		(layer "F.Cu")
-		(at 106.2125 53.9)
+		(at 106.2125 53.8)
 		(descr "LED SMD 0603 (1608 Metric), square (rectangular) end terminal, IPC-7351 nominal, (Body size source: http://www.tortai-tech.com/upload/download/2011102023233369053.pdf), generated with kicad-footprint-generator")
 		(tags "LED handsolder")
@@
 	(footprint "LED_SMD:LED_0603_1608Metric_Pad1.05x0.95mm_HandSolder"
 		(layer "F.Cu")
-		(at 106.2125 55.9)
+		(at 106.2125 55.8)
 		(descr "LED SMD 0603 (1608 Metric), square (rectangular) end terminal, IPC-7351 nominal, (Body size source: http://www.tortai-tech.com/upload/download/2011102023233369053.pdf), generated with kicad-footprint-generator")
 		(tags "LED handsolder")
@@
 	(footprint "LED_SMD:LED_0603_1608Metric_Pad1.05x0.95mm_HandSolder"
 		(layer "F.Cu")
-		(at 106.2125 51.9)
+		(at 106.2125 51.8)
 		(descr "LED SMD 0603 (1608 Metric), square (rectangular) end terminal, IPC-7351 nominal, (Body size source: http://www.tortai-tech.com/upload/download/2011102023233369053.pdf), generated with kicad-footprint-generator")
 		(tags "LED handsolder")
@@
 		(layer "Dwgs.User")
 	)
+	(gr_text "3V3"
+		(at 110.4 52.2 0)
+		(layer "F.SilkS")
+		(effects
+			(font
+				(size 0.6 0.6)
+				(thickness 0.15)
+			)
+			(justify left bottom)
+		)
+	)
+	(gr_text "5V"
+		(at 110.4 54.2 0)
+		(layer "F.SilkS")
+		(effects
+			(font
+				(size 0.6 0.6)
+				(thickness 0.15)
+			)
+			(justify left bottom)
+		)
+	)
+	(gr_text "12V"
+		(at 110.4 56.2 0)
+		(layer "F.SilkS")
+		(effects
+			(font
+				(size 0.6 0.6)
+				(thickness 0.15)
+			)
+			(justify left bottom)
+		)
+	)
+	(gr_text "24V"
+		(at 110.4 58.2 0)
+		(layer "F.SilkS")
+		(effects
+			(font
+				(size 0.6 0.6)
+				(thickness 0.15)
+			)
+			(justify left bottom)
+		)
+	)
+	(gr_text "IND"
+		(at 158.2 91.4 0)
+		(layer "F.SilkS")
+		(effects
+			(font
+				(size 0.6 0.6)
+				(thickness 0.15)
+			)
+			(justify left bottom)
+		)
+	)
 	(gr_text "BAT 2\n"
 		(at 128.4 87 0)
@@
 	)
 	(gr_text "SWITCH"
-		(at 107.86 99.02 90)
+		(at 107.2 98.2 90)
 		(layer "F.SilkS")
 		(effects
@@
 	)
 	(gr_text "24V\n\n"
-		(at 114 69.5 90)
+		(at 114 69.2 90)
 		(layer "F.SilkS")
 		(effects
@@
 	)
 	(gr_text "LED1"
-		(at 157 65.005 90)
+		(at 157 65.6 90)
 		(layer "F.SilkS")
 		(effects
@@
 	)
 	(gr_text "LED2\n"
-		(at 157 73.005 90)
+		(at 157 73.2 90)
 		(layer "F.SilkS")
 		(effects
@@
 	)
 	(gr_text "ACT1\n"
-		(at 157 80.005 90)
+		(at 157 80.4 90)
 		(layer "F.SilkS")
 		(effects
@@
 	)
 	(gr_text "ACT2\n\n"
-		(at 158.5 88.005 90)
+		(at 158.6 88 90)
 		(layer "F.SilkS")
 		(effects
@@
 	)
 	(gr_text "ALTAIR Power HAT\nBen D'Agnillo\nMarch 2026 - v1.0"
-		(at 106.4 49.4 0)
+		(at 106.4 49.6 0)
 		(layer "B.SilkS")
 		(effects
@@
 	)
 	(via
-		(at 134.5 73.65)
+		(at 135 73.65)
 		(size 0.6)
 		(drill 0.3)
@@
 	)
 	(via
-		(at 133.5 73.65)
+		(at 134 73.65)
 		(size 0.6)
 		(drill 0.3)
@@
 	)
 	(via
-		(at 135.5 73.65)
+		(at 136 73.65)
 		(size 0.6)
 		(drill 0.3)
@@
 	)
 	(segment
-		(start 110.4 57.2875)
-		(end 110.4 60)
+		(start 109.5 55.9)
+		(end 110.4 56.8)
 		(width 0.254)
 		(layer "F.Cu")
@@
 	(segment
 		(start 109.0125 55.9)
-		(end 107.0875 55.9)
+		(end 109.5 55.9)
 		(width 0.254)
 		(layer "F.Cu")
@@
 	)
 	(segment
-		(start 109.0125 55.9)
-		(end 110.4 57.2875)
+		(start 109.0125 55.8)
+		(end 107.0875 55.8)
+		(width 0.254)
+		(layer "F.Cu")
+		(net "+12V")
+	)
+	(segment
+		(start 110.4 56.8)
+		(end 110.4 60)
 		(width 0.254)
 		(layer "F.Cu")
@@
 	)
 	(segment
-		(start 105.3375 53.9)
-		(end 103.325 53.9)
+		(start 105.3375 53.8)
+		(end 103.325 53.8)
 		(width 0.254)
 		(layer "F.Cu")
@@
 	)
 	(segment
-		(start 109.0125 51.9)
-		(end 107.0875 51.9)
+		(start 109.0125 51.8)
+		(end 107.0875 51.8)
 		(width 0.254)
 		(layer "F.Cu")
@@
 	)
 	(segment
-		(start 105.3375 51.9)
-		(end 103.325 51.9)
+		(start 105.3375 51.8)
+		(end 103.325 51.8)
 		(width 0.254)
 		(layer "F.Cu")
@@
 	)
 	(segment
+		(start 125.42814 88.27814)
+		(end 127.15 90)
+		(width 1.2)
+		(layer "F.Cu")
+		(net "/VBAT2+")
+	)
+	(segment
+		(start 125.42814 84.555348)
+		(end 125.42814 88.27814)
+		(width 1.2)
+		(layer "F.Cu")
+		(net "/VBAT2+")
+	)
+	(segment
 		(start 160.0175 70.4875)
 		(end 160.5 70.005)
@@
 	)
 	(segment
-		(start 137.125 55.405)
+		(start 139.06 55.6)
 		(end 139.255 55.405)
 		(width 1)
@@
 	)
 	(segment
+		(start 137.32 55.6)
+		(end 139.06 55.6)
+		(width 1)
+		(layer "F.Cu")
+		(net "Net-(J6-Pin_2)")
+	)
+	(segment
 		(start 150.89 61)
 		(end 149.425 62.465)
@@
 	(segment
 		(start 135.65 53.93)
-		(end 137.125 55.405)
+		(end 137.32 55.6)
 		(width 1)
 		(layer "F.Cu")
@@
 	)
 	(segment
-		(start 125.42814 88.27814)
-		(end 127.15 90)
-		(width 1.2)
-		(layer "F.Cu")
-		(net "/VBAT2+")
-	)
-	(segment
-		(start 125.42814 84.555348)
-		(end 125.42814 88.27814)
-		(width 1.2)
-		(layer "F.Cu")
-		(net "/VBAT2+")
-	)
-	(segment
-		(start 109.0125 53.9)
-		(end 110.3 53.9)
+		(start 109.0125 53.8)
+		(end 110.3 53.8)
 		(width 0.254)
 		(layer "F.Cu")
@@
 	)
 	(segment
-		(start 110.3 53.9)
-		(end 110.8 54.4)
+		(start 110.3 53.8)
+		(end 110.8 54.3)
 		(width 0.254)
 		(layer "F.Cu")
@@
 	)
 	(segment
-		(start 109.0125 53.9)
-		(end 107.0875 53.9)
+		(start 109.0125 53.8)
+		(end 107.0875 53.8)
 		(width 0.254)
 		(layer "F.Cu")
@@
 	)
 	(via
-		(at 110.8 54.4)
+		(at 110.8 54.3)
 		(size 0.6)
 		(drill 0.3)
@@
 	)
 	(segment
-		(start 105.3375 55.9)
-		(end 103.325 55.9)
+		(start 105.3375 55.8)
+		(end 103.325 55.8)
 		(width 0.254)
 		(layer "F.Cu")

Commit message: ordered
Parts:
- C13, C17, C19, C26, C27, C28, C33, C39, C42, C43, C46, C48, C8: footprint Capacitor_SMD:C_0603_1608Metric_Pad1.08x0.95mm_HandSolder -> Capacitor_SMD:C_0805_2012Metric
- moved C42 4.65 mm to (148.0, 78.4)
- moved C17 2.60 mm to (113.8, 60.8)
- moved C26 1.91 mm to (156.6, 82.2)
- moved C27 1.80 mm to (113.8, 58.0)
- moved C25 1.60 mm to (156.6, 84.0)
- moved C40 1.40 mm to (148.0, 74.6)
- moved C28 1.30 mm to (113.8, 55.6)
- moved R34 1.30 mm to (120.0, 59.2)
- moved C38 1.25 mm to (148.0, 76.4)
- moved C39 1.02 mm to (120.8, 80.6)
- moved C41 0.71 mm to (118.6, 80.6)
- moved C23 0.60 mm to (134.3, 49.0)
- moved C48 0.40 mm to (113.2, 48.0)
- moved C43 0.40 mm to (116.4, 80.6)
- moved C46 0.21 mm to (159.2, 53.2)
Routing:
- net +5V: track 43.0 -> 45.5 mm
- net +12V: track 146.2 -> 148.4 mm
- net +24V: track 24.5 -> 24.8 mm, vias 21 -> 22
- net GND: vias 69 -> 71

Commit message: fixing power board
Parts:
- removed Q3: BC847, Package_TO_SOT_SMD:SOT-23
- removed R3: 10k, Resistor_SMD:R_0603_1608Metric_Pad0.98x0.95mm_HandSolder
- removed R4: 100k, Resistor_SMD:R_0603_1608Metric_Pad0.98x0.95mm_HandSolder
- added R15: 10k, Resistor_SMD:R_0603_1608Metric_Pad0.98x0.95mm_HandSolder, F.Cu at (120.0, 86.5)
- added R38: 10k, Resistor_SMD:R_0603_1608Metric_Pad0.98x0.95mm_HandSolder, F.Cu at (116.5, 81.5)
- R27: value 4.7k -> 10k
- R28: value 100 -> 330
- R29: value 200k -> 1M
- moved R25 3.95 mm to (119.2, 80.5), turned to 90 degrees
- moved R26 3.78 mm to (110.5, 77.8)
- moved R24 3.58 mm to (116.5, 83.2), turned to 0 degrees
- moved R7 3.26 mm to (122.8, 85.5), turned to 90 degrees
- moved D7 2.79 mm to (115.5, 79.5), turned to 180 degrees
- moved R5 2.56 mm to (122.2, 52.8)
- moved D11 1.25 mm to (121.0, 89.8), turned to -90 degrees
- moved C21 0.92 mm to (119.6, 84.8), turned to 180 degrees
- moved R29 0.91 mm to (107.5, 78.5)
- moved R27 0.90 mm to (113.5, 82.5)
- moved R28 0.79 mm to (107.5, 81.5), turned to -90 degrees
- moved R9 0.75 mm to (121.8, 82.8)
- moved C12 0.56 mm to (112.2, 77.8)
- moved U4 0.56 mm to (110.8, 81.8), turned to 180 degrees
- moved D41 0.32 mm to (125.8, 82.1)
Connections:
- D11 pad 1: /VBAT_24V -> Net-(D11-K)
- D7 pad 1: /power/24V_SWITCH -> Net-(D7-K)
- Q4 pad 2: Net-(Q3-C) -> GND
- R5 pad 1: Net-(Q3-C) -> GND
- R5 pad 2: +5V -> /power/5V_SNS-
- U1 pad 6: /I2C_SDA -> /I2C_SCL
- U1 pad 7: /I2C_SCL -> /I2C_SDA
Routing:
- net /power/5V_SNS-: track 31.3 -> 42.4 mm
- net Net-(Q3-B): track 7.90 -> 0.00 mm
- net Net-(Q3-C): track 5.33 -> 0.00 mm
- net Net-(U4-REF): track 9.35 -> 13.7 mm
- net /VBAT_24V: track 2.20 -> 5.70 mm
- net /power/24V_SWITCH: track 11.8 -> 9.50 mm
- net Net-(D7-K): track 0.00 -> 2.27 mm
- net Net-(D7-A): track 12.0 -> 9.79 mm
- net Net-(D11-K): track 0.00 -> 2.04 mm
- net +5V: track 45.5 -> 43.5 mm
- net Net-(D11-A): track 14.0 -> 15.0 mm
- net Net-(Q2-G): track 2.44 -> 1.79 mm
- net Net-(Q1-G): track 5.49 -> 6.09 mm
- net GND: track 7.02 -> 7.00 mm, vias 71 -> 68
Other:
- board text removed: "{ "ViaStitching": "0.4", "stitch_zone_0": { "HSpacing": "3", "VSpacing": "3", "HOffset": "0", "VOffset": "0", "EdgeMargin": "0", "PadMargin": "0", "Clearance": "0", "ViaSize": "0.6", "ViaDrill": "0.3", "Randomize": false, "ClearOwn": true, "IncludeOtherLayers": true, "BlockFootprintZones": true, "AllowUnderPadSameNet": false, "TargetViaCountMode": false, "TargetViaCount": "100", "TargetPattern": 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"

Commit message: power rev 1.1
Parts:
- removed C44: 100nF, Capacitor_SMD:C_0603_1608Metric_Pad1.08x0.95mm_HandSolder
- added C49: 100nF, Capacitor_SMD:C_0603_1608Metric_Pad1.08x0.95mm_HandSolder, F.Cu at (196.5, 77.5)
- added C50: 100nF, Capacitor_SMD:C_0603_1608Metric_Pad1.08x0.95mm_HandSolder, F.Cu at (183.3, 77.6)
- added Q6: IRF7341PBF, Package_SO:SOIC-8_3.9x4.9mm_P1.27mm, F.Cu at (152.8, 64.9)
- added R16: 100, Resistor_SMD:R_0603_1608Metric_Pad0.98x0.95mm_HandSolder, F.Cu at (145.7, 71.8)
- added R17: 0.1, Resistor_SMD:R_2512_6332Metric, F.Cu at (195.8, 93.1)
- added R3: 100, Resistor_SMD:R_0603_1608Metric_Pad0.98x0.95mm_HandSolder, F.Cu at (143.6, 64.4)
- added R6: 0.1, Resistor_SMD:R_2512_6332Metric, F.Cu at (153.3, 58.5)
- added U10: LM358, Package_SO:SOIC-8_3.9x4.9mm_P1.27mm, F.Cu at (139.1, 70.0)
- U2: value LDD-700LS -> INA2180A2IDGKR; footprint LD-700LS:SOP254P1280X930-16N -> INA2180:DGK8_TEX
- U6: value LDD-700LS -> MCP4728; footprint LD-700LS:SOP254P1280X930-16N -> Package_SO:MSOP-10_3x3mm_P0.5mm
- moved C30 47.0 mm to (178.0, 74.4)
- moved U6 19.0 mm to (139.8, 78.9), turned to 180 degrees
- moved U2 12.1 mm to (152.6, 70.7), turned to 0 degrees
- moved J6 7.70 mm to (160.3, 72.7)
- moved J1 7.47 mm to (160.3, 65.1)
- moved JP2 1.29 mm to (156.4, 71.3)
- moved JP3 1.29 mm to (153.8, 71.3)
Connections:
- C30 pad 1: GND -> +3V3
- C30 pad 2: +24V -> GND
- J1 pad 1: Net-(J1-Pin_1) -> +24V
- J6 pad 1: Net-(J6-Pin_1) -> +24V
- U2 pad 1: +24V -> /expansion/LED1_SNS_OUT
- U2 pad 2: Net-(J1-Pin_2) -> GND
- U2 pad 3: Net-(J1-Pin_2) -> /expansion/LED1_SNS+
- U2 pad 4: Net-(J1-Pin_2) -> GND
- U2 pad 5: Net-(J1-Pin_2) -> /expansion/LED2_SNS+
- U2 pad 6: Net-(J1-Pin_2) -> GND
- U2 pad 7: Net-(J1-Pin_1) -> /expansion/LED2_SNS_OUT
- U2 pad 8: Net-(J1-Pin_1) -> +3V3
- U6 pad 1: +24V -> +3V3
- U6 pad 10: Net-(J6-Pin_2) -> GND
- U6 pad 2: Net-(J6-Pin_2) -> /expansion/I2C_SCL
- U6 pad 3: Net-(J6-Pin_2) -> /expansion/I2C_SDA
- U6 pad 4: Net-(J6-Pin_2) -> unconnected-(U6-~{LDAC}-Pad4)
- U6 pad 5: Net-(J6-Pin_2) -> unconnected-(U6-RDY/~{BSY}-Pad5)
- U6 pad 6: Net-(J6-Pin_2) -> /expansion/AOUT_A
- U6 pad 7: Net-(J6-Pin_1) -> /expansion/AOUT_B
- U6 pad 8: Net-(J6-Pin_1) -> /expansion/AOUT_C
- U6 pad 9: Net-(J6-Pin_2) -> /expansion/AOUT_D
Routing:
- net Net-(J6-Pin_2): track 52.1 -> 0.00 mm
- net Net-(J1-Pin_2): track 50.1 -> 0.00 mm
- net /LED_PWM_1: track 36.6 -> 2.84 mm
- net Net-(J1-Pin_1): track 19.9 -> 0.00 mm
- net Net-(J6-Pin_1): track 12.6 -> 0.00 mm
- net +3V3: track 136.2 -> 144.5 mm, vias 7 -> 6
- net /expansion/V_ACT: track 23.2 -> 16.9 mm
- net +24V: track 24.8 -> 28.8 mm, vias 22 -> 20
- net /power/24V_SNS: track 52.8 -> 55.7 mm
- net +12V: track 148.4 -> 149.7 mm, vias 6 -> 5
- net +5V: track 43.5 -> 44.6 mm, vias 35 -> 34
- net Net-(Q6B-G2): track 0.00 -> 0.38 mm, vias 0 -> 1
- net GND: vias 68 -> 53

Commit message: update
Parts:
- removed R15, R38: 10k, Resistor_SMD:R_0603_1608Metric_Pad0.98x0.95mm_HandSolder
- added R30: 10k, Resistor_SMD:R_0603_1608Metric_Pad0.98x0.95mm_HandSolder, F.Cu at (112.5, 81.5)
- moved C49 50.4 mm to (146.8, 69.5), turned to 180 degrees
- moved C50 46.7 mm to (138.4, 65.0)
- moved R17 44.5 mm to (154.0, 78.0), turned to 90 degrees
- moved C30 39.8 mm to (138.2, 75.2), turned to 180 degrees
- moved R6 21.5 mm to (149.0, 79.5), turned to 90 degrees
- moved U6 13.0 mm to (134.0, 67.2), turned to -90 degrees
- moved U2 12.4 mm to (142.2, 77.5), turned to 90 degrees
- moved R25 10.0 mm to (109.4, 78.5), turned to 180 degrees
- moved R3 8.86 mm to (147.2, 72.5)
- moved U4 6.97 mm to (117.5, 80.0), turned to -90 degrees
- moved D7 5.71 mm to (110.2, 81.8), turned to 90 degrees
- moved R24 5.67 mm to (113.4, 78.5), turned to 180 degrees
- moved R16 4.43 mm to (146.8, 67.5)
- moved Q6 3.70 mm to (151.9, 68.5), turned to 90 degrees
- moved R7 3.58 mm to (122.0, 82.0), turned to 180 degrees
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Connections:
- C21 pad 2: Net-(Q1-G) -> Net-(D11-A)
- D11 pad 1: Net-(D11-K) -> /VBAT_24V
- D7 pad 1: Net-(D7-K) -> /power/24V_SWITCH
- J11 pad 1: +5V -> /SERVO_1
- J11 pad 2: /SERVO_1 -> +5V
- J12 pad 1: +5V -> /SERVO_2
- J12 pad 2: /SERVO_2 -> +5V
- J16 pad 2: Net-(D11-A) -> Net-(J16-Pin_2)
- Q1 pad 2: Net-(Q1-G) -> Net-(D11-A)
- R27 pad 2: Net-(D7-A) -> Net-(U4-K)
- R9 pad 1: Net-(D11-A) -> Net-(J16-Pin_2)
- R9 pad 2: Net-(Q1-G) -> Net-(D11-A)
- U10 pad 1: Net-(R3-Pad1) -> Net-(R16-Pad1)
- U10 pad 2: /expansion/LED1_SNS_OUT -> /expansion/LED2_SNS_OUT
- U10 pad 3: /expansion/AOUT_A -> /expansion/AOUT_B
- U10 pad 5: /expansion/AOUT_B -> /expansion/AOUT_A
- U10 pad 6: /expansion/LED2_SNS_OUT -> /expansion/LED1_SNS_OUT
- U10 pad 7: Net-(R16-Pad1) -> Net-(R3-Pad1)
- U2 pad 1: /expansion/LED1_SNS_OUT -> /expansion/LED2_SNS_OUT
- U2 pad 3: /expansion/LED1_SNS+ -> /expansion/LED2_SNS+
- U2 pad 5: /expansion/LED2_SNS+ -> /expansion/LED1_SNS+
- U2 pad 7: /expansion/LED2_SNS_OUT -> /expansion/LED1_SNS_OUT
- U4 pad 1: Net-(D7-A) -> Net-(U4-K)
- U6 pad 2: /expansion/I2C_SCL -> /I2C_SCL
- U6 pad 3: /expansion/I2C_SDA -> /I2C_SDA
- U6 pad 4: unconnected-(U6-~{LDAC}-Pad4) -> /LED_PWM_1
Routing:
- net /LED_PWM_1: track 2.84 -> 34.6 mm
- net /LED_PWM_2: track 27.6 -> 0.00 mm, vias 1 -> 0
- net /expansion/LED2_SNS+: track 0.00 -> 19.6 mm
- net +3V3: track 144.5 -> 163.6 mm, vias 6 -> 7
- net /I2C_SDA: track 30.3 -> 48.7 mm, vias 0 -> 1
- net /expansion/LED2_SNS_OUT: track 0.00 -> 14.4 mm
- net /I2C_SCL: track 28.3 -> 42.3 mm, vias 0 -> 2
- net /expansion/LED1_SNS+: track 0.00 -> 13.5 mm
- net /expansion/AOUT_A: track 0.00 -> 13.0 mm
- net Net-(J1-Pin_2): track 0.00 -> 12.1 mm
- net Net-(J16-Pin_2): track 0.00 -> 11.0 mm
- net Net-(J6-Pin_2): track 0.00 -> 9.49 mm
- net Net-(U4-K): track 0.00 -> 8.71 mm
- net /expansion/LED1_SNS_OUT: track 0.00 -> 8.69 mm
- net Net-(R16-Pad1): track 0.00 -> 7.87 mm
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
Commit message: jlc order
Parts:
- removed C23, C24: 100nF, Capacitor_SMD:C_0603_1608Metric_Pad1.08x0.95mm_HandSolder
- added C2: 100nF, Capacitor_SMD:C_0603_1608Metric_Pad1.08x0.95mm_HandSolder, F.Cu at (147.0, 53.8)
- added J20: Conn_01x04_Socket, Connector_JST:JST_GH_SM04B-GHS-TB_1x04-1MP_P1.25mm_Horizontal, F.Cu at (160.5, 55.3)
- added U11: ADS1113IDGS, Package_SO:TSSOP-10_3x3mm_P0.5mm, F.Cu at (152.5, 54.5)
- C45, C46: moved to B.Cu
- J1, J6: value Conn_01x02_Pin -> Conn_01x04_Socket; footprint Terminal_Block_Custom:1x02_P2.54mm_Horizontal -> Connector_JST:JST_GH_SM04B-GHS-TB_1x04-1MP_P1.25mm_Horizontal
- U4: footprint Package_TO_SOT_SMD:SOT-23 -> TL431:DBZ0003A_L
- moved R14 45.7 mm to (154.5, 47.5), turned to 90 degrees
- moved D5 43.7 mm to (156.8, 47.5), turned to -90 degrees
- moved C46 6.93 mm to (155.2, 47.5), turned to 90 degrees
- moved C45 4.32 mm to (157.2, 47.5), turned to -90 degrees
- moved J4 4.06 mm to (151.3, 48.0)
- moved J11 4.00 mm to (128.3, 48.0)
- moved J15 3.88 mm to (144.3, 48.0)
- moved J12 3.82 mm to (137.5, 48.0)
- moved J3 3.75 mm to (160.5, 83.8)
- moved J7 3.25 mm to (160.5, 90.8)
- moved J6 1.56 mm to (160.5, 74.2)
- moved C30 1.25 mm to (138.2, 76.5), turned to -90 degrees
- moved J1 0.37 mm to (160.5, 64.8)
Connections:
- J1 pad 2: Net-(J1-Pin_2) -> +24V
- J6 pad 2: Net-(J6-Pin_2) -> +24V
- Q6 pad 5: Net-(J6-Pin_2) -> Net-(J6-Pin_3)
- Q6 pad 6: Net-(J6-Pin_2) -> Net-(J6-Pin_3)
- Q6 pad 7: Net-(J1-Pin_2) -> Net-(J1-Pin_3)
- Q6 pad 8: Net-(J1-Pin_2) -> Net-(J1-Pin_3)
Routing:
- net /IND: track 40.1 -> 8.00 mm
- net +5V: track 45.4 -> 64.8 mm, vias 35 -> 4
- net /I2C_SCL: track 42.3 -> 61.5 mm
- net Net-(J1-Pin_2): track 12.1 -> 0.00 mm
- net Net-(J6-Pin_3): track 0.00 -> 11.3 mm
- net Net-(J1-Pin_3): track 0.00 -> 11.3 mm
- net /I2C_SDA: track 48.7 -> 59.4 mm, vias 1 -> 2
- net Net-(J6-Pin_2): track 9.49 -> 0.00 mm
- net /expansion/V_ACT: track 21.9 -> 28.9 mm, vias 2 -> 0
- net +24V: track 21.2 -> 27.0 mm, vias 19 -> 21
- net /expansion/NTC_DIFF-: track 0.00 -> 5.71 mm
- net /MOTOR_1_B: track 39.8 -> 35.3 mm, vias 0 -> 2
- net /expansion/NTC_DIFF+: track 0.00 -> 3.95 mm
- net /MOTOR_1_A: track 41.4 -> 37.4 mm, vias 0 -> 2
- net Net-(J3-Pin_1): track 4.58 -> 8.06 mm
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Other:
- board text added: "-"
- board text added: "NTC"

Commit message: still trying to order. last minute fixes
Parts:
- removed J10: Screw_Terminal_01x02, Terminal_Block_Custom:1x02_P2.54mm_Horizontal
- moved F1 1.00 mm to (121.2, 89.8)
Connections:
- J16 pad 1: /VBAT_24V -> GND
Routing:
- net /VBAT_24V: track 9.24 -> 9.06 mm, vias 0 -> 9
