File: power_db_hat/power.kicad_sch (KiCad schematic)
At the start: 23 parts, among them J10 Screw_Terminal_01x02, J16 Screw_Terminal_01x02, Q2 AO4407A, Q3 AO4407A, U4 TL431DBZ

Commit message: lol
Parts:
- J10, J16: footprint TerminalBlock:TerminalBlock_MaiXu_MX126-5.0-02P_1x02_P5.00mm -> TerminalBlock:TerminalBlock_Xinya_XY308-2.54-2P_1x02_P2.54mm_Horizontal
- Q2, Q3: footprint (none) -> Package_SO:SOIC-8-1EP_3.9x4.9mm_P1.27mm_EP2.41x3.81mm
Changed lines of the file:
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@@
 			)
 		)
-		(property "Footprint" "TerminalBlock:TerminalBlock_MaiXu_MX126-5.0-02P_1x02_P5.00mm"
+		(property "Footprint" "TerminalBlock:TerminalBlock_Xinya_XY308-2.54-2P_1x02_P2.54mm_Horizontal"
 			(at 72.39 44.45 0)
 			(hide yes)
@@
 			)
 		)
-		(property "Footprint" ""
+		(property "Footprint" "Package_SO:SOIC-8-1EP_3.9x4.9mm_P1.27mm_EP2.41x3.81mm"
 			(at 238.76 39.37 0)
 			(hide yes)
@@
 			)
 		)
-		(property "Footprint" "TerminalBlock:TerminalBlock_MaiXu_MX126-5.0-02P_1x02_P5.00mm"
+		(property "Footprint" "TerminalBlock:TerminalBlock_Xinya_XY308-2.54-2P_1x02_P2.54mm_Horizontal"
 			(at 55.88 36.83 0)
 			(hide yes)
@@
 			)
 		)
-		(property "Footprint" ""
+		(property "Footprint" "Package_SO:SOIC-8-1EP_3.9x4.9mm_P1.27mm_EP2.41x3.81mm"
 			(at 118.11 46.99 0)
 			(hide yes)

Commit message: update
Parts:
- removed D16: TVS_26V, Diode_SMD:D_0603_1608Metric_Pad1.05x0.95mm_HandSolder, symbol Device:D_Zener
- removed D52, D6: D_Schottky, Diode_SMD:D_SMA-SMB_Universal_Handsoldering, symbol Device:D_Schottky
- removed Q3: AO4407A, Package_SO:SOIC-8-1EP_3.9x4.9mm_P1.27mm_EP2.41x3.81mm, symbol Simulation_SPICE:PMOS
- added D11: D_Zener, Diode_SMD:D_0603_1608Metric_Pad1.05x0.95mm_HandSolder, symbol Device:D_Zener
- added Q1, Q4: FDS6681Z, FDS6681Z:FDS6681Z_SOP-8, symbol Simulation_SPICE:PMOS
- added Q3: BC847, Package_TO_SOT_SMD:SOT-23, symbol Transistor_BJT:BC847
- added R3: 10k, symbol Device:R_US
- added R4, R5: 100k, symbol Device:R_US
- D7: value TVS_26V -> D_Zener; footprint Diode_SMD:D_SMA-SMB_Universal_Handsoldering -> Diode_SMD:D_0603_1608Metric_Pad1.05x0.95mm_HandSolder
- Q2: value AO4407A -> FDS6681Z; footprint Package_SO:SOIC-8-1EP_3.9x4.9mm_P1.27mm_EP2.41x3.81mm -> FDS6681Z:FDS6681Z_SOP-8
Connections:
- net 24V_SNS: now also Q2.3 (D); no longer Q2.1 (D)
- net 24V_SWITCH: now also D7.1 (K), Q2.1 (S), Q1.3 (D); no longer D7.2 (A), Q2.3 (S)
- net 5V_SNS: now also Q4.3 (D), R5.2
- net GND: now also Q3.2 (E), R4.1
- net VIN_24V: now also J16.1 (Pin_1), D11.1 (K), Q1.1 (S); no longer J16.2 (Pin_2)
- net bucks/BUCK_OUT_5V: now also Q4.1 (S), R3.2
- net at D43.1 (K), R7.2, R9.1: now also J16.2 (Pin_2), D11.2 (A); no longer J16.1 (Pin_1)
- net at R27.2, R28.1, U4.1 (K): now also D7.2 (A); no longer D7.1 (K)
- net at C21.2, R9.2: now also Q1.2 (G)
- new net: Q3.1 (B), R3.1, R4.2
- new net: Q3.3 (C), Q4.2 (G), R5.1
Other:
- note added: "18V Zener"
- note added: "24V supply low voltage disconnect"
- note removed: "12V supply low voltage disconnect"
- moved on the sheet: J16

Commit message: lol
Parts:
- R3, R4, R5: footprint (none) -> Resistor_SMD:R_0603_1608Metric_Pad0.98x0.95mm_HandSolder
Changed lines of the file:
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@@
 			)
 		)
-		(property "Footprint" ""
+		(property "Footprint" "Resistor_SMD:R_0603_1608Metric_Pad0.98x0.95mm_HandSolder"
 			(at 72.644 121.666 90)
 			(hide yes)
@@
 			)
 		)
-		(property "Footprint" ""
+		(property "Footprint" "Resistor_SMD:R_0603_1608Metric_Pad0.98x0.95mm_HandSolder"
 			(at 105.664 119.126 90)
 			(hide yes)
@@
 			)
 		)
-		(property "Footprint" ""
+		(property "Footprint" "Resistor_SMD:R_0603_1608Metric_Pad0.98x0.95mm_HandSolder"
 			(at 72.644 133.096 90)
 			(hide yes)

Commit message: LMAO
Connections:
- net 5V_SNS renamed +5V
Other:
- sheet bucks ports: added 12V_SNS+, 12V_SNS-, 5V_SNS+, 5V_SNS-; removed none
- sheet current/voltage_monitor ports: added 12V_SNS+, 12V_SNS-, 5V_SNS+, 5V_SNS-; removed 5V_IN
- note added: "Prevent rail contention"

Commit message: updated 3d models for power
Parts:
- J10, J16: footprint TerminalBlock:TerminalBlock_Xinya_XY308-2.54-2P_1x02_P2.54mm_Horizontal -> Terminal_Block_Custom:1x02_P2.54mm_Horizontal
Changed lines of the file:
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@@
 			)
 		)
-		(property "Footprint" "TerminalBlock:TerminalBlock_Xinya_XY308-2.54-2P_1x02_P2.54mm_Horizontal"
+		(property "Footprint" "Terminal_Block_Custom:1x02_P2.54mm_Horizontal"
 			(at 72.39 41.91 0)
 			(hide yes)
@@
 			)
 		)
-		(property "Footprint" "TerminalBlock:TerminalBlock_Xinya_XY308-2.54-2P_1x02_P2.54mm_Horizontal"
+		(property "Footprint" "Terminal_Block_Custom:1x02_P2.54mm_Horizontal"
 			(at 55.88 36.83 0)
 			(hide yes)

Commit message: working on BOM
Changed lines of the file:
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@@
 	(text "18V Zener"
 		(exclude_from_sim no)
-		(at 100.076 28.702 0)
+		(at 97.79 31.496 0)
 		(effects
 			(font

Commit message: complete BOM
Parts:
- removed D15, D43: TVS_26V, Diode_SMD:D_0603_1608Metric_Pad1.05x0.95mm_HandSolder, symbol Device:D_Zener
- D11, D7: footprint Diode_SMD:D_0603_1608Metric_Pad1.05x0.95mm_HandSolder -> Diode_SMD:D_SOD-323_HandSoldering

Commit message: lol
Parts:
- R28: value 100 -> 330
Other:
- note added: "Switch J16: Float → OFF GND → ON (~46mA) R28 (330Ω) limits LVD gate inrush 1.5kΩ on pin 2 required - no series resistor on D11, direct short will destroy it TODO rev: add series resistor in series with D11 cathode to source to limit zener current"
- note added: "TL431 reference and cathode pins are reversed in the footprint. FIX THIS"
- note removed: "Short pin 1 to pin 2 (VDD) for OFF Short pin 1 to GND for ON"
Changed lines of the file:
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@@
-		)
-	)
-	(text "TODO simulate\n"
-		(exclude_from_sim no)
-		(at 53.848 64.516 0)
-		(effects
-			(font
-				(size 1.27 1.27)
-			)
 		)
 	)
@@
 		)
 	)
-	(text "Short pin 1 to pin 2 (VDD) for OFF\nShort pin 1 to GND for ON"
+	(text "Switch J16:\n\nFloat → OFF\nGND → ON (~46mA)\n\nR28 (330Ω) limits LVD gate inrush\n1.5kΩ on pin 2 required - no series resistor on D11, direct short will destroy it\nTODO rev: add series resistor in series with D11 cathode to source to limit zener current\n"
 		(exclude_from_sim no)
-		(at 54.102 72.644 0)
+		(at 146.812 70.358 0)
+		(effects
+			(font
+				(size 1.27 1.27)
+			)
+		)
+	)
+	(text "TL431 reference and cathode pins are reversed in the footprint. FIX THIS"
+		(exclude_from_sim no)
+		(at 222.504 78.74 0)
 		(effects
 			(font
@@
 			)
 		)
-		(property "Value" "100"
+		(property "Value" "330"
 			(at 232.664 57.912 90)
 			(show_name no)
