File: power_db_hat/power.kicad_sch (KiCad schematic)
At the start: 24 parts, among them J10 Screw_Terminal_01x02, J16 Screw_Terminal_01x02, Q1 FDS6681Z, Q2 FDS6681Z, Q3 BC847, Q4 FDS6681Z, U4 TL431DBZ

Commit message: bringup updates
Parts:
- added R30: 10k, Resistor_SMD:R_0603_1608Metric_Pad0.98x0.95mm_HandSolder, symbol Device:R_US
- R27: value 4.7k -> 10k
- R29: value 200k -> 1M
Connections:
- net +5V: no longer R5.2
- net GND: now also R5.1; no longer Q3.2 (E)
- net at R3.1, R4.2: no longer Q3.1 (B)
- net at D7.2 (A), R27.2, R28.1: now also R30.1; no longer U4.1 (K)
- new net: R30.2, U4.1 (K)
- new net: Q4.2 (G), R5.2
- now unconnected: Q3.3 (C)
Other:
- note added: "1M measured to disconnect from ON state at roughly 20.7V"
- note added: "Prevent rail contention when 5V powered externally"
- note added: "Replaced R27 with 10k from 4.7k to reduce current due to excess heat dissipation before"
- note added: "Switch J16: Float → OFF GND → ON (~46mA, no load) R28 (330Ω) limits LVD gate inrush 10kΩ on pin 2 required - no series resistor on D11, direct short will destroy it TODO rev: add series resistor in series with D11 cathode to source to limit zener current"
- note removed: "Prevent rail contention"
- note removed: "Switch J16: Float → OFF GND → ON (~46mA) R28 (330Ω) limits LVD gate inrush 1.5kΩ on pin 2 required - no series resistor on D11, direct short will destroy it TODO rev: add series resistor in series with D11 cathode to source to limit zener current"
- moved on the sheet: D7, R27, R28, U4

Commit message: fixing power board
Parts:
- removed Q3: BC847, Package_TO_SOT_SMD:SOT-23, symbol Transistor_BJT:BC847
- removed R3, R30: 10k, Resistor_SMD:R_0603_1608Metric_Pad0.98x0.95mm_HandSolder, symbol Device:R_US
- removed R4: 100k, Resistor_SMD:R_0603_1608Metric_Pad0.98x0.95mm_HandSolder, symbol Device:R_US
- added R15, R38: 10k, Resistor_SMD:R_0603_1608Metric_Pad0.98x0.95mm_HandSolder, symbol Device:R_US
Connections:
- net bucks/BUCK_OUT_5V is gone; now on net BUCK_OUT_5V: Q4.1 (S)
- net 24V_SWITCH: now also R38.2; no longer D7.1 (K)
- net GND: now also Q4.2 (G)
- net VIN_24V: now also R15.2; no longer D11.1 (K)
- net at D7.2 (A), R27.2, R28.1: now also U4.1 (K)
- net BUCK_OUT_5V: now reaches R5.2
- net BUCK_OUT_5V: no longer Q4.2 (G)
- new net: D7.1 (K), R38.1
- new net: D11.1 (K), R15.1
Other:
- moved on the sheet: C21, R27, R28, R7

Commit message: update
Parts:
- removed R15, R38: 10k, Resistor_SMD:R_0603_1608Metric_Pad0.98x0.95mm_HandSolder, symbol Device:R_US
- added R30: 10k, Resistor_SMD:R_0603_1608Metric_Pad0.98x0.95mm_HandSolder, symbol Device:R_US
Connections:
- net 24V_SWITCH: now also D7.1 (K)
- net VIN_24V: now also D11.1 (K)
- net at J16.2 (Pin_2), R9.1: no longer D11.2 (A), R7.2
- net at D7.2 (A), R28.1: now also R30.1; no longer R27.2, U4.1 (K)
- net at C21.2, Q1.2 (G), R9.2: now also D11.2 (A), R7.2
- new net: R27.2, R30.2, U4.1 (K)
Other:
- note removed: "Replaced R27 with 10k from 4.7k to reduce current due to excess heat dissipation before"
- moved on the sheet: D11, R7

Commit message: jlc order
Parts:
- U4: footprint Package_TO_SOT_SMD:SOT-23 -> TL431:DBZ0003A_L
Changed lines of the file:
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@@
 			)
 		)
-		(property "Footprint" "Package_TO_SOT_SMD:SOT-23"
+		(property "Footprint" "TL431:DBZ0003A_L"
 			(at 219.456 60.96 0)
 			(hide yes)

Commit message: still trying to order. last minute fixes
Parts:
- removed J10: Screw_Terminal_01x02, Terminal_Block_Custom:1x02_P2.54mm_Horizontal, symbol Connector:Screw_Terminal_01x02
Connections:
- net GND: now also J16.1 (Pin_1)
- net VIN_24V: no longer J16.1 (Pin_1)
Other:
- note removed: "extra ground connector to simplify BOM and save space"
- moved on the sheet: J16
Changed lines of the file:
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@@
-		)
-	)
-	(text "extra ground connector to \nsimplify BOM and save space\n"
-		(exclude_from_sim no)
-		(at 54.356 31.496 0)
-		(effects
-			(font
-				(size 1.27 1.27)
-			)
 		)
 	)
@@
 	)
 	(junction
-		(at 85.09 29.21)
-		(diameter 0)
-		(color 0 0 0 0)
-	)
-	(junction
 		(at 199.39 58.42)
 		(diameter 0)
@@
 	)
 	(junction
-		(at 57.15 41.91)
-		(diameter 0)
-		(color 0 0 0 0)
-	)
-	(junction
 		(at 96.52 44.45)
 		(diameter 0)
@@
 	(wire
 		(pts
-			(xy 77.47 41.91) (xy 85.09 41.91)
-		)
-		(stroke
-			(width 0)
-			(type default)
-		)
-	)
-	(wire
-		(pts
 			(xy 214.63 67.31) (xy 248.92 67.31)
 		)
@@
 	(wire
 		(pts
-			(xy 85.09 29.21) (xy 85.09 41.91)
-		)
-		(stroke
-			(width 0)
-			(type default)
-		)
-	)
-	(wire
-		(pts
 			(xy 201.93 111.76) (xy 205.74 111.76)
 		)
@@
 	(wire
 		(pts
-			(xy 57.15 41.91) (xy 58.42 41.91)
-		)
-		(stroke
-			(width 0)
-			(type default)
-		)
-	)
-	(wire
-		(pts
 			(xy 96.52 44.45) (xy 105.41 44.45)
 		)
@@
 		(pts
 			(xy 199.39 67.31) (xy 204.47 67.31)
-		)
-		(stroke
-			(width 0)
-			(type default)
-		)
-	)
-	(wire
-		(pts
-			(xy 55.88 41.91) (xy 57.15 41.91)
 		)
 		(stroke
@@
 	(symbol
 		(lib_id "Connector:Screw_Terminal_01x02")
-		(at 72.39 41.91 0)
-		(mirror y)
+		(at 72.39 46.99 180)
 		(unit 1)
 		(body_style 1)
@@
 		(dnp no)
 		(property "Reference" "J16"
-			(at 72.136 47.752 0)
+			(at 72.136 41.148 0)
 			(show_name no)
 			(do_not_autoplace no)
@@
 		)
 		(property "Value" "Screw_Terminal_01x02"
-			(at 72.39 48.26 0)
+			(at 72.39 40.64 0)
 			(hide yes)
 			(show_name no)
@@
 		)
 		(property "Footprint" "Terminal_Block_Custom:1x02_P2.54mm_Horizontal"
-			(at 72.39 41.91 0)
+			(at 72.39 46.99 0)
 			(hide yes)
 			(show_name no)
@@
 		)
 		(property "Datasheet" ""
-			(at 72.39 41.91 0)
+			(at 72.39 46.99 0)
 			(hide yes)
 			(show_name no)
@@
 		)
 		(property "Description" "Generic screw terminal, single row, 01x02, script generated (kicad-library-utils/schlib/autogen/connector/)"
-			(at 72.39 41.91 0)
+			(at 72.39 46.99 0)
 			(hide yes)
 			(show_name no)
@@
 				(path "/e63e39d7-6ac0-4ffd-8aa3-1841a4541b55/fd5e5e33-5dc6-45b9-b42d-1fb287c03766"
 					(reference "J16")
+					(unit 1)
+				)
+			)
+		)
+	)
+	(symbol
+		(lib_id "power:GND")
+		(at 77.47 46.99 0)
+		(unit 1)
+		(body_style 1)
+		(exclude_from_sim no)
+		(in_bom yes)
+		(on_board yes)
+		(in_pos_files yes)
+		(dnp no)
+		(fields_autoplaced yes)
+		(property "Reference" "#PWR021"
+			(at 77.47 53.34 0)
+			(hide yes)
+			(show_name no)
+			(do_not_autoplace no)
+			(effects
+				(font
+					(size 1.27 1.27)
+				)
+			)
+		)
+		(property "Value" "GND"
+			(at 77.47 52.07 0)
+			(show_name no)
+			(do_not_autoplace no)
+			(effects
+				(font
+					(size 1.27 1.27)
+				)
+			)
+		)
+		(property "Footprint" ""
+			(at 77.47 46.99 0)
+			(hide yes)
+			(show_name no)
+			(do_not_autoplace no)
+			(effects
+				(font
+					(size 1.27 1.27)
+				)
+			)
+		)
+		(property "Datasheet" ""
+			(at 77.47 46.99 0)
+			(hide yes)
+			(show_name no)
+			(do_not_autoplace no)
+			(effects
+				(font
+					(size 1.27 1.27)
+				)
+			)
+		)
+		(property "Description" "Power symbol creates a global label with name \"GND\" , ground"
+			(at 77.47 46.99 0)
+			(hide yes)
+			(show_name no)
+			(do_not_autoplace no)
+			(effects
+				(font
+					(size 1.27 1.27)
+				)
+			)
+		)
+		(pin "1"
+		)
+		(instances
+			(project "power_db_hat"
+				(path "/e63e39d7-6ac0-4ffd-8aa3-1841a4541b55/fd5e5e33-5dc6-45b9-b42d-1fb287c03766"
+					(reference "#PWR021")
 					(unit 1)
 				)
@@
 	)
 	(symbol
-		(lib_id "power:GND")
-		(at 57.15 41.91 0)
-		(unit 1)
-		(body_style 1)
-		(exclude_from_sim no)
-		(in_bom yes)
-		(on_board yes)
-		(in_pos_files yes)
-		(dnp no)
-		(fields_autoplaced yes)
-		(property "Reference" "#PWR044"
-			(at 57.15 48.26 0)
-			(hide yes)
-			(show_name no)
-			(do_not_autoplace no)
-			(effects
-				(font
-					(size 1.27 1.27)
-				)
-			)
-		)
-		(property "Value" "GND"
-			(at 57.15 46.99 0)
-			(show_name no)
-			(do_not_autoplace no)
-			(effects
-				(font
-					(size 1.27 1.27)
-				)
-			)
-		)
-		(property "Footprint" ""
-			(at 57.15 41.91 0)
-			(hide yes)
-			(show_name no)
-			(do_not_autoplace no)
-			(effects
-				(font
-					(size 1.27 1.27)
-				)
-			)
-		)
-		(property "Datasheet" ""
-			(at 57.15 41.91 0)
-			(hide yes)
-			(show_name no)
-			(do_not_autoplace no)
-			(effects
-				(font
-					(size 1.27 1.27)
-				)
-			)
-		)
-		(property "Description" "Power symbol creates a global label with name \"GND\" , ground"
-			(at 57.15 41.91 0)
-			(hide yes)
-			(show_name no)
-			(do_not_autoplace no)
-			(effects
-				(font
-					(size 1.27 1.27)
-				)
-			)
-		)
-		(pin "1"
-		)
-		(instances
-			(project "power_db_hat"
-				(path "/e63e39d7-6ac0-4ffd-8aa3-1841a4541b55/fd5e5e33-5dc6-45b9-b42d-1fb287c03766"
-					(reference "#PWR044")
-					(unit 1)
-				)
-			)
-		)
-	)
-	(symbol
 		(lib_name "PMOS_1")
 		(lib_id "Simulation_SPICE:PMOS")
@@
 					(unit 1)
 				)
-			)
-		)
-	)
-	(symbol
-		(lib_id "Connector:Screw_Terminal_01x02")
-		(at 55.88 36.83 90)
-		(unit 1)
-		(body_style 1)
-		(exclude_from_sim no)
-		(in_bom yes)
-		(on_board yes)
-		(in_pos_files yes)
-		(dnp no)
-		(property "Reference" "J10"
-			(at 53.086 36.83 0)
-			(show_name no)
-			(do_not_autoplace no)
-			(effects
-				(font
-					(size 1.27 1.27)
-				)
-			)
-		)
-		(property "Value" "Screw_Terminal_01x02"
-			(at 62.23 36.83 0)
-			(hide yes)
-			(show_name no)
-			(do_not_autoplace no)
-			(effects
-				(font
-					(size 1.27 1.27)
-				)
-			)
-		)
-		(property "Footprint" "Terminal_Block_Custom:1x02_P2.54mm_Horizontal"
-			(at 55.88 36.83 0)
-			(hide yes)
-			(show_name no)
-			(do_not_autoplace no)
-			(effects
-				(font
-					(size 1.27 1.27)
-				)
-			)
-		)
-		(property "Datasheet" ""
-			(at 55.88 36.83 0)
-			(hide yes)
-			(show_name no)
-			(do_not_autoplace no)
-			(effects
-				(font
-					(size 1.27 1.27)
-				)
-			)
-		)
-		(property "Description" "Generic screw terminal, single row, 01x02, script generated (kicad-library-utils/schlib/autogen/connector/)"
-			(at 55.88 36.83 0)
-			(hide yes)
-			(show_name no)
-			(do_not_autoplace no)
-			(effects
-				(font
-					(size 1.27 1.27)
-				)
-			)
-		)
-		(pin "2"
-		)
-		(pin "1"
-		)
-		(instances
-			(project "power_db_hat"
-				(path "/e63e39d7-6ac0-4ffd-8aa3-1841a4541b55/fd5e5e33-5dc6-45b9-b42d-1fb287c03766"
-					(reference "J10")
-					(unit 1)
-				)
