File: power_db_hat/servos+gpio.kicad_sch (KiCad schematic)
At the start: 26 parts, among them J1 Conn_01x02_Pin, J11 Conn_01x03_Pin, J12 Conn_01x03_Pin, J15 Screw_Terminal_01x02, J3 Screw_Terminal_01x02, J4 Screw_Terminal_01x02, J6 Conn_01x02_Pin, J7 Screw_Terminal_01x02, U2 LDD-700LS, U6 LDD-700LS, U8 DRV8212P, U9 DRV8212P

Commit message: updated 3d models for power
Parts:
- J1, J15, J3, J4, J6, J7: footprint TerminalBlock:TerminalBlock_Xinya_XY308-2.54-2P_1x02_P2.54mm_Horizontal -> Terminal_Block_Custom:1x02_P2.54mm_Horizontal
Changed lines of the file:
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@@
 			)
 		)
-		(property "Footprint" "TerminalBlock:TerminalBlock_Xinya_XY308-2.54-2P_1x02_P2.54mm_Horizontal"
+		(property "Footprint" "Terminal_Block_Custom:1x02_P2.54mm_Horizontal"
 			(at 149.86 130.81 0)
 			(hide yes)
@@
 			)
 		)
-		(property "Footprint" "TerminalBlock:TerminalBlock_Xinya_XY308-2.54-2P_1x02_P2.54mm_Horizontal"
+		(property "Footprint" "Terminal_Block_Custom:1x02_P2.54mm_Horizontal"
 			(at 264.16 101.6 0)
 			(hide yes)
@@
 			)
 		)
-		(property "Footprint" "TerminalBlock:TerminalBlock_Xinya_XY308-2.54-2P_1x02_P2.54mm_Horizontal"
+		(property "Footprint" "Terminal_Block_Custom:1x02_P2.54mm_Horizontal"
 			(at 233.68 34.29 0)
 			(hide yes)
@@
 			)
 		)
-		(property "Footprint" "TerminalBlock:TerminalBlock_Xinya_XY308-2.54-2P_1x02_P2.54mm_Horizontal"
+		(property "Footprint" "Terminal_Block_Custom:1x02_P2.54mm_Horizontal"
 			(at 245.11 62.23 0)
 			(hide yes)
@@
 			)
 		)
-		(property "Footprint" "TerminalBlock:TerminalBlock_Xinya_XY308-2.54-2P_1x02_P2.54mm_Horizontal"
+		(property "Footprint" "Terminal_Block_Custom:1x02_P2.54mm_Horizontal"
 			(at 72.39 132.08 0)
 			(hide yes)
@@
 			)
 		)
-		(property "Footprint" "TerminalBlock:TerminalBlock_Xinya_XY308-2.54-2P_1x02_P2.54mm_Horizontal"
+		(property "Footprint" "Terminal_Block_Custom:1x02_P2.54mm_Horizontal"
 			(at 262.89 137.16 0)
 			(hide yes)

Commit message: ordered
Parts:
- C19, C26: footprint Capacitor_SMD:C_0603_1608Metric_Pad1.08x0.95mm_HandSolder -> Capacitor_SMD:C_0805_2012Metric
Changed lines of the file:
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@@
 			)
 		)
-		(property "Footprint" "Capacitor_SMD:C_0603_1608Metric_Pad1.08x0.95mm_HandSolder"
+		(property "Footprint" "Capacitor_SMD:C_0805_2012Metric"
 			(at 67.31 117.1448 0)
 			(hide yes)
@@
 			)
 		)
-		(property "Footprint" "Capacitor_SMD:C_0603_1608Metric_Pad1.08x0.95mm_HandSolder"
+		(property "Footprint" "Capacitor_SMD:C_0805_2012Metric"
 			(at 142.24 115.8748 0)
 			(hide yes)

Commit message: fixing power board
Parts:
- removed U2, U6: LDD-700LS, LD-700LS:SOP254P1280X930-16N, symbol LDD-700LS:LDD-700LS
- added C49: 100nF, Capacitor_SMD:C_0603_1608Metric_Pad1.08x0.95mm_HandSolder, symbol Device:C
- added JP4, JP6: SolderJumper_2_Open, Jumper:SolderJumper-2_P1.3mm_Open_TrianglePad1.0x1.5mm, symbol Jumper:SolderJumper_2_Open
- added Q3: IRF7309PBF, Package_SO:SOIC-8_3.9x4.9mm_P1.27mm, symbol Transistor_FET:IRF7309PBF
- added R16, R3: 180, Resistor_SMD:R_0603_1608Metric_Pad0.98x0.95mm_HandSolder, symbol Device:R_US
- added R17, R4: 10k, Resistor_SMD:R_0603_1608Metric_Pad0.98x0.95mm_HandSolder, symbol Device:R_US
- added R18, R6: 2, Resistor_SMD:R_0603_1608Metric_Pad0.98x0.95mm_HandSolder, symbol Device:R_US
- added U10, U2: LM358, symbol Amplifier_Operational:LM358
- added U6: MCP4728, Package_SO:MSOP-10_3x3mm_P0.5mm, symbol Analog_DAC:MCP4728
Connections:
- net +12V: now also JP4.1 (A)
- net +24V: now also JP6.1 (A)
- net GND: now also C49.1, R18.1, R6.1, U2.4 (V-), U6.10 (VSS)
- net LED_SUPPLY: now reaches J1.1 (Pin_1)
- net LED_SUPPLY: now also J6.1 (Pin_1), C49.2, JP4.2 (B), JP6.2 (B), U2.8 (V+), U6.1 (VDD)
- net at J1.2 (Pin_2): now also Q3.7 (D1), Q3.8 (D1)
- net at J6.2 (Pin_2): now also Q3.5 (D2), Q3.6 (D2)
- new net: Q3.1 (S1), R4.1, R6.2, U10.2 (-)
- new net: Q3.2 (G1), R3.2, R4.2
- new net: Q3.3 (S2), R17.1, R18.2, U10.6 (-)
- new net: Q3.4 (G2), R16.2, R17.2
- new net: R16.1, U10.7
- new net: R3.1, U10.1
- new net AOUT_A: U10.3 (+), U6.6 (VOUTA)
- new net AOUT_B: U10.5 (+), U6.7 (VOUTB)
- new net AOUT_C: U6.8 (VOUTC)
- new net AOUT_D: U6.9 (VOUTD)
- new net I2C_SCL: U6.2 (SCL)
- new net I2C_SDA: U6.3 (SDA)
Other:
- moved on the sheet: C30, C44, J1, J6

Commit message: power rev 1.1
Parts:
- removed C44: 100nF, Capacitor_SMD:C_0603_1608Metric_Pad1.08x0.95mm_HandSolder, symbol Device:C
- removed JP4, JP6: SolderJumper_2_Open, Jumper:SolderJumper-2_P1.3mm_Open_TrianglePad1.0x1.5mm, symbol Jumper:SolderJumper_2_Open
- removed Q3: IRF7309PBF, Package_SO:SOIC-8_3.9x4.9mm_P1.27mm, symbol Transistor_FET:IRF7309PBF
- removed R18: 2, Resistor_SMD:R_0603_1608Metric_Pad0.98x0.95mm_HandSolder, symbol Device:R_US
- removed R4: 10k, Resistor_SMD:R_0603_1608Metric_Pad0.98x0.95mm_HandSolder, symbol Device:R_US
- added C50: 100nF, Capacitor_SMD:C_0603_1608Metric_Pad1.08x0.95mm_HandSolder, symbol Device:C
- added Q6: IRF7341PBF, Package_SO:SOIC-8_3.9x4.9mm_P1.27mm, symbol Transistor_FET:IRF7341PBF
- added U2: INA2180A2IDGKR, INA2180:DGK8_TEX, symbol INA2180:INA2180A2IDGKR
- R16, R3: value 180 -> 100
- R17: value 10k -> 0.1; footprint Resistor_SMD:R_0603_1608Metric_Pad0.98x0.95mm_HandSolder -> Resistor_SMD:R_2512_6332Metric
- R6: value 2 -> 0.1; footprint Resistor_SMD:R_0603_1608Metric_Pad0.98x0.95mm_HandSolder -> Resistor_SMD:R_2512_6332Metric
- U10: renamed from U2; footprint (none) -> Package_SO:SOIC-8_3.9x4.9mm_P1.27mm
- U10: footprint (none) -> Package_SO:SOIC-8_3.9x4.9mm_P1.27mm
Connections:
- net +24V: now also C49.2, J1.1 (Pin_1), J6.1 (Pin_1), U10.8 (V+); no longer C30.2
- net +3V3: now also C30.1, U6.1 (VDD), C50.1, U2.8 (VS)
- net GND: now also C30.2, R17.1, C50.2, U2.2 (IN-1), U2.4 (GND), U2.6 (IN-2); no longer C30.1
- net LED1_SNS+: now reaches R6.2
- net LED1_SNS+: now also Q6.1 (S1), U2.3 (IN+1); no longer U10.2 (-)
- net at R3.2: now also Q6.2 (G1)
- net LED2_SNS_OUT: now reaches U10.6 (-)
- net LED2_SNS_OUT: now also U2.7 (OUT2); no longer R17.1
- net at R16.2: now also Q6.4 (G2); no longer R17.2
- net at J1.2 (Pin_2): now also Q6.7 (D1), Q6.8 (D1)
- net at J6.2 (Pin_2): now also Q6.5 (D2), Q6.6 (D2)
- removed net LED_SUPPLY: C49.2, J1.1 (Pin_1), J6.1 (Pin_1), U10.8 (V+), U6.1 (VDD)
- new net LED1_SNS_OUT: U10.2 (-), U2.1 (OUT1)
- new net LED2_SNS+: Q6.3 (S2), R17.2, U2.5 (IN+2)
Other:
- moved on the sheet: C10, C19, C20, C23, C24, C25, C26, C49, C5, J1, J11, J12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

Commit message: update
Connections:
- net +5V: now also J11.2 (Pin_2), J12.2 (Pin_2); no longer J11.1 (Pin_1), J12.1 (Pin_1)
- net AOUT_A: now also U10.5 (+); no longer U10.3 (+)
- net AOUT_B: now also U10.3 (+); no longer U10.5 (+)
- net LED1_SNS+: now also U2.5 (IN+2); no longer U2.3 (IN+1)
- net LED1_SNS_OUT: now also U10.6 (-), U2.7 (OUT2); no longer U10.2 (-), U2.1 (OUT1)
- net LED2_SNS+: now also U2.3 (IN+1); no longer U2.5 (IN+2)
- net LED2_SNS_OUT: now also U10.2 (-), U2.1 (OUT1); no longer U10.6 (-), U2.7 (OUT2)
- net PWM_1: now also J11.1 (Pin_1); no longer J11.2 (Pin_2)
- net PWM_2: now also J12.1 (Pin_1); no longer J12.2 (Pin_2)
- net ~{LDAC}: now reaches U6.4 (~{LDAC})
- net at R16.1: now also U10.1; no longer U10.7
- net at R3.1: now also U10.7; no longer U10.1
- no-connect marks 0 -> 1
Other:
- moved on the sheet: C50, U6

Commit message: jlc order
Parts:
- removed C23, C24: 100nF, Capacitor_SMD:C_0603_1608Metric_Pad1.08x0.95mm_HandSolder, symbol Device:C
- removed J1, J6: Conn_01x02_Pin, Terminal_Block_Custom:1x02_P2.54mm_Horizontal, symbol Connector:Conn_01x02_Pin
- added C2: 100nF, Capacitor_SMD:C_0603_1608Metric_Pad1.08x0.95mm_HandSolder, symbol Device:C
- added J1, J20, J6: Conn_01x04_Socket, Connector_JST:JST_GH_SM04B-GHS-TB_1x04-1MP_P1.25mm_Horizontal, symbol Connector:Conn_01x04_Socket
- added U11: ADS1113IDGS, Package_SO:TSSOP-10_3x3mm_P0.5mm, symbol Analog_ADC:ADS1113IDGS
Connections:
- net +24V: now also J1.1 (Pin_1), J1.2 (Pin_2), J6.1 (Pin_1), J6.2 (Pin_2)
- net +5V: now also C2.1, J20.3 (Pin_3), U11.8 (VDD)
- net GND: now also C2.2, J20.2 (Pin_2), U11.3 (GND)
- net I2C_SCL: now also U11.1 (ADDR), U11.10 (SCL)
- net I2C_SDA: now also U11.9 (SDA)
- net at Q6.7 (D1), Q6.8 (D1): now also J1.3 (Pin_3), J1.4 (Pin_4)
- net at Q6.5 (D2), Q6.6 (D2): now also J6.3 (Pin_3), J6.4 (Pin_4)
- new net NTC_DIFF+: J20.4 (Pin_4), U11.5 (AIN1)
- new net NTC_DIFF-: J20.1 (Pin_1), U11.4 (AIN0)
Other:
- moved on the sheet: C30, C49, Q6A, Q6B, R16, R17, R3, R6, U10A, U10B, U10C, U2
