File: power_db_hat/servos+gpio.kicad_sch (KiCad schematic)
At the start: 34 parts, among them J1 Conn_01x04_Socket, J11 Conn_01x03_Pin, J12 Conn_01x03_Pin, J15 Screw_Terminal_01x02, J20 Conn_01x04_Socket, J3 Screw_Terminal_01x02, J4 Screw_Terminal_01x02, J6 Conn_01x04_Socket, J7 Screw_Terminal_01x02, Q6 IRF7341PBF, U10 LM358, U11 ADS1113IDGS, U2 INA2180A2IDGKR, U6 MCP4728, U8 DRV8212P, U9 DRV8212P

Commit message: post 2nd revision update
Other:
- note added: "Delay in 3v3 rail power on causes race condition for current driver"
Changed lines of the file:
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@@
+		)
+	)
+	(text "Delay in 3v3 rail power on causes race condition for current driver"
+		(exclude_from_sim no)
+		(at 119.126 195.58 0)
+		(effects
+			(font
+				(size 1.27 1.27)
+			)
 		)
 	)
