File: interface_db_hat/GPS.kicad_sch (KiCad schematic)
At the start: 9 parts, among them J4 Conn_Coaxial_Small, U1 MAX-M10M-00B

Commit message: lol
Parts:
- U1: footprint MAX-M10M-00B:XCVR_MAX-M10M-00B -> MAX-M10M:XCVR_MAX-M10M-00B
Changed lines of the file:
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@@
 			)
 		)
-		(property "Footprint" "MAX-M10M-00B:XCVR_MAX-M10M-00B"
+		(property "Footprint" "MAX-M10M:XCVR_MAX-M10M-00B"
 			(at 134.62 93.98 0)
 			(effects
