File: interface_db_hat/GPS.kicad_sch (KiCad schematic)
At the start: 9 parts, among them J4 Conn_Coaxial_Small, U1 MAX-M10M-00B

Commit message: complete BOM
Parts:
- C3: value 40pF -> 47pF; footprint Capacitor_SMD:C_0603_1608Metric_Pad1.08x0.95mm_HandSolder -> Capacitor_SMD:C_0402_1005Metric
- U1: footprint MAX-M10M:XCVR_MAX-M10M-00B -> MAXX-M10M:XCVR_MAX-M10M-00B
Changed lines of the file:
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@@
 			)
 		)
-		(property "Footprint" "MAX-M10M:XCVR_MAX-M10M-00B"
+		(property "Footprint" "MAXX-M10M:XCVR_MAX-M10M-00B"
 			(at 134.62 93.98 0)
 			(hide yes)
@@
 			)
 		)
-		(property "Value" "40pF"
+		(property "Value" "47pF"
 			(at 91.44 44.45 90)
 			(show_name no)
@@
 			)
 		)
-		(property "Footprint" "Capacitor_SMD:C_0603_1608Metric_Pad1.08x0.95mm_HandSolder"
+		(property "Footprint" "Capacitor_SMD:C_0402_1005Metric"
 			(at 87.63 50.4952 0)
 			(hide yes)

Commit message: update
Parts:
- L1: footprint Inductor_SMD:L_0603_1608Metric_Pad1.05x0.95mm_HandSolder -> Inductor_SMD:L_0402_1005Metric
Changed lines of the file:
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@@
 			)
 		)
-		(property "Footprint" "Inductor_SMD:L_0603_1608Metric_Pad1.05x0.95mm_HandSolder"
+		(property "Footprint" "Inductor_SMD:L_0402_1005Metric"
 			(at 72.39 45.72 0)
 			(hide yes)

Commit message: update
Other:
- moved on the sheet: J4
Changed lines of the file:
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@@
 	(wire
 		(pts
-			(xy 29.21 49.53) (xy 31.75 49.53)
+			(xy 46.99 49.53) (xy 49.53 49.53)
 		)
 		(stroke
@@
 	(wire
 		(pts
-			(xy 29.21 49.53) (xy 29.21 54.61)
+			(xy 46.99 49.53) (xy 46.99 54.61)
 		)
 		(stroke
@@
 	(wire
 		(pts
-			(xy 36.83 49.53) (xy 72.39 49.53)
+			(xy 54.61 49.53) (xy 72.39 49.53)
 		)
 		(stroke
@@
 	)
 	(label "GPS_SIG"
-		(at 40.64 49.53 0)
+		(at 54.61 49.53 0)
 		(effects
 			(font
@@
 	(symbol
 		(lib_id "Connector:Conn_Coaxial_Small")
-		(at 34.29 49.53 180)
+		(at 52.07 49.53 180)
 		(unit 1)
 		(body_style 1)
@@
 		(fields_autoplaced yes)
 		(property "Reference" "J4"
-			(at 34.8095 43.18 0)
+			(at 52.5895 43.18 0)
 			(show_name no)
 			(do_not_autoplace no)
@@
 		)
 		(property "Value" "Conn_Coaxial_Small"
-			(at 34.8095 45.72 0)
+			(at 52.5895 45.72 0)
 			(show_name no)
 			(do_not_autoplace no)
@@
 		)
 		(property "Footprint" "Connector_Coaxial:SMA_Amphenol_132289_EdgeMount"
-			(at 34.29 49.53 0)
+			(at 52.07 49.53 0)
 			(hide yes)
 			(show_name no)
@@
 		)
 		(property "Datasheet" ""
-			(at 34.29 49.53 0)
+			(at 52.07 49.53 0)
 			(hide yes)
 			(show_name no)
@@
 		)
 		(property "Description" "small coaxial connector (BNC, SMA, SMB, SMC, Cinch/RCA, LEMO, ...)"
-			(at 34.29 49.53 0)
+			(at 52.07 49.53 0)
 			(hide yes)
 			(show_name no)
@@
 	(symbol
 		(lib_id "power:GND")
-		(at 29.21 54.61 0)
+		(at 46.99 54.61 0)
 		(unit 1)
 		(body_style 1)
@@
 		(fields_autoplaced yes)
 		(property "Reference" "#PWR025"
-			(at 29.21 60.96 0)
+			(at 46.99 60.96 0)
 			(hide yes)
 			(show_name no)
@@
 		)
 		(property "Value" "GND"
-			(at 29.21 59.69 0)
+			(at 46.99 59.69 0)
 			(show_name no)
 			(do_not_autoplace no)
@@
 		)
 		(property "Footprint" ""
-			(at 29.21 54.61 0)
+			(at 46.99 54.61 0)
 			(hide yes)
 			(show_name no)
@@
 		)
 		(property "Datasheet" ""
-			(at 29.21 54.61 0)
+			(at 46.99 54.61 0)
 			(hide yes)
 			(show_name no)
@@
 		)
 		(property "Description" "Power symbol creates a global label with name \"GND\" , ground"
-			(at 29.21 54.61 0)
-			(hide yes)
-			(show_name no)
+			(at 46.99 54.61 0)
+			(hide yes)
+			(show_name no)

Commit message: update
Parts:
- C2: LCSC (none) -> C16194197
- C3: KiLib_Generator (none) -> SMD_2terminal_chip_molded; LCSC (none) -> C76970
- L1: KiLib_Generator (none) -> SMD_2terminal_chip_molded
Changed lines of the file:
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@@
+			)
+		)
+		(property "LCSC" "C16194197"
+			(at 168.91 71.12 0)
+			(hide yes)
+			(show_name no)
+			(do_not_autoplace no)
+			(effects
+				(font
+					(size 1.27 1.27)
+				)
 			)
 		)
@@
 			)
 		)
+		(property "KiLib_Generator" "SMD_2terminal_chip_molded"
+			(at 72.39 45.72 0)
+			(hide yes)
+			(show_name no)
+			(do_not_autoplace no)
+			(effects
+				(font
+					(size 1.27 1.27)
+				)
+			)
+		)
 		(pin "1"
 		)
@@
 			(at 91.44 49.53 0)
 			(hide yes)
+			(show_name no)
+			(do_not_autoplace no)
+			(effects
+				(font
+					(size 1.27 1.27)
+				)
+			)
+		)
+		(property "LCSC" "C76970"
+			(at 91.44 49.53 90)
+			(hide yes)
+			(show_name no)
+			(do_not_autoplace no)
+			(effects
+				(font
+					(size 1.27 1.27)
+				)
+			)
+		)
+		(property "KiLib_Generator" "SMD_2terminal_chip_molded"
+			(at 91.44 49.53 0)
+			(hide yes)

Commit message: Revert "update"
This reverts commit ded726db31db978a67aba241c9369c22f126eee0.
Parts:
- C2: LCSC C16194197 -> (none)
- C3: KiLib_Generator SMD_2terminal_chip_molded -> (none); LCSC C76970 -> (none)
- L1: KiLib_Generator SMD_2terminal_chip_molded -> (none)
Changed lines of the file:
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@@
-			)
-		)
-		(property "LCSC" "C16194197"
-			(at 168.91 71.12 0)
-			(hide yes)
-			(show_name no)
-			(do_not_autoplace no)
-			(effects
-				(font
-					(size 1.27 1.27)
-				)
 			)
 		)
@@
 			)
 		)
-		(property "KiLib_Generator" "SMD_2terminal_chip_molded"
-			(at 72.39 45.72 0)
-			(hide yes)
-			(show_name no)
-			(do_not_autoplace no)
-			(effects
-				(font
-					(size 1.27 1.27)
-				)
-			)
-		)
 		(pin "1"
 		)
@@
 			(at 91.44 49.53 0)
 			(hide yes)
-			(show_name no)
-			(do_not_autoplace no)
-			(effects
-				(font
-					(size 1.27 1.27)
-				)
-			)
-		)
-		(property "LCSC" "C76970"
-			(at 91.44 49.53 90)
-			(hide yes)
-			(show_name no)
-			(do_not_autoplace no)
-			(effects
-				(font
-					(size 1.27 1.27)
-				)
-			)
-		)
-		(property "KiLib_Generator" "SMD_2terminal_chip_molded"
-			(at 91.44 49.53 0)
-			(hide yes)
