File: interface_db_hat/interface_db_hat.kicad_pcb (KiCad board)
At the start: 2 copper layers, 65 x 56 mm, 5 parts, among them J1 GPIO

Commit message: UPDATE
Parts:
- added BZ1: Buzzer, Buzzer_Beeper:Buzzer_12x9.5RM7.6, F.Cu at (173.9, 74.5)
- added C1: 100nF, Capacitor_SMD:C_0603_1608Metric_Pad1.08x0.95mm_HandSolder, F.Cu at (244.1, 65.3)
- added C2: 100nF, Capacitor_SMD:C_0603_1608Metric_Pad1.08x0.95mm_HandSolder, F.Cu at (223.2, 106.6)
- added C3: 40pF, Capacitor_SMD:C_0603_1608Metric_Pad1.08x0.95mm_HandSolder, B.Cu at (149.5, 91.0)
- added C30: 100nF, Capacitor_SMD:C_0603_1608Metric_Pad1.08x0.95mm_HandSolder, F.Cu at (244.1, 67.8)
- added C4: 100nF, Capacitor_SMD:C_0603_1608Metric_Pad1.08x0.95mm_HandSolder, F.Cu at (207.8, 65.3)
- added C5: 100nF, Capacitor_SMD:C_0603_1608Metric_Pad1.08x0.95mm_HandSolder, F.Cu at (207.8, 67.8)
- added D1: 5V, Diode_SMD:D_0603_1608Metric_Pad1.05x0.95mm_HandSolder, F.Cu at (122.6, 54.2)
- added D10: TVS_3V3, Diode_SMD:D_0402_1005Metric_Pad0.77x0.64mm_HandSolder, F.Cu at (122.6, 56.8)
- added D11: TVS_13V, Diode_SMD:D_0603_1608Metric_Pad1.05x0.95mm_HandSolder, F.Cu at (122.6, 59.4)
- added D14: TVS_3V3, Diode_SMD:D_0402_1005Metric_Pad0.77x0.64mm_HandSolder, F.Cu at (105.0, 64.0)
- added D15: TVS_3V3, Diode_SMD:D_0402_1005Metric_Pad0.77x0.64mm_HandSolder, F.Cu at (122.6, 64.6)
- added D16: TVS_3V3, Diode_SMD:D_0402_1005Metric_Pad0.77x0.64mm_HandSolder, F.Cu at (122.6, 67.2)
- added D17: TVS_3V3, Diode_SMD:D_0402_1005Metric_Pad0.77x0.64mm_HandSolder, F.Cu at (107.1, 65.0)
- added D18: TVS_3V3, Diode_SMD:D_0402_1005Metric_Pad0.77x0.64mm_HandSolder, F.Cu at (105.0, 66.0)
- added D19: TVS_3V3, Diode_SMD:D_0402_1005Metric_Pad0.77x0.64mm_HandSolder, F.Cu at (107.1, 67.0)
- added D2: LED_R, LED_SMD:LED_0603_1608Metric_Pad1.05x0.95mm_HandSolder, F.Cu at (253.4, 113.8)
- added D20: TVS_3V3, Diode_SMD:D_0402_1005Metric_Pad0.77x0.64mm_HandSolder, F.Cu at (105.0, 68.0)
- added D21: TVS_3V3, Diode_SMD:D_0402_1005Metric_Pad0.77x0.64mm_HandSolder, F.Cu at (107.1, 69.0)
- added D22: TVS_3V3, Diode_SMD:D_0402_1005Metric_Pad0.77x0.64mm_HandSolder, F.Cu at (105.0, 70.0)
- added D23: TVS_3V3, Diode_SMD:D_0402_1005Metric_Pad0.77x0.64mm_HandSolder, F.Cu at (107.0, 71.0)
- added D24: TVS_3V3, Diode_SMD:D_0402_1005Metric_Pad0.77x0.64mm_HandSolder, F.Cu at (127.0, 64.6)
- added D25: TVS_3V3, Diode_SMD:D_0402_1005Metric_Pad0.77x0.64mm_HandSolder, F.Cu at (127.0, 67.2)
- added D26: TVS_3V3, Diode_SMD:D_0402_1005Metric_Pad0.77x0.64mm_HandSolder, F.Cu at (127.0, 69.8)
- added D27: TVS_3V3, Diode_SMD:D_0402_1005Metric_Pad0.77x0.64mm_HandSolder, F.Cu at (127.0, 72.4)
- added D28: TVS_3V3, Diode_SMD:D_0402_1005Metric_Pad0.77x0.64mm_HandSolder, F.Cu at (127.0, 75.0)
- added D29: TVS_3V3, Diode_SMD:D_0402_1005Metric_Pad0.77x0.64mm_HandSolder, F.Cu at (131.4, 54.2)
- added D3: LED_R, LED_SMD:LED_0603_1608Metric_Pad1.05x0.95mm_HandSolder, F.Cu at (253.4, 116.4)
- added D30: TVS_3V3, Diode_SMD:D_0402_1005Metric_Pad0.77x0.64mm_HandSolder, F.Cu at (131.4, 56.8)
- added D31: TVS_3V3, Diode_SMD:D_0402_1005Metric_Pad0.77x0.64mm_HandSolder, F.Cu at (131.4, 59.4)
- added D32: TVS_3V3, Diode_SMD:D_0402_1005Metric_Pad0.77x0.64mm_HandSolder, F.Cu at (131.4, 62.0)
- added D33: TVS_3V3, Diode_SMD:D_0402_1005Metric_Pad0.77x0.64mm_HandSolder, F.Cu at (131.4, 64.6)
- added D34: TVS_3V3, Diode_SMD:D_0402_1005Metric_Pad0.77x0.64mm_HandSolder, F.Cu at (131.4, 67.2)
- added D35: TVS_3V3, Diode_SMD:D_0402_1005Metric_Pad0.77x0.64mm_HandSolder, F.Cu at (131.4, 69.8)
- added D36: TVS_3V3, Diode_SMD:D_0402_1005Metric_Pad0.77x0.64mm_HandSolder, F.Cu at (129.9, 91.0)
- added D37: TVS_3V3, Diode_SMD:D_0402_1005Metric_Pad0.77x0.64mm_HandSolder, F.Cu at (131.0, 88.5)
- added D38: TVS_3V3, Diode_SMD:D_0402_1005Metric_Pad0.77x0.64mm_HandSolder, F.Cu at (135.0, 91.0)
- added D39: TVS_3V3, Diode_SMD:D_0402_1005Metric_Pad0.77x0.64mm_HandSolder, F.Cu at (131.4, 72.4)
- added D4: LED_R, LED_SMD:LED_0603_1608Metric_Pad1.05x0.95mm_HandSolder, F.Cu at (253.4, 119.0)
- added D40: TVS_13V, Diode_SMD:D_0603_1608Metric_Pad1.05x0.95mm_HandSolder, F.Cu at (131.4, 75.0)
- added D41: TVS_3V3, Diode_SMD:D_0402_1005Metric_Pad0.77x0.64mm_HandSolder, F.Cu at (135.8, 54.2)
- added D42: TVS_3V3, Diode_SMD:D_0402_1005Metric_Pad0.77x0.64mm_HandSolder, F.Cu at (135.8, 56.8)
- added D43: TVS_3V3, Diode_SMD:D_0402_1005Metric_Pad0.77x0.64mm_HandSolder, F.Cu at (135.8, 59.4)
- added D44: TVS_3V3, Diode_SMD:D_0402_1005Metric_Pad0.77x0.64mm_HandSolder, F.Cu at (135.8, 62.0)
- added D45: TVS_3V3, Diode_SMD:D_0402_1005Metric_Pad0.77x0.64mm_HandSolder, F.Cu at (135.8, 64.6)
- added D46: TVS_3V3, Diode_SMD:D_0402_1005Metric_Pad0.77x0.64mm_HandSolder, F.Cu at (135.8, 67.2)
- added D47: TVS_3V3, Diode_SMD:D_0402_1005Metric_Pad0.77x0.64mm_HandSolder, F.Cu at (105.5, 58.1)
- added D48: TVS_3V3, Diode_SMD:D_0402_1005Metric_Pad0.77x0.64mm_HandSolder, F.Cu at (105.5, 53.6)
- added D6: LED_R, LED_SMD:LED_0603_1608Metric_Pad1.05x0.95mm_HandSolder, F.Cu at (253.4, 121.5)
- added J2: Conn_02x06_Counter_Clockwise, Connector_PinSocket_2.54mm:PinSocket_2x06_P2.54mm_Vertical, F.Cu at (123.0, 97.0)
- added J3: Conn_02x06_Counter_Clockwise, Connector_PinSocket_2.54mm:PinSocket_2x06_P2.54mm_Vertical, F.Cu at (144.5, 55.8)
- added J4: Conn_Coaxial_Small, Connector_Coaxial:SMA_Amphenol_132289_EdgeMount, B.Cu at (149.5, 96.1)
- added J5: Conn_01x04_Pin, Connector_JST:JST_SH_SM04B-SRSS-TB_1x04-1MP_P1.00mm_Horizontal, F.Cu at (131.5, 96.5)
- added J6: Conn_01x04_Pin, Connector_JST:JST_SH_SM04B-SRSS-TB_1x04-1MP_P1.00mm_Horizontal, F.Cu at (104.0, 88.5)
- added J7: Conn_01x20_Pin, Connector_PinHeader_1.00mm:PinHeader_1x20_P1.00mm_Vertical, F.Cu at (102.0, 64.0)
- added J8: Conn_01x03_Pin, Connector_PinHeader_2.54mm:PinHeader_1x03_P2.54mm_Horizontal, F.Cu at (102.0, 59.6)
- added JP1: SolderJumper_2_Open, Jumper:SolderJumper-2_P1.3mm_Open_TrianglePad1.0x1.5mm, B.Cu at (142.5, 91.3)
- added JP6: SolderJumper_2_Open, Jumper:SolderJumper-2_P1.3mm_Open_TrianglePad1.0x1.5mm, F.Cu at (215.3, 111.3)
- added L1: 101nH, Inductor_SMD:L_0603_1608Metric_Pad1.05x0.95mm_HandSolder, B.Cu at (146.4, 92.0)
- added Q1: BC817, Package_TO_SOT_SMD:SOT-23_Handsoldering, F.Cu at (256.1, 96.2)
- added R1: 10k, Resistor_SMD:R_0603_1608Metric_Pad0.98x0.95mm_HandSolder, F.Cu at (244.1, 70.3)
- added R10: 330, Resistor_SMD:R_0603_1608Metric_Pad0.98x0.95mm_HandSolder, F.Cu at (257.7, 113.7)
- added R11: 1k, Resistor_SMD:R_0603_1608Metric_Pad0.98x0.95mm_HandSolder, F.Cu at (257.7, 116.2)
- added R12: 4.7k, Resistor_SMD:R_0603_1608Metric_Pad0.98x0.95mm_HandSolder, F.Cu at (257.7, 118.8)
- added R13: 330, Resistor_SMD:R_0603_1608Metric_Pad0.98x0.95mm_HandSolder, F.Cu at (244.1, 72.8)
- added R14: 330, Resistor_SMD:R_0603_1608Metric_Pad0.98x0.95mm_HandSolder, F.Cu at (257.7, 121.3)
- added R15: 330, Resistor_SMD:R_0603_1608Metric_Pad0.98x0.95mm_HandSolder, F.Cu at (244.1, 75.3)
- added R2: 10k, Resistor_SMD:R_0603_1608Metric_Pad0.98x0.95mm_HandSolder, F.Cu at (223.2, 114.1)
- added R3: 4.7k, Resistor_SMD:R_0603_1608Metric_Pad0.98x0.95mm_HandSolder, F.Cu at (223.2, 116.6)
- added R35: 4.7k, Resistor_SMD:R_0603_1608Metric_Pad0.98x0.95mm_HandSolder, F.Cu at (207.8, 77.8)
- added R36: 4.7k, Resistor_SMD:R_0603_1608Metric_Pad0.98x0.95mm_HandSolder, F.Cu at (212.2, 65.3)
- added R38: 10k, Resistor_SMD:R_0603_1608Metric_Pad0.98x0.95mm_HandSolder, F.Cu at (212.2, 67.8)
- added R4: 10k, Resistor_SMD:R_0603_1608Metric_Pad0.98x0.95mm_HandSolder, F.Cu at (223.2, 119.1)
- added R42: 33, Resistor_SMD:R_0603_1608Metric_Pad0.98x0.95mm_HandSolder, F.Cu at (244.1, 77.8)
- added R43: 33, Resistor_SMD:R_0603_1608Metric_Pad0.98x0.95mm_HandSolder, F.Cu at (244.1, 80.3)
- added R44: 33, Resistor_SMD:R_0603_1608Metric_Pad0.98x0.95mm_HandSolder, F.Cu at (248.4, 65.3)
- added R45: 33, Resistor_SMD:R_0603_1608Metric_Pad0.98x0.95mm_HandSolder, F.Cu at (248.4, 67.8)
- added R46: 33, Resistor_SMD:R_0603_1608Metric_Pad0.98x0.95mm_HandSolder, F.Cu at (248.4, 70.3)
- added R47: 33, Resistor_SMD:R_0603_1608Metric_Pad0.98x0.95mm_HandSolder, F.Cu at (248.4, 72.8)
- added R48: 33, Resistor_SMD:R_0603_1608Metric_Pad0.98x0.95mm_HandSolder, F.Cu at (248.4, 75.3)
- added R49: 33, Resistor_SMD:R_0603_1608Metric_Pad0.98x0.95mm_HandSolder, F.Cu at (248.4, 77.8)
- added R50: 33, Resistor_SMD:R_0603_1608Metric_Pad0.98x0.95mm_HandSolder, F.Cu at (248.4, 80.3)
- added R51: 33, Resistor_SMD:R_0603_1608Metric_Pad0.98x0.95mm_HandSolder, F.Cu at (252.8, 65.3)
- added R52: 33, Resistor_SMD:R_0603_1608Metric_Pad0.98x0.95mm_HandSolder, F.Cu at (252.8, 67.8)
- added R53: 33, Resistor_SMD:R_0603_1608Metric_Pad0.98x0.95mm_HandSolder, F.Cu at (252.8, 70.3)
- added R54: 33, Resistor_SMD:R_0603_1608Metric_Pad0.98x0.95mm_HandSolder, F.Cu at (252.8, 72.8)
- added R55: 33, Resistor_SMD:R_0603_1608Metric_Pad0.98x0.95mm_HandSolder, F.Cu at (252.8, 75.3)
- added R56: 33, Resistor_SMD:R_0603_1608Metric_Pad0.98x0.95mm_HandSolder, F.Cu at (252.8, 77.8)
- added R57: 33, Resistor_SMD:R_0603_1608Metric_Pad0.98x0.95mm_HandSolder, F.Cu at (252.8, 80.3)
- added R58: 33, Resistor_SMD:R_0603_1608Metric_Pad0.98x0.95mm_HandSolder, F.Cu at (257.1, 65.3)
- added R59: 33, Resistor_SMD:R_0603_1608Metric_Pad0.98x0.95mm_HandSolder, F.Cu at (257.1, 67.8)
- added R6: 10k, Resistor_SMD:R_0603_1608Metric_Pad0.98x0.95mm_HandSolder, F.Cu at (207.8, 70.3)
- added R60: 33, Resistor_SMD:R_0603_1608Metric_Pad0.98x0.95mm_HandSolder, F.Cu at (257.1, 70.3)
- added R61: 33, Resistor_SMD:R_0603_1608Metric_Pad0.98x0.95mm_HandSolder, F.Cu at (257.1, 72.8)
- added R63: 33, Resistor_SMD:R_0603_1608Metric_Pad0.98x0.95mm_HandSolder, F.Cu at (132.0, 85.0)
- added R64: 33, Resistor_SMD:R_0603_1608Metric_Pad0.98x0.95mm_HandSolder, F.Cu at (134.0, 87.5)
- added R65: 33, Resistor_SMD:R_0603_1608Metric_Pad0.98x0.95mm_HandSolder, F.Cu at (108.9, 54.6)
- added R66: 33, Resistor_SMD:R_0603_1608Metric_Pad0.98x0.95mm_HandSolder, F.Cu at (108.9, 57.1)
- added R7: 10k, Resistor_SMD:R_0603_1608Metric_Pad0.98x0.95mm_HandSolder, F.Cu at (207.8, 72.8)
- added R8: 10k, Resistor_SMD:R_0603_1608Metric_Pad0.98x0.95mm_HandSolder, F.Cu at (207.8, 75.3)
- added TP1: TestPoint_2Pole, Connector_PinHeader_2.54mm:PinHeader_1x02_P2.54mm_Vertical, F.Cu at (248.9, 107.6)
- added TP2: TestPoint_2Pole, Connector_PinHeader_2.54mm:PinHeader_1x02_P2.54mm_Vertical, F.Cu at (253.5, 107.6)
- added TP3: TestPoint, TestPoint:TestPoint_Pad_D2.5mm, F.Cu at (248.9, 114.8)
- added TP4: TestPoint, TestPoint:TestPoint_Pad_D2.5mm, F.Cu at (248.9, 119.3)
- added U1: MAX-M10M-00B, MAX-M10M:XCVR_MAX-M10M-00B, B.Cu at (146.2, 81.8)
- added U2: TCA9617ADGKR, TCA9617:DGK0008A, F.Cu at (134.5, 80.0)
- added U6: MCP23008-xSO, Package_SO:SOIC-18W_7.5x11.6mm_P1.27mm, F.Cu at (162.8, 65.5)
Connections:
- J1 pad 10: /GPIO15/RXD0 -> /HAT_connections/GPIO15/RXD0
- J1 pad 11: /GPIO17 -> /IVC_SW_1
- J1 pad 12: /GPIO18/PCM.CLK -> /GPS_PPS
- J1 pad 13: /GPIO27 -> /IVC_SW_1_SOL
- J1 pad 15: /GPIO22 -> /IVC_SW_1_SOL
- J1 pad 16: /GPIO23 -> /SPI_CS3
- J1 pad 18: /GPIO24 -> /SPI_CS4
- J1 pad 19: /GPIO10/SPI0.MOSI -> /SPI_MOSI
- J1 pad 21: /GPIO9/SPI0.MISO -> /SPI_MISO
- J1 pad 22: /GPIO25 -> /SERVO_1
- J1 pad 23: /GPIO11/SPI0.SCLK -> /SPI_SCLK
- J1 pad 24: /GPIO8/SPI0.CE0 -> /SPI_CS1
- J1 pad 26: /GPIO7/SPI0.CE1 -> /SPI_CS2
- J1 pad 27: /ID_SDA -> /INT_SLCTB
- J1 pad 28: /ID_SCL -> /SERVO_2
- J1 pad 29: /GPIO5 -> /INT_HLD
- J1 pad 3: /GPIO2/SDA1 -> /I2C_SDA
- J1 pad 31: /GPIO6 -> /INT_RST
- J1 pad 32: /GPIO12/PWM0 -> /BUZZER
- J1 pad 33: /GPIO13/PWM1 -> /LED_1
- J1 pad 35: /GPIO19/PCM.FS -> /INT_SLCTA
- J1 pad 36: /GPIO16 -> /SERVO_3
- J1 pad 37: /GPIO26 -> /LED_2
- J1 pad 38: /GPIO20/PCM.DIN -> /IND_2
- J1 pad 40: /GPIO21/PCM.DOUT -> /HAT_connections/EXP_INT
- J1 pad 5: /GPIO3/SCL1 -> /I2C_SCL
- J1 pad 7: /GPIO4/GPCLK0 -> /IVC_SW_2
- J1 pad 8: /GPIO14/TXD0 -> /HAT_connections/GPIO14/TXD0
Other:
- outline, holes or cut-outs redrawn
- board text removed: "CAMERA (OPTIONAL)"
- board text removed: "DISPLAY (OPTIONAL)"
