File: interface_db_hat/interface_db_hat.kicad_pcb (KiCad board)
At the start: 2 copper layers, 65 x 56 mm, 112 parts, among them J1 GPIO, J2 Conn_02x06_Counter_Clockwise, J3 Conn_02x06_Counter_Clockwise, J4 Conn_Coaxial_Small, J5 Conn_01x04_Pin, J6 Conn_01x04_Pin, J7 Conn_01x20_Pin, J8 Conn_01x03_Pin, Q1 BC817, U1 MAX-M10M-00B, U2 TCA9617ADGKR, U6 MCP23008-xSO

Commit message: lol
Parts:
- removed D1: 5V, Diode_SMD:D_0603_1608Metric_Pad1.05x0.95mm_HandSolder
- removed D14, D15, D16, D17, D18, D19, D20, D21, D22, D23, D24, D25, D26, D27, D28, D29, D30, D31, D32, D33, D34, D35, D39, D41, D42, D43, D44, D45, D46: TVS_3V3, Diode_SMD:D_0402_1005Metric_Pad0.77x0.64mm_HandSolder
- removed D40: TVS_13V, Diode_SMD:D_0603_1608Metric_Pad1.05x0.95mm_HandSolder
- removed J2: Conn_02x06_Counter_Clockwise, Connector_PinSocket_2.54mm:PinSocket_2x06_P2.54mm_Vertical
- removed JP6: SolderJumper_2_Open, Jumper:SolderJumper-2_P1.3mm_Open_TrianglePad1.0x1.5mm
- removed R13: 330, Resistor_SMD:R_0603_1608Metric_Pad0.98x0.95mm_HandSolder
- removed R38, R6: 10k, Resistor_SMD:R_0603_1608Metric_Pad0.98x0.95mm_HandSolder
- removed U6: MCP23008-xSO, Package_SO:SOIC-18W_7.5x11.6mm_P1.27mm
- added C31: 22uF, Capacitor_SMD:C_0603_1608Metric_Pad1.08x0.95mm_HandSolder, F.Cu at (131.0, 58.5)
- added C32: 100nF, Capacitor_SMD:C_0603_1608Metric_Pad1.08x0.95mm_HandSolder, F.Cu at (133.5, 58.5)
- added C33: 100nF, Capacitor_SMD:C_0603_1608Metric_Pad1.08x0.95mm_HandSolder, F.Cu at (136.0, 58.5)
- added C34: 22uF, Capacitor_SMD:C_0603_1608Metric_Pad1.08x0.95mm_HandSolder, F.Cu at (138.5, 58.5)
- added C35: 100nF, Capacitor_SMD:C_0603_1608Metric_Pad1.08x0.95mm_HandSolder, F.Cu at (141.0, 58.5)
- added C36: 22uF, Capacitor_SMD:C_0603_1608Metric_Pad1.08x0.95mm_HandSolder, F.Cu at (143.6, 58.5)
- added C6: 100nF, Capacitor_SMD:C_0603_1608Metric_Pad1.08x0.95mm_HandSolder, F.Cu at (139.1, 53.0)
- added D7: LED_R, LED_SMD:LED_0603_1608Metric_Pad1.05x0.95mm_HandSolder, F.Cu at (132.0, 53.0)
- added J10: Conn_02x06_Counter_Clockwise, Connector_PinSocket_2.54mm:PinSocket_2x06_P2.54mm_Vertical, F.Cu at (102.5, 87.0)
- added J9: Conn_02x06_Counter_Clockwise, Connector_PinSocket_2.54mm:PinSocket_2x06_P2.54mm_Vertical, F.Cu at (149.8, 53.5)
- added JP7: SolderJumper_2_Open, Jumper:SolderJumper-2_P1.3mm_Open_TrianglePad1.0x1.5mm, F.Cu at (162.5, 66.5)
- added R16: 330, Resistor_SMD:R_0603_1608Metric_Pad0.98x0.95mm_HandSolder, F.Cu at (134.6, 53.0)
- added R17: 330, Resistor_SMD:R_0603_1608Metric_Pad0.98x0.95mm_HandSolder, F.Cu at (173.3, 82.1)
- added R39: 10k, Resistor_SMD:R_0603_1608Metric_Pad0.98x0.95mm_HandSolder, F.Cu at (162.5, 63.5)
- added R9: 10k, Resistor_SMD:R_0603_1608Metric_Pad0.98x0.95mm_HandSolder, F.Cu at (162.5, 61.0)
- added U7: MCP23017x-x-SO, Package_SO:SOIC-28W_7.5x17.9mm_P1.27mm, F.Cu at (150.5, 66.5)
- BZ1: footprint Buzzer_Beeper:Buzzer_12x9.5RM7.6 -> Buzzer_Beeper:Buzzer_CUI_CPT-9019S-SMT
- C2, D47, D48, R2, R3, R4, R65, R66: moved to B.Cu
- C3, J4, JP1, L1, U1: moved to F.Cu
- moved C1 142.5 mm to (102.5, 81.0), turned to 90 degrees
- moved TP3 140.6 mm to (112.5, 80.5), turned to 90 degrees
- moved C30 139.7 mm to (105.0, 81.0), turned to 90 degrees
- moved R61 138.8 mm to (120.0, 94.3), turned to -90 degrees
- moved R59 137.7 mm to (122.0, 94.4), turned to -90 degrees
- moved R60 137.6 mm to (121.0, 90.4), turned to -90 degrees
- moved TP2 137.6 mm to (116.0, 113.0), turned to 90 degrees
- moved TP4 137.4 mm to (117.0, 80.5), turned to 90 degrees
- moved R1 137.0 mm to (107.5, 81.0), turned to 90 degrees
- moved R58 136.5 mm to (123.0, 90.4), turned to -90 degrees
- moved TP1 133.3 mm to (116.0, 117.6), turned to 90 degrees
- moved R57 129.5 mm to (124.0, 94.4), turned to -90 degrees
- moved D2 129.5 mm to (133.9, 63.9)
- moved D3 129.5 mm to (133.9, 66.5)
- moved D4 129.5 mm to (133.9, 69.1)
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Connections:
- D6 pad 2: /IND -> /IND_0
- J1 pad 11: /IVC_SW_1 -> /STRT2
- J1 pad 29: /INT_HLD -> /INT_SLCTA
- J1 pad 31: /INT_RST -> /LED_PWM_1
- J1 pad 33: /LED_1 -> /LED_PWM_2
- J1 pad 35: /INT_SLCTA -> /~{DRDY1}
- J1 pad 36: /SERVO_3 -> /HAT_connections/GPIO16
- J1 pad 37: /LED_2 -> /~{DRDY2}
- J1 pad 38: /IND_2 -> /HAT_connections/EXP_INT_A
- J1 pad 40: /HAT_connections/EXP_INT -> /HAT_connections/EXP_INT_B
- J1 pad 7: /IVC_SW_2 -> /STRT1
- J3 pad 1: /I2C_SCL -> /I2C_SDA
- J3 pad 10: GND -> /IND_4
- J3 pad 11: /LED_2 -> /LED_PWM_1
- J3 pad 12: /LED_1 -> GND
- J3 pad 2: /I2C_SDA -> GND
- J3 pad 4: /SERVO_1 -> GND
- J3 pad 5: /SERVO_2 -> /I2C_SCL
- J3 pad 6: /SERVO_3 -> /IND_2
- J3 pad 8: GND -> /IND_3
- J3 pad 9: /IND_2 -> /LED_PWM_2
- R15 pad 1: +5V -> /BUZZER
- R15 pad 2: Net-(BZ1--) -> Net-(Q1-B)
- R45 pad 1: /IVC_SW_1_SOL -> /IVC_SW_2_SOL
Other:
- board text added: "EXT I2C"
- board text added: "GPS ANT"
- board text added: "PD I/O"
- board text added: "PD POWER"
- board text added: "PI UART"
- board text removed: "PoE"

Commit message: update
Connections:
- D6 pad 2: /IND_0 -> /IND_1
- D7 pad 2: /IND_1 -> /IND_2
- J3 pad 10: /IND_4 -> GND
- J3 pad 2: GND -> /MOTOR_1_A
- J3 pad 4: GND -> /MOTOR_1_B
- J3 pad 6: /IND_2 -> /MOTOR_2_A
- J3 pad 8: /IND_3 -> /MOTOR_2_B
- U7 pad 1: /IND_1 -> /MOTOR_1
- U7 pad 2: /IND_2 -> /MOTOR_2
- U7 pad 21: /IND_5 -> /IND_1
- U7 pad 22: /IND_6 -> /IND_2
- U7 pad 27: /IND_0 -> /IND_3
- U7 pad 3: /IND_3 -> /MOTOR_3
- U7 pad 4: /IND_4 -> /MOTOR_4
Changed lines of the file:
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@@
 			(layers "F.Cu" "F.Mask" "F.Paste")
 			(roundrect_rratio 0.25)
-			(net "/IND_1")
+			(net "/MOTOR_1")
 			(pinfunction "GPB0_1")
 			(pintype "bidirectional")
@@
 			(layers "F.Cu" "F.Mask" "F.Paste")
 			(roundrect_rratio 0.25)
-			(net "/IND_2")
+			(net "/MOTOR_2")
 			(pinfunction "GPB1_2")
 			(pintype "bidirectional")
@@
 			(layers "F.Cu" "F.Mask" "F.Paste")
 			(roundrect_rratio 0.25)
-			(net "/IND_3")
+			(net "/MOTOR_3")
 			(pinfunction "GPB2_3")
 			(pintype "bidirectional")
@@
 			(layers "F.Cu" "F.Mask" "F.Paste")
 			(roundrect_rratio 0.25)
-			(net "/IND_4")
+			(net "/MOTOR_4")
 			(pinfunction "GPB3_4")
 			(pintype "bidirectional")
@@
 			(layers "F.Cu" "F.Mask" "F.Paste")
 			(roundrect_rratio 0.25)
-			(net "/IND_5")
+			(net "/IND_1")
 			(pinfunction "GPA0_21")
 			(pintype "bidirectional")
@@
 			(layers "F.Cu" "F.Mask" "F.Paste")
 			(roundrect_rratio 0.25)
-			(net "/IND_6")
+			(net "/IND_2")
 			(pinfunction "GPA1_22")
 			(pintype "bidirectional")
@@
 			(layers "F.Cu" "F.Mask" "F.Paste")
 			(roundrect_rratio 0.25)
-			(net "/IND_0")
+			(net "/IND_3")
 			(pinfunction "GPA6_27")
 			(pintype "bidirectional")
@@
 			(layers "*.Cu" "*.Mask")
 			(remove_unused_layers no)
-			(net "GND")
+			(net "/MOTOR_1_A")
 			(pinfunction "Pin_2_2")
 			(pintype "passive")
@@
 			(layers "*.Cu" "*.Mask")
 			(remove_unused_layers no)
-			(net "GND")
+			(net "/MOTOR_1_B")
 			(pinfunction "Pin_4_4")
 			(pintype "passive")
@@
 			(layers "*.Cu" "*.Mask")
 			(remove_unused_layers no)
-			(net "/IND_2")
+			(net "/MOTOR_2_A")
 			(pinfunction "Pin_6_6")
 			(pintype "passive")
@@
 			(layers "*.Cu" "*.Mask")
 			(remove_unused_layers no)
-			(net "/IND_3")
+			(net "/MOTOR_2_B")
 			(pinfunction "Pin_8_8")
 			(pintype "passive")
@@
 			(layers "*.Cu" "*.Mask")
 			(remove_unused_layers no)
-			(net "/IND_4")
+			(net "GND")
 			(pinfunction "Pin_10_10")
 			(pintype "passive")
@@
 			(layers "F.Cu" "F.Mask" "F.Paste")
 			(roundrect_rratio 0.25)
-			(net "/IND_1")
+			(net "/IND_2")
 			(pinfunction "A_2")
 			(pintype "passive")
@@
 			(layers "F.Cu" "F.Mask" "F.Paste")
 			(roundrect_rratio 0.25)
-			(net "/IND_0")
+			(net "/IND_1")
 			(pinfunction "A_2")
 			(pintype "passive")

Commit message: working on interface board
Parts:
- removed C35: 100nF, Capacitor_SMD:C_0603_1608Metric_Pad1.08x0.95mm_HandSolder
- removed C36: 22uF, Capacitor_SMD:C_0603_1608Metric_Pad1.08x0.95mm_HandSolder
- removed J7: Conn_01x20_Pin, Connector_PinHeader_1.00mm:PinHeader_1x20_P1.00mm_Vertical
- added C45: 100nF, Capacitor_SMD:C_0603_1608Metric_Pad1.08x0.95mm_HandSolder, F.Cu at (90.2, 83.3)
- added C46: 22uF, Capacitor_SMD:C_0603_1608Metric_Pad1.08x0.95mm_HandSolder, F.Cu at (90.2, 85.8)
- added J2: DF19G-20P-1H52, DF-19:CONN20_DF19G_HIR, F.Cu at (129.5, 96.5)
- moved JP1 15.5 mm to (158.0, 90.8)
- moved BZ1 11.2 mm to (124.5, 69.5)
- moved L1 8.38 mm to (154.4, 91.5), turned to 0 degrees
- moved U2 7.63 mm to (115.5, 66.0)
- moved U1 6.00 mm to (154.5, 81.6)
- moved R61 4.66 mm to (120.0, 89.7)
- moved R42 4.66 mm to (139.0, 85.8)
- moved R43 4.66 mm to (138.0, 89.8)
- moved R44 4.66 mm to (137.0, 85.8)
- moved R45 4.66 mm to (136.0, 89.8)
- moved R46 4.66 mm to (135.0, 85.8)
- moved R47 4.66 mm to (134.0, 89.8)
- moved R48 4.66 mm to (133.0, 85.8)
- moved R49 4.66 mm to (132.0, 89.8)
- moved R50 4.66 mm to (131.0, 85.8)
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Connections:
- J10 pad 1: +3V3 -> GND
- J10 pad 11: +5V -> +12V
- J10 pad 2: +12V -> GND
- J10 pad 3: +3V3 -> GND
- J10 pad 4: +12V -> GND
- J10 pad 5: +5V -> +12V
- J10 pad 6: +12V -> GND
- J10 pad 7: +5V -> +12V
- J10 pad 8: +12V -> GND
- J10 pad 9: +5V -> +12V
- J3 pad 1: /I2C_SDA -> +5V
- J3 pad 11: /LED_PWM_1 -> /I2C_SCL
- J3 pad 12: GND -> /I2C_SDA
- J3 pad 2: /MOTOR_1_A -> +5V
- J3 pad 3: GND -> +5V
- J3 pad 4: /MOTOR_1_B -> +5V
- J3 pad 5: /I2C_SCL -> +5V
- J3 pad 6: /MOTOR_2_A -> +5V
- J3 pad 7: GND -> +5V
- J3 pad 8: /MOTOR_2_B -> +5V
- J3 pad 9: /LED_PWM_2 -> GND
- J9 pad 1: /SERVO_1 -> /SERVO_2
- J9 pad 10: GND -> /LED_PWM_1
- J9 pad 11: GND -> /IND_3
- J9 pad 12: GND -> /LED_PWM_2
- J9 pad 2: GND -> /MOTOR_1_B
- J9 pad 3: /SERVO_2 -> /SERVO_1
- J9 pad 4: GND -> /MOTOR_1_A
- J9 pad 5: /SERVO_3 -> +3V3
- J9 pad 6: GND -> /MOTOR_2_B
- J9 pad 7: /SERVO_4 -> +3V3
- J9 pad 8: GND -> /MOTOR_2_A
- U7 pad 1: /MOTOR_1 -> /MOTOR_1_B
- U7 pad 2: /MOTOR_2 -> /MOTOR_1_A
- U7 pad 3: /MOTOR_3 -> /MOTOR_2_B
- U7 pad 4: /MOTOR_4 -> /MOTOR_2_A
Routing:
- net +12V: track 0.00 -> 21.8 mm
- net /I2C_SDA: track 0.00 -> 8.97 mm
- net Net-(J2-Pad2): track 0.00 -> 6.65 mm
- net Net-(J2-Pad18): track 0.00 -> 6.65 mm
- net Net-(J2-Pad4): track 0.00 -> 6.65 mm
- net Net-(J2-Pad16): track 0.00 -> 6.65 mm
- net Net-(J2-Pad6): track 0.00 -> 6.65 mm
- net Net-(J2-Pad14): track 0.00 -> 6.65 mm
- net Net-(J2-Pad8): track 0.00 -> 6.65 mm
- net Net-(J2-Pad12): track 0.00 -> 6.65 mm
- net Net-(J2-Pad10): track 0.00 -> 6.65 mm
- net Net-(J2-Pad20): track 0.00 -> 6.57 mm
- net /I2C_SCL: track 0.00 -> 5.38 mm
- net Net-(J2-Pad1): track 0.00 -> 2.74 mm
- net Net-(J2-Pad3): track 0.00 -> 2.65 mm
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- added copper zone on B.Cu, net (none)
- added copper zone on F.Cu, net (none)
- added copper zone on In1.Cu, net (none)
- added copper zone on In1.Cu, net +3V3
- added copper zone on In2.Cu, net GND
Other:
- copper layers 2 -> 4

Commit message: almomst done
Parts:
- removed C1: 100nF, Capacitor_SMD:C_0603_1608Metric_Pad1.08x0.95mm_HandSolder
- removed R1, R39: 10k, Resistor_SMD:R_0603_1608Metric_Pad0.98x0.95mm_HandSolder
- added JP8: SolderJumper_2_Open, Jumper:SolderJumper-2_P1.3mm_Open_TrianglePad1.0x1.5mm, B.Cu at (129.9, 71.6)
- C2, D47, D48, R2, R3, R4, R65, R66: moved to F.Cu
- C33, C34, JP7, TP1, TP2: moved to B.Cu
- GND: renamed from TP4; footprint TestPoint:TestPoint_Pad_D2.5mm -> TestPoint:TestPoint_Pad_1.0x1.0mm
- TP3: footprint TestPoint:TestPoint_Pad_D2.5mm -> TestPoint:TestPoint_Pad_1.0x1.0mm
- moved R35 64.0 mm to (118.7, 57.0), turned to 90 degrees
- moved C46 63.5 mm to (145.7, 55.0), turned to 180 degrees
- moved C45 63.2 mm to (145.7, 53.2)
- moved R7 60.8 mm to (113.9, 69.3), turned to -90 degrees
- moved R8 59.8 mm to (114.1, 74.7), turned to 90 degrees
- moved R36 59.7 mm to (118.7, 53.3), turned to -90 degrees
- moved C2 55.1 mm to (148.7, 73.9), turned to 180 degrees
- moved C5 52.9 mm to (117.3, 74.2)
- moved TP3 49.3 mm to (161.2, 73.2)
- moved C4 48.7 mm to (121.4, 74.1)
- moved R2 48.3 mm to (147.4, 85.5)
- moved GND 47.0 mm to (163.5, 73.2)
- moved R4 44.5 mm to (147.6, 79.3), turned to -90 degrees
- moved R3 43.4 mm to (153.3, 73.8), turned to 0 degrees
- moved D10 40.5 mm to (110.6, 92.6), turned to 180 degrees
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Connections:
- D2 pad 1: Net-(D2-K) -> GND
- D2 pad 2: +3V3 -> Net-(D2-A)
- D3 pad 1: Net-(D3-K) -> GND
- D3 pad 2: +5V -> Net-(D3-A)
- D4 pad 1: Net-(D4-K) -> GND
- D4 pad 2: +12V -> Net-(D4-A)
- D6 pad 1: Net-(D6-K) -> GND
- D6 pad 2: /IND_1 -> Net-(D6-A)
- D7 pad 1: Net-(D7-K) -> GND
- D7 pad 2: /IND_2 -> Net-(D7-A)
- J1 pad 11: /STRT2 -> /HAT_connections/GPIO17
- J1 pad 13: /IVC_SW_1_SOL -> /SPI_CS4
- J1 pad 15: /IVC_SW_1_SOL -> /SPI_CS3
- J1 pad 16: /SPI_CS3 -> /HAT_connections/GPIO23
- J1 pad 18: /SPI_CS4 -> /STRT2
- J1 pad 22: /SERVO_1 -> /~{DRDY1}
- J1 pad 24: /SPI_CS1 -> /SPI_CS2
- J1 pad 26: /SPI_CS2 -> /SPI_CS1
- J1 pad 27: /INT_SLCTB -> /~{DRDY2}
- J1 pad 28: /SERVO_2 -> /STRT1
- J1 pad 29: /INT_SLCTA -> /INT_SLCTB
- J1 pad 31: /LED_PWM_1 -> /HAT_connections/EXP_INT_B
- J1 pad 32: /BUZZER -> /HAT_connections/GPIO12/PWM0
- J1 pad 33: /LED_PWM_2 -> /HAT_connections/EXP_INT_A
- J1 pad 35: /~{DRDY1} -> /SERVO_2
- J1 pad 36: /HAT_connections/GPIO16 -> /BUZZER
- J1 pad 37: /~{DRDY2} -> /SERVO_1
- J1 pad 38: /HAT_connections/EXP_INT_A -> /LED_PWM_1
- J1 pad 40: /HAT_connections/EXP_INT_B -> /LED_PWM_2
- J1 pad 7: /STRT1 -> /INT_SLCTA
- J6 pad 1: +12V -> GND
- J6 pad 2: GND -> +3V3
- J6 pad 3: +3V3 -> GND
- J6 pad 4: GND -> +12V
- R10 pad 1: Net-(D2-K) -> +3V3
- R10 pad 2: GND -> Net-(D2-A)
- R11 pad 1: Net-(D3-K) -> +5V
- R11 pad 2: GND -> Net-(D3-A)
- R12 pad 1: Net-(D4-K) -> +12V
- R12 pad 2: GND -> Net-(D4-A)
- R14 pad 1: Net-(D6-K) -> /IND_1
- R14 pad 2: GND -> Net-(D6-A)
- R16 pad 1: Net-(D7-K) -> /IND_2
- R16 pad 2: GND -> Net-(D7-A)
- R9 pad 1: /HAT_connections/GPIO16 -> /HAT_connections/GPIO12/PWM0
- U7 pad 1: /MOTOR_1_B -> /MOTOR_2_A
- U7 pad 15: Net-(U7-A0) -> GND
- U7 pad 16: Net-(U7-A0) -> GND
- U7 pad 18: /HAT_connections/GPIO16 -> /HAT_connections/GPIO12/PWM0
- U7 pad 2: /MOTOR_1_A -> /MOTOR_2_B
- U7 pad 23: /IVC_SW_2 -> /IVC_SW_2_SOL
- U7 pad 24: /IVC_SW_1 -> /IVC_SW_1_SOL
- U7 pad 25: /IVC_SW_1_SOL -> /IVC_SW_1
- U7 pad 26: /IVC_SW_2_SOL -> /IVC_SW_2
- U7 pad 28: /HAT_connections/I2CB_EN -> /~{GPS_RST}
- U7 pad 3: /MOTOR_2_B -> /MOTOR_1_A
- U7 pad 4: /MOTOR_2_A -> /MOTOR_1_B
- U7 pad 8: /~{GPS_RST} -> /HAT_connections/I2CB_EN
Routing:
- net +5V: track 0.00 -> 99.4 mm, vias 0 -> 3
- net /INT_SLCTB: track 0.00 -> 80.7 mm, vias 0 -> 1
- net /STRT1: track 0.00 -> 79.5 mm, vias 0 -> 2
- net /~{DRDY2}: track 0.00 -> 78.9 mm, vias 0 -> 1
- net /SPI_CS2: track 0.00 -> 73.3 mm, vias 0 -> 1
- net /I2C_SCL: track 5.38 -> 78.3 mm, vias 0 -> 2
- net /SPI_CS1: track 0.00 -> 72.3 mm, vias 0 -> 1
- net /I2C_SDA: track 8.97 -> 80.6 mm, vias 0 -> 2
- net +3V3: track 2.58 -> 68.6 mm, vias 1 -> 12
- net /SPI_SCLK: track 0.00 -> 53.0 mm, vias 0 -> 1
- net /SPI_MISO: track 0.00 -> 52.6 mm, vias 0 -> 1
- net /SPI_CS4: track 0.00 -> 52.1 mm, vias 0 -> 1
- net /SPI_CS3: track 0.00 -> 52.1 mm, vias 0 -> 1
- net /~{DRDY1}: track 0.00 -> 51.5 mm, vias 0 -> 1
- net /STRT2: track 0.00 -> 50.8 mm, vias 0 -> 1
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- added copper zone on In2.Cu, net +3V3
- added copper zone on B.Cu, net +5V
- added copper zone on F.Cu, net +5V
- added copper zone on In1.Cu, net +5V
- added copper zone on B.Cu, net GND
- added copper zone on F.Cu, net GND
- added copper zone on In1.Cu, net GND
- removed copper zone on B.Cu, net (none)
- removed copper zone on F.Cu, net (none)
- removed copper zone on In1.Cu, net (none)
- removed copper zone on In1.Cu, net +3V3
- removed copper zone on In2.Cu, net GND
Other:
- board text added: "12V"
- board text added: "3V3"
- board text added: "5V"
- board text added: "ALTAIR Interface HAT Ben D'Agnillo March 2026 - v1.0"
- board text added: "GND"
- board text added: "IND1"
- board text added: "IND2"

Commit message: complete BOM
Parts:
- removed D11: TVS_13V, Diode_SMD:D_0603_1608Metric_Pad1.05x0.95mm_HandSolder
- removed GND: TestPoint, TestPoint:TestPoint_Pad_1.0x1.0mm
- added TP4: TestPoint, TestPoint:TestPoint_Pad_1.0x1.0mm, F.Cu at (163.6, 73.2)
- C3: value 40pF -> 47pF; footprint Capacitor_SMD:C_0603_1608Metric_Pad1.08x0.95mm_HandSolder -> Capacitor_SMD:C_0402_1005Metric
- L1: footprint Inductor_SMD:L_0603_1608Metric_Pad1.05x0.95mm_HandSolder -> Inductor_SMD:L_0402_1005Metric
- TP1, TP2: moved to F.Cu
- U1: footprint MAX-M10M:XCVR_MAX-M10M-00B -> MAXX-M10M:XCVR_MAX-M10M-00B
- moved JP1 2.10 mm to (155.9, 90.8)
- moved L1 1.38 mm to (153.0, 91.5)
- moved C3 0.36 mm to (151.0, 91.0)
- turned TP1 to 180 degrees
- turned TP2 to 180 degrees
Routing:
- net /SPI_CS2: track 73.3 -> 70.6 mm
- net /GPS/VCC_RF: track 5.67 -> 4.38 mm
- net /GPS/GPS_SIG: track 7.25 -> 6.27 mm
- net /GPS/RF_IN: track 3.41 -> 4.16 mm
- net GND: vias 89 -> 109

Commit message: exported files, working on BOM orders
Changed lines of the file:
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@@
 		(grid_origin 100 100)
 		(pcbplotparams
-			(layerselection 0x00000000_00000000_00000000_000000a5)
+			(layerselection 0x00000000_00000000_55555555_5755f5ff)
 			(plot_on_all_layers_selection 0x00000000_00000000_00000000_00000000)
 			(disableapertmacros no)
 			(usegerberextensions yes)
-			(usegerberattributes no)
-			(usegerberadvancedattributes no)
+			(usegerberattributes yes)
+			(usegerberadvancedattributes yes)
 			(creategerberjobfile no)
 			(dashed_line_dash_ratio 12)
@@
 			(plotpadnumbers no)
 			(hidednponfab no)
-			(sketchdnponfab yes)
-			(crossoutdnponfab yes)
+			(sketchdnponfab no)
+			(crossoutdnponfab no)
 			(subtractmaskfromsilk no)
 			(outputformat 1)
 			(mirror no)
-			(drillshape 1)
+			(drillshape 0)
 			(scaleselection 1)
-			(outputdirectory "")
+			(outputdirectory "Fabrication outputs/NC Drill/")
 		)
 	)
@@
 		(tags "buzzer piezo")
 		(property "Reference" "BZ1"
-			(at 0 -5.5 90)
+			(at 0 -5.5 270)
 			(layer "F.SilkS")
-			(hide yes)
 			(effects
 				(font
@@
 		)
 		(property "Value" "Buzzer"
-			(at 0 5.5 90)
+			(at 0 5.5 270)
 			(layer "F.Fab")
-			(hide yes)
 			(effects
 				(font
@@
 			)
 		)
-		(property "Description" "Buzzer, polarized"
+		(property "Description" ""
 			(at 0 0 270)
 			(unlocked yes)
@@
 		(sheetname "/")
 		(sheetfile "interface_db_hat.kicad_sch")
-		(units
-			(unit
-				(name "A")
-				(pins "1" "2")
-			)
-		)
 		(attr smd)
 		(duplicate_pad_numbers_are_jumpers no)
@@
 		)
 		(fp_text user "${REFERENCE}"
-			(at 0 0 90)
+			(at 0 0 270)
 			(layer "F.Fab")
 			(effects
@@
 		)
 		(embedded_fonts no)
-		(model "${KICAD10_3DMODEL_DIR}/Buzzer_Beeper.3dshapes/Buzzer_CUI_CPT-9019S-SMT.step"
+		(model "${KIPRJMOD}/Imported Components/Buzzer/SMT-0952-T-5V-R_PUI.step"
 			(offset
 				(xyz 0 0 0)

Commit message: ordered
Parts:
- C31, C34, C46: footprint Capacitor_SMD:C_0603_1608Metric_Pad1.08x0.95mm_HandSolder -> Capacitor_SMD:C_0805_2012Metric
- moved C32 7.87 mm to (116.2, 93.2), turned to 90 degrees
- moved C46 0.60 mm to (145.7, 55.6)
- moved C45 0.60 mm to (145.7, 53.8)
- moved C34 0.30 mm to (108.4, 59.5)
Routing:
- net +12V: track 34.1 -> 29.6 mm
