File: interface_db_hat/interface_db_hat.kicad_sch (KiCad schematic)
At the start: 55 parts, among them J2 Conn_02x06_Counter_Clockwise, J3 Conn_02x10_Counter_Clockwise, J6 Conn_01x04_Pin, J7 Conn_01x20_Pin, Q1 BC817

Commit message: lol
Parts:
- removed J3: Conn_02x10_Counter_Clockwise, symbol Connector_Generic:Conn_02x10_Counter_Clockwise
- added J3: Conn_02x06_Counter_Clockwise, Connector_PinSocket_2.54mm:PinSocket_2x06_P2.54mm_Vertical, symbol Connector_Generic:Conn_02x06_Counter_Clockwise
- added R1: 10k, symbol Device:R_US
- R5: value R_US -> 1k
Connections:
- net +3V3: now also R1.2
- net GND: now also J3.3 (Pin_3), J3.7 (Pin_7)
- net I2C_SCL: now also J3.1 (Pin_1)
- net I2C_SDA: now also J3.2 (Pin_2)
- net ~{SYS_RESET} renamed ~{PD_RESET}
- net ~{PD_RESET}: now also R1.1
- new net IND_2: J3.10 (Pin_10)
- new net LED_1: J3.12 (Pin_12)
- new net LED_2: J3.11 (Pin_11)
- new net SERVO_1: J3.4 (Pin_4)
- new net SERVO_2: J3.5 (Pin_5)
- new net SERVO_3: J3.6 (Pin_6)
Other:
- sheet HAT_connections ports: added none; removed GPA7, PD_RST
- moved on the sheet: BZ1, Q1, R5

Commit message: UPDATE
Parts:
- removed D14, D17, D18, D19, D20, D21, D22, D23, D24, D25, D26, D27, D28, D29, D30, D31, D32, D33, D34, D35: TVS_3V3, Diode_SMD:D_0603_1608Metric_Pad1.05x0.95mm_HandSolder, symbol Device:D_Zener
- removed R5: 1k, symbol Device:R_US
- removed TP1, TP2: TestPoint_2Pole, Connector_PinHeader_2.54mm:PinHeader_1x02_P2.54mm_Vertical, symbol Connector:TestPoint_2Pole
- added D15, D16, D39, D41, D42, D43, D44, D45, D46: TVS_3V3, Diode_SMD:D_0402_1005Metric_Pad0.77x0.64mm_HandSolder, symbol Device:D_Zener
- added R13, R15: 330, Resistor_SMD:R_0603_1608Metric_Pad0.98x0.95mm_HandSolder, symbol Device:R_US
- BZ1: value WT-1205 -> Buzzer; footprint (none) -> Buzzer_Beeper:Buzzer_12x9.5RM7.6
- D10: footprint Diode_SMD:D_0603_1608Metric_Pad1.05x0.95mm_HandSolder -> Diode_SMD:D_0402_1005Metric_Pad0.77x0.64mm_HandSolder
- R1: footprint (none) -> Resistor_SMD:R_0603_1608Metric_Pad0.98x0.95mm_HandSolder
Connections:
- net +3V3: now also J2.7 (Pin_7), J2.8 (Pin_8), D46.1 (K)
- net +5V: now also R15.1; no longer J2.7 (Pin_7), J2.8 (Pin_8)
- net BUZZER: now also R13.1
- net GND: now also J3.10 (Pin_10), J3.8 (Pin_8), D15.2 (A), D16.2 (A), D39.2 (A), D41.2 (A), D42.2 (A), D43.2 (A), D44.2 (A), D45.2 (A), D46.2 (A)
- net I2C_SCL: now also D44.1 (K)
- net I2C_SDA: now also D45.1 (K)
- net IND_2: now also J3.9 (Pin_9), D43.1 (K); no longer J3.10 (Pin_10)
- net IVC_SW_1_SOL: no longer R45.1
- net LED_1: now also D41.1 (K)
- net LED_2: now also D42.1 (K)
- net SERVO_1: now also D39.1 (K)
- net SERVO_2: now also D16.1 (K)
- net SERVO_3: now also D15.1 (K)
- net at BZ1.2 (-), Q1.3 (C): now also R15.2
- net at Q1.1 (B): now also R13.2
- new net IVC_SW_2_SOL: R45.1
Other:
- added sheet test_points_and_indicators (test_points_and_indicators.kicad_sch)
- sheet GPS ports: added I2C_SCL, I2C_SDA; removed GPS_RXD, GPS_TXD
- sheet HAT_connections ports: added GPB0, GPB1, GPB2, GPB3, GPB4, GPB5, GPB6, GPB7; removed RXDO, TXDO
- note added: "PD Pin Timing low priority - SYS_RESET, INT_SLCTB, INT_SLCTA, IVC_SW_1, IVC_SW_2, DRDY1, DRDY2"
- moved on the sheet: BZ1, C1, C30, D1, D10, D11, D40, J2, J3, J6, J7, Q1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

Commit message: lol
Parts:
- removed D1: 5V, Diode_SMD:D_0603_1608Metric_Pad1.05x0.95mm_HandSolder, symbol Device:D_Zener
- removed D15, D16, D39, D41, D42, D43, D44, D45, D46: TVS_3V3, Diode_SMD:D_0402_1005Metric_Pad0.77x0.64mm_HandSolder, symbol Device:D_Zener
- removed D40: TVS_13V, Diode_SMD:D_0603_1608Metric_Pad1.05x0.95mm_HandSolder, symbol Device:D_Zener
- removed J2: Conn_02x06_Counter_Clockwise, Connector_PinSocket_2.54mm:PinSocket_2x06_P2.54mm_Vertical, symbol Connector_Generic:Conn_02x06_Counter_Clockwise
- removed R13: 330, Resistor_SMD:R_0603_1608Metric_Pad0.98x0.95mm_HandSolder, symbol Device:R_US
- added C31, C34, C36: 22uF, Capacitor_SMD:C_0603_1608Metric_Pad1.08x0.95mm_HandSolder, symbol Device:C
- added C32, C33, C35: 100nF, Capacitor_SMD:C_0603_1608Metric_Pad1.08x0.95mm_HandSolder, symbol Device:C
- added J10, J9: Conn_02x06_Counter_Clockwise, Connector_PinSocket_2.54mm:PinSocket_2x06_P2.54mm_Vertical, symbol Connector_Generic:Conn_02x06_Odd_Even
- added R17: 330, Resistor_SMD:R_0603_1608Metric_Pad0.98x0.95mm_HandSolder, symbol Device:R_US
- BZ1: footprint Buzzer_Beeper:Buzzer_12x9.5RM7.6 -> Buzzer_Beeper:Buzzer_CUI_CPT-9019S-SMT
- J3: symbol Connector_Generic:Conn_02x06_Counter_Clockwise -> Connector_Generic:Conn_02x06_Odd_Even
Connections:
- net LED_1 is gone; now on net GND: J3.12 (Pin_12)
- net LED_2 is gone; now on net LED_PWM_1: J3.11 (Pin_11)
- net +12V: now also C31.1, C32.2, J10.2 (Pin_2), J10.4 (Pin_4), J10.6 (Pin_6), J10.8 (Pin_8)
- net +3V3: now also C35.2, C36.1, J10.1 (Pin_1), J10.3 (Pin_3)
- net +5V: now also C33.2, C34.1, J10.11 (Pin_11), J10.5 (Pin_5), J10.7 (Pin_7), J10.9 (Pin_9), R17.1; no longer R15.1
- net BUZZER: now also R15.1
- net GND: now also J3.2 (Pin_2), J3.4 (Pin_4), C31.2, C32.1, C33.1, C34.2, C35.1, C36.2, J10.10 (Pin_10), J10.12 (Pin_12), J9.10 (Pin_10), J9.11 (Pin_11), J9.12 (Pin_12), J9.2 (Pin_2), J9.4 (Pin_4), J9.6 (Pin_6), J9.8 (Pin_8), J9.9 (Pin_9); no longer J3.10 (Pin_10), J3.8 (Pin_8)
- net I2C_SCL: now also J3.5 (Pin_5); no longer J3.1 (Pin_1)
- net I2C_SDA: now also J3.1 (Pin_1); no longer J3.2 (Pin_2)
- net IND_2: now also J3.6 (Pin_6); no longer J3.9 (Pin_9)
- net IND_3: now also J3.8 (Pin_8)
- net IND_4: now also J3.10 (Pin_10)
- net LED_PWM_2: now also J3.9 (Pin_9)
- net SERVO_1: now also J9.1 (Pin_1); no longer J3.4 (Pin_4)
- net SERVO_2: now also J9.3 (Pin_3); no longer J3.5 (Pin_5)
- net SERVO_3: now also J9.5 (Pin_5); no longer J3.6 (Pin_6)
- net SERVO_4: now also J9.7 (Pin_7)
- net at BZ1.2 (-), Q1.3 (C): now also R17.2; no longer R15.2
- net at Q1.1 (B): now also R15.2
Other:
- sheet test_points_and_indicators ports: added IND_0, IND_1; removed IND
- moved on the sheet: J3

Commit message: termination
Connections:
- net IND_4 is gone; now on net GND: J3.10 (Pin_10)
- net GND: no longer J3.2 (Pin_2), J3.4 (Pin_4)
- net IND_2: no longer J3.6 (Pin_6)
- net IND_3: no longer J3.8 (Pin_8)
- new net MOTOR_1: J3.2 (Pin_2)
- new net MOTOR_2: J3.4 (Pin_4)
- new net MOTOR_3: J3.6 (Pin_6)
- new net MOTOR_4: J3.8 (Pin_8)
Changed lines of the file:
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@@
+	)
+	(junction
+		(at 76.2 139.7)
+		(diameter 0)
+		(color 0 0 0 0)
 	)
 	(junction
@@
 	)
 	(junction
+		(at 76.2 142.24)
+		(diameter 0)
+		(color 0 0 0 0)
+	)
+	(junction
 		(at 171.45 106.68)
 		(diameter 0)
@@
 	)
 	(junction
-		(at 77.47 139.7)
-		(diameter 0)
-		(color 0 0 0 0)
-	)
-	(junction
 		(at 38.1 160.02)
 		(diameter 0)
@@
 	)
 	(junction
-		(at 77.47 142.24)
-		(diameter 0)
-		(color 0 0 0 0)
-	)
-	(junction
 		(at 69.85 160.02)
 		(diameter 0)
@@
 	)
 	(junction
-		(at 76.2 129.54)
-		(diameter 0)
-		(color 0 0 0 0)
-	)
-	(junction
 		(at 123.19 158.75)
 		(diameter 0)
@@
 	(wire
 		(pts
-			(xy 76.2 132.08) (xy 80.01 132.08)
-		)
-		(stroke
-			(width 0)
-			(type default)
-		)
-	)
-	(wire
-		(pts
 			(xy 45.72 68.58) (xy 53.34 68.58)
 		)
@@
 	(wire
 		(pts
-			(xy 77.47 129.54) (xy 77.47 139.7)
-		)
-		(stroke
-			(width 0)
-			(type default)
-		)
-	)
-	(wire
-		(pts
 			(xy 45.72 76.2) (xy 53.34 76.2)
 		)
@@
 	(wire
 		(pts
-			(xy 60.96 142.24) (xy 77.47 142.24)
+			(xy 60.96 142.24) (xy 76.2 142.24)
 		)
 		(stroke
@@
 	(wire
 		(pts
+			(xy 76.2 127) (xy 78.74 127)
+		)
+		(stroke
+			(width 0)
+			(type default)
+		)
+	)
+	(wire
+		(pts
 			(xy 223.52 53.34) (xy 228.6 53.34)
 		)
@@
 	(wire
 		(pts
+			(xy 76.2 134.62) (xy 78.74 134.62)
+		)
+		(stroke
+			(width 0)
+			(type default)
+		)
+	)
+	(wire
+		(pts
 			(xy 171.45 118.11) (xy 171.45 120.65)
 		)
@@
 	(wire
 		(pts
-			(xy 76.2 134.62) (xy 80.01 134.62)
-		)
-		(stroke
-			(width 0)
-			(type default)
-		)
-	)
-	(wire
-		(pts
 			(xy 255.27 118.11) (xy 255.27 123.19)
 		)
@@
 	(wire
 		(pts
-			(xy 76.2 137.16) (xy 80.01 137.16)
-		)
-		(stroke
-			(width 0)
-			(type default)
-		)
-	)
-	(wire
-		(pts
 			(xy 60.96 134.62) (xy 60.96 142.24)
 		)
@@
 	(wire
 		(pts
+			(xy 76.2 129.54) (xy 78.74 129.54)
+		)
+		(stroke
+			(width 0)
+			(type default)
+		)
+	)
+	(wire
+		(pts
+			(xy 76.2 137.16) (xy 76.2 139.7)
+		)
+		(stroke
+			(width 0)
+			(type default)
+		)
+	)
+	(wire
+		(pts
 			(xy 45.72 78.74) (xy 53.34 78.74)
 		)
@@
 	(wire
 		(pts
-			(xy 76.2 127) (xy 76.2 129.54)
-		)
-		(stroke
-			(width 0)
-			(type default)
-		)
-	)
-	(wire
-		(pts
 			(xy 245.11 123.19) (xy 255.27 123.19)
 		)
@@
 	(wire
 		(pts
-			(xy 77.47 139.7) (xy 76.2 139.7)
-		)
-		(stroke
-			(width 0)
-			(type default)
-		)
-	)
-	(wire
-		(pts
 			(xy 223.52 45.72) (xy 228.6 45.72)
 		)
@@
 	(wire
 		(pts
-			(xy 77.47 139.7) (xy 77.47 142.24)
-		)
-		(stroke
-			(width 0)
-			(type default)
-		)
-	)
-	(wire
-		(pts
 			(xy 95.25 60.96) (xy 100.33 60.96)
 		)
@@
 	(wire
 		(pts
+			(xy 76.2 139.7) (xy 76.2 142.24)
+		)
+		(stroke
+			(width 0)
+			(type default)
+		)
+	)
+	(wire
+		(pts
 			(xy 166.37 55.88) (xy 168.91 55.88)
 		)
@@
 	(wire
 		(pts
-			(xy 76.2 129.54) (xy 77.47 129.54)
+			(xy 76.2 132.08) (xy 78.74 132.08)
 		)
 		(stroke
@@
 		(pts
 			(xy 45.72 96.52) (xy 53.34 96.52)
+		)
+		(stroke
+			(width 0)
+			(type default)
+		)
+	)
+	(wire
+		(pts
+			(xy 76.2 142.24) (xy 77.47 142.24)
 		)
 		(stroke
@@
 		)
 	)
-	(label "IND_4"
+	(label "MOTOR_4"
 		(at 45.72 50.8 180)
 		(effects
@@
 		)
 	)
-	(label "IND_2"
-		(at 80.01 132.08 0)
-		(effects
-			(font
-				(size 1.27 1.27)
-			)
-			(justify left bottom)
-		)
-	)
-	(label "IND_0"
+	(label "IND_1"
 		(at 139.7 30.48 180)
 		(effects
@@
 		)
 	)
-	(label "IND_1"
+	(label "MOTOR_1"
 		(at 45.72 43.18 180)
 		(effects
@@
 		)
 	)
-	(label "IND_0"
+	(label "IND_3"
 		(at 45.72 38.1 180)
 		(effects
@@
 		)
 	)
+	(label "MOTOR_1"
+		(at 78.74 127 0)
+		(effects
+			(font
+				(size 1.27 1.27)
+			)
+			(justify left bottom)
+		)
+	)
 	(label "I2C_SCL"
 		(at 138.43 59.69 180)
@@
 		)
 	)
-	(label "IND_6"
+	(label "IND_2"
 		(at 49.53 25.4 180)
 		(effects
@@
 		)
 	)
-	(label "IND_2"
+	(label "MOTOR_2"
 		(at 45.72 45.72 180)
 		(effects
@@
 		)
 	)
-	(label "IND_3"
-		(at 80.01 134.62 0)
-		(effects
-			(font
-				(size 1.27 1.27)
-			)
-			(justify left bottom)
-		)
-	)
 	(label "IVC_SW_1_SOL"
 		(at 49.53 33.02 180)
@@
 		)
 	)
-	(label "IND_3"
+	(label "MOTOR_3"
 		(at 45.72 48.26 180)
 		(effects
@@
 		)
 	)
-	(label "IND_1"
+	(label "IND_2"
 		(at 139.7 33.02 180)
 		(effects
@@
 		)
 	)
-	(label "IND_5"
+	(label "IND_1"
 		(at 49.53 22.86 180)
 		(effects
@@
 		)
 	)
+	(label "MOTOR_2"
+		(at 78.74 129.54 0)
+		(effects
+			(font
+				(size 1.27 1.27)
+			)
+			(justify left bottom)
+		)
+	)
 	(label "SPI_MISO"
 		(at 223.52 55.88 180)
@@
 		)
 	)
-	(label "IND_4"
-		(at 80.01 137.16 0)
+	(label "MOTOR_4"
+		(at 78.74 134.62 0)
 		(effects
 			(font
@@
 		)
 	)
+	(label "MOTOR_3"
+		(at 78.74 132.08 0)
+		(effects
+			(font
+				(size 1.27 1.27)
+			)
+			(justify left bottom)
+		)
+	)

Commit message: update
Connections:
- net MOTOR_1: no longer J3.2 (Pin_2)
- net MOTOR_2: no longer J3.4 (Pin_4)
- net MOTOR_3: no longer J3.6 (Pin_6)
- net MOTOR_4: no longer J3.8 (Pin_8)
- new net MOTOR_1_A: J3.2 (Pin_2)
- new net MOTOR_1_B: J3.4 (Pin_4)
- new net MOTOR_2_A: J3.6 (Pin_6)
- new net MOTOR_2_B: J3.8 (Pin_8)
Other:
- note added: "TODO ESC CONNECTIONS"
- moved on the sheet: J9
Changed lines of the file:
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@@
 		)
 	)
+	(text "TODO ESC CONNECTIONS"
+		(exclude_from_sim no)
+		(at 167.132 142.494 0)
+		(effects
+			(font
+				(size 1.27 1.27)
+			)
+		)
+	)
 	(junction
-		(at 129.54 146.05)
+		(at 123.19 133.35)
 		(diameter 0)
 		(color 0 0 0 0)
@@
 	)
 	(junction
-		(at 116.84 156.21)
+		(at 110.49 143.51)
 		(diameter 0)
 		(color 0 0 0 0)
@@
 	)
 	(junction
-		(at 129.54 151.13)
+		(at 123.19 138.43)
 		(diameter 0)
 		(color 0 0 0 0)
@@
 	)
 	(junction
-		(at 129.54 153.67)
+		(at 123.19 140.97)
 		(diameter 0)
 		(color 0 0 0 0)
@@
 	)
 	(junction
-		(at 129.54 156.21)
+		(at 123.19 143.51)
 		(diameter 0)
 		(color 0 0 0 0)
 	)
 	(junction
-		(at 129.54 148.59)
+		(at 123.19 135.89)
 		(diameter 0)
 		(color 0 0 0 0)
@@
 	)
 	(junction
-		(at 123.19 158.75)
+		(at 116.84 146.05)
 		(diameter 0)
 		(color 0 0 0 0)
@@
 	(wire
 		(pts
-			(xy 129.54 156.21) (xy 129.54 158.75)
+			(xy 123.19 143.51) (xy 123.19 146.05)
 		)
 		(stroke
@@
 	(wire
 		(pts
-			(xy 129.54 143.51) (xy 129.54 146.05)
+			(xy 123.19 130.81) (xy 123.19 133.35)
 		)
 		(stroke
@@
 	(wire
 		(pts
-			(xy 111.76 151.13) (xy 116.84 151.13)
+			(xy 105.41 138.43) (xy 110.49 138.43)
 		)
 		(stroke
@@
 	(wire
 		(pts
-			(xy 111.76 143.51) (xy 116.84 143.51)
+			(xy 105.41 130.81) (xy 110.49 130.81)
 		)
 		(stroke
@@
 	(wire
 		(pts
-			(xy 111.76 146.05) (xy 116.84 146.05)
+			(xy 105.41 133.35) (xy 110.49 133.35)
 		)
 		(stroke
@@
 	(wire
 		(pts
-			(xy 129.54 153.67) (xy 129.54 156.21)
+			(xy 123.19 140.97) (xy 123.19 143.51)
 		)
 		(stroke
@@
 	(wire
 		(pts
-			(xy 129.54 148.59) (xy 129.54 151.13)
+			(xy 123.19 135.89) (xy 123.19 138.43)
 		)
 		(stroke
@@
 	(wire
 		(pts
-			(xy 116.84 153.67) (xy 116.84 156.21)
+			(xy 110.49 140.97) (xy 110.49 143.51)
 		)
 		(stroke
@@
 	(wire
 		(pts
-			(xy 123.19 158.75) (xy 129.54 158.75)
+			(xy 116.84 146.05) (xy 123.19 146.05)
 		)
 		(stroke
@@
 	(wire
 		(pts
-			(xy 116.84 158.75) (xy 123.19 158.75)
+			(xy 110.49 146.05) (xy 116.84 146.05)
 		)
 		(stroke
@@
 	(wire
 		(pts
-			(xy 129.54 151.13) (xy 129.54 153.67)
+			(xy 123.19 138.43) (xy 123.19 140.97)
 		)
 		(stroke
@@
 	(wire
 		(pts
-			(xy 116.84 156.21) (xy 116.84 158.75)
+			(xy 110.49 143.51) (xy 110.49 146.05)
 		)
 		(stroke
@@
 	(wire
 		(pts
-			(xy 111.76 148.59) (xy 116.84 148.59)
+			(xy 105.41 135.89) (xy 110.49 135.89)
 		)
 		(stroke
@@
 	(wire
 		(pts
-			(xy 129.54 146.05) (xy 129.54 148.59)
+			(xy 123.19 133.35) (xy 123.19 135.89)
 		)
 		(stroke
@@
 		)
 	)
+	(label "MOTOR_1_B"
+		(at 78.74 129.54 0)
+		(effects
+			(font
+				(size 1.27 1.27)
+			)
+			(justify left bottom)
+		)
+	)
 	(label "I2C_SCL"
 		(at 100.33 76.2 0)
@@
 	)
 	(label "SERVO_3"
-		(at 111.76 148.59 180)
+		(at 105.41 135.89 180)
 		(effects
 			(font
@@
 		)
 	)
-	(label "SERVO_1"
-		(at 45.72 93.98 180)
+	(label "MOTOR_2_A"
+		(at 78.74 132.08 0)
 		(effects
 			(font
 				(size 1.27 1.27)
 			)
-			(justify right bottom)
+			(justify left bottom)
 		)
 	)
-	(label "SPI_SCLK"
-		(at 223.52 48.26 180)
+	(label "SERVO_1"
+		(at 45.72 93.98 180)
 		(effects
 			(font
@@
 		)
 	)
-	(label "MOTOR_1"
-		(at 78.74 127 0)
+	(label "SPI_SCLK"
+		(at 223.52 48.26 180)
 		(effects
 			(font
 				(size 1.27 1.27)
 			)
-			(justify left bottom)
+			(justify right bottom)
 		)
 	)
@@
 	)
 	(label "SERVO_4"
-		(at 111.76 151.13 180)
+		(at 105.41 138.43 180)
 		(effects
 			(font
@@
 	)
 	(label "SERVO_2"
-		(at 111.76 146.05 180)
+		(at 105.41 133.35 180)
 		(effects
 			(font
@@
 		)
 	)
+	(label "MOTOR_2_B"
+		(at 78.74 134.62 0)
+		(effects
+			(font
+				(size 1.27 1.27)
+			)
+			(justify left bottom)
+		)
+	)
 	(label "~{DRDY1}"
 		(at 223.52 68.58 180)
@@
 		)
 	)
+	(label "MOTOR_1_A"
+		(at 78.74 127 0)
+		(effects
+			(font
+				(size 1.27 1.27)
+			)
+			(justify left bottom)
+		)
+	)
 	(label "~{DRDY2}"
 		(at 45.72 91.44 180)
@@
 		)
 	)
-	(label "MOTOR_2"
-		(at 78.74 129.54 0)
-		(effects
-			(font
-				(size 1.27 1.27)
-			)
-			(justify left bottom)
-		)
-	)
 	(label "SPI_MISO"
 		(at 223.52 55.88 180)
@@
 		)
 	)
-	(label "MOTOR_4"
-		(at 78.74 134.62 0)
-		(effects
-			(font
-				(size 1.27 1.27)
-			)
-			(justify left bottom)
-		)
-	)
 	(label "SERVO_1"
-		(at 111.76 143.51 180)
+		(at 105.41 130.81 180)
 		(effects
 			(font
@@
 		)
 	)
-	(label "MOTOR_3"
-		(at 78.74 132.08 0)
-		(effects
-			(font
-				(size 1.27 1.27)
-			)
-			(justify left bottom)
-		)
-	)
 	(label "IVC_SW_1"
 		(at 223.52 35.56 180)
@@
 	(symbol
 		(lib_id "Connector_Generic:Conn_02x06_Odd_Even")
-		(at 121.92 148.59 0)
+		(at 115.57 135.89 0)
 		(unit 1)
 		(body_style 1)
@@
 		(fields_autoplaced yes)
 		(property "Reference" "J9"
-			(at 123.19 137.16 0)
+			(at 116.84 124.46 0)
 			(show_name no)
 			(do_not_autoplace no)
@@
 		)
 		(property "Value" "Conn_02x06_Counter_Clockwise"
-			(at 123.19 139.7 0)
+			(at 116.84 127 0)
 			(show_name no)
 			(do_not_autoplace no)
@@
 		)
 		(property "Footprint" "Connector_PinSocket_2.54mm:PinSocket_2x06_P2.54mm_Vertical"
-			(at 121.92 148.59 0)
+			(at 115.57 135.89 0)
 			(hide yes)
 			(show_name no)
@@
 		)
 		(property "Datasheet" ""
-			(at 121.92 148.59 0)
+			(at 115.57 135.89 0)
 			(hide yes)
 			(show_name no)
@@
 		)
 		(property "Description" "Generic connector, double row, 02x06, odd/even pin numbering scheme (row 1 odd numbers, row 2 even numbers), script generated (kicad-library-utils/schlib/autogen/connector/)"
-			(at 121.92 148.59 0)
+			(at 115.57 135.89 0)
 			(hide yes)
 			(show_name no)
@@
 	(symbol
 		(lib_id "power:GND")
-		(at 123.19 158.75 0)
+		(at 116.84 146.05 0)
 		(unit 1)
 		(body_style 1)
@@
 		(dnp no)
 		(property "Reference" "#PWR057"
-			(at 123.19 165.1 0)
+			(at 116.84 152.4 0)
 			(hide yes)
 			(show_name no)
@@
 		)
 		(property "Value" "GND"
-			(at 123.19 163.83 0)
+			(at 116.84 151.13 0)
 			(show_name no)
 			(do_not_autoplace no)
@@
 		)
 		(property "Footprint" ""
-			(at 123.19 158.75 0)
+			(at 116.84 146.05 0)
 			(hide yes)
 			(show_name no)
@@
 		)
 		(property "Datasheet" ""
-			(at 123.19 158.75 0)
+			(at 116.84 146.05 0)
 			(hide yes)
 			(show_name no)
@@
 		)
 		(property "Description" "Power symbol creates a global label with name \"GND\" , ground"
-			(at 123.19 158.75 0)
+			(at 116.84 146.05 0)
 			(hide yes)
 			(show_name no)

Commit message: working on interface board
Parts:
- removed C35: 100nF, Capacitor_SMD:C_0603_1608Metric_Pad1.08x0.95mm_HandSolder, symbol Device:C
- removed C36: 22uF, Capacitor_SMD:C_0603_1608Metric_Pad1.08x0.95mm_HandSolder, symbol Device:C
- removed J7: Conn_01x20_Pin, Connector_PinHeader_1.00mm:PinHeader_1x20_P1.00mm_Vertical, symbol Connector:Conn_01x20_Pin
- added C45: 100nF, Capacitor_SMD:C_0603_1608Metric_Pad1.08x0.95mm_HandSolder, symbol Device:C
- added C46: 22uF, Capacitor_SMD:C_0603_1608Metric_Pad1.08x0.95mm_HandSolder, symbol Device:C
- added J2: DF19G-20P-1H52, DF-19:CONN20_DF19G_HIR, symbol DF-19:DF19G-20P-1H52
Connections:
- net SERVO_3 is gone; now on net +3V3: J9.5 (Pin_5)
- net SERVO_4 is gone; now on net +3V3: J9.7 (Pin_7)
- net +12V: now also J10.11 (Pin_11), J10.5 (Pin_5), J10.7 (Pin_7), J10.9 (Pin_9); no longer J10.2 (Pin_2), J10.4 (Pin_4), J10.6 (Pin_6), J10.8 (Pin_8)
- net +3V3: now also C45.2, C46.1; no longer J10.1 (Pin_1), J10.3 (Pin_3)
- net +5V: now also J3.1 (Pin_1), J3.2 (Pin_2), J3.3 (Pin_3), J3.4 (Pin_4), J3.5 (Pin_5), J3.6 (Pin_6), J3.7 (Pin_7), J3.8 (Pin_8); no longer J10.11 (Pin_11), J10.5 (Pin_5), J10.7 (Pin_7), J10.9 (Pin_9)
- net GND: now also J10.1 (Pin_1), J10.2 (Pin_2), J10.3 (Pin_3), J10.4 (Pin_4), J10.6 (Pin_6), J10.8 (Pin_8), J3.9 (Pin_9), C45.1, C46.2, J2.21 (SHIELD), J2.22 (SHIELD); no longer J3.12 (Pin_12), J3.3 (Pin_3), J3.7 (Pin_7), J9.10 (Pin_10), J9.11 (Pin_11), J9.12 (Pin_12), J9.2 (Pin_2), J9.4 (Pin_4), J9.6 (Pin_6), J9.8 (Pin_8)
- net I2C_SCL: now also J3.11 (Pin_11); no longer J3.5 (Pin_5)
- net I2C_SDA: now also J3.12 (Pin_12); no longer J3.1 (Pin_1)
- net IND_3: now also J9.11 (Pin_11)
- net LED_PWM_1: now also J9.10 (Pin_10); no longer J3.11 (Pin_11)
- net LED_PWM_2: now also J9.12 (Pin_12); no longer J3.9 (Pin_9)
- net MOTOR_1_A: now also J9.4 (Pin_4); no longer J3.2 (Pin_2)
- net MOTOR_1_B: now also J9.2 (Pin_2); no longer J3.4 (Pin_4)
- net MOTOR_2_A: now also J9.8 (Pin_8); no longer J3.6 (Pin_6)
- net MOTOR_2_B: now also J9.6 (Pin_6); no longer J3.8 (Pin_8)
- net SERVO_1: now also J9.3 (Pin_3); no longer J9.1 (Pin_1)
- net SERVO_2: now also J9.1 (Pin_1); no longer J9.3 (Pin_3)
- net at R55.2: now also J2.7
- net at R43.2: now also J2.19
- net at R57.2: now also J2.5
- net at R50.2: now also J2.12
- net at R61.2: now also J2.1
- net at R52.2: now also J2.10
- net at R51.2: now also J2.11
- net at R49.2: now also J2.13
- net at R48.2: now also J2.14
- net at R47.2: now also J2.15
- net at R46.2: now also J2.16
- net at R45.2: now also J2.17
- net at R44.2: now also J2.18
- net at R60.2: now also J2.2
- net at R42.2: now also J2.20
- net at R59.2: now also J2.3
- net at R58.2: now also J2.4
- net at R56.2: now also J2.6
- net at R54.2: now also J2.8
- net at R53.2: now also J2.9
Other:
- moved on the sheet: C31, C32, C33, C34, J9

Commit message: almomst done
Parts:
- removed C1: 100nF, Capacitor_SMD:C_0603_1608Metric_Pad1.08x0.95mm_HandSolder, symbol Device:C
- removed R1: 10k, Resistor_SMD:R_0603_1608Metric_Pad0.98x0.95mm_HandSolder, symbol Device:R_US
Connections:
- net +12V: now also J6.4 (Pin_4); no longer J6.1 (Pin_1)
- net +3V3: now also J6.2 (Pin_2); no longer J6.3 (Pin_3)
- net GND: now also J6.1 (Pin_1), J6.3 (Pin_3); no longer J6.2 (Pin_2), J6.4 (Pin_4)
Other:
- sheet HAT_connections ports: added GPA7; removed GPB7, GPIO_14
