File: interface_db_hat/HAT_connections.kicad_sch (KiCad schematic)
At the start: 23 parts, among them J1 GPIO, J5 Conn_01x04_Pin, J8 Conn_01x03_Pin, U2 TCA9617ADGKR, U7 MCP23017x-x-SO

Commit message: post 2nd revision update
Connections:
- net EXP_INT_A: no longer J1.33 (Pin_33)
- net EXP_INT_B: no longer J1.31 (Pin_31)
- new net GPIO_10: J1.31 (Pin_31)
- new net GPIO_12: J1.33 (Pin_33)
Changed lines of the file:
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@@
-		)
-	)
-	(label "EXP_INT_A"
-		(at 62.23 72.39 180)
-		(effects
-			(font
-				(size 1.27 1.27)
-			)
-			(justify right bottom)
 		)
 	)
@@
 		)
 	)
-	(label "EXP_INT_B"
-		(at 62.23 69.85 180)
-		(effects
-			(font
-				(size 1.27 1.27)
-			)
-			(justify right bottom)
-		)
-	)
