File: Ion-0/_restore_backup_2026-05-28T16-58-34-781/Ion-0.kicad_sch (KiCad schematic)
At the start: 15 parts, among them J1 Beaglebone-green-P9, J2 Beaglebone-green-P8, J3 Conn_02x06_Odd_Even, J4 Conn_02x06_Odd_Even, J5 Conn_02x06_Odd_Even

Commit message: midway through
Connections:
- net GPIO_38: now reaches J2.3 (Pin_3)
- net GPIO_34: now reaches J2.5 (Pin_5)
- net GPIO_50: no longer names the net of J1.14 (Pin_14)
- net GPIO_60: no longer names the net of J1.12 (Pin_12)
Changed lines of the file:
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@@
-	)
-	(no_connect
-		(at 90.17 26.67)
 	)
 	(no_connect
@@
 	)
 	(no_connect
-		(at 90.17 29.21)
-	)
-	(no_connect
 		(at 90.17 69.85)
 	)
@@
 	)
 	(no_connect
+		(at 48.26 35.56)
+	)
+	(no_connect
 		(at 48.26 55.88)
 	)
@@
 	)
 	(no_connect
+		(at 48.26 38.1)
+	)
+	(no_connect
 		(at 102.87 29.21)
 	)
@@
 	(wire
 		(pts
-			(xy 48.26 38.1) (xy 50.8 38.1)
-		)
-		(stroke
-			(width 0)
-			(type default)
-		)
-	)
-	(wire
-		(pts
 			(xy 34.29 76.2) (xy 34.29 78.74)
 		)
@@
 	(wire
 		(pts
+			(xy 87.63 29.21) (xy 90.17 29.21)
+		)
+		(stroke
+			(width 0)
+			(type default)
+		)
+	)
+	(wire
+		(pts
 			(xy 133.35 166.37) (xy 139.7 166.37)
 		)
@@
 	(wire
 		(pts
+			(xy 87.63 26.67) (xy 90.17 26.67)
+		)
+		(stroke
+			(width 0)
+			(type default)
+		)
+	)
+	(wire
+		(pts
 			(xy 233.68 29.21) (xy 238.76 29.21)
 		)
@@
 		(pts
 			(xy 25.4 163.83) (xy 25.4 171.45)
-		)
-		(stroke
-			(width 0)
-			(type default)
-		)
-	)
-	(wire
-		(pts
-			(xy 48.26 35.56) (xy 50.8 35.56)
 		)
 		(stroke
@@
 		)
 	)
-	(label "GPIO_50"
+	(label "GPIO_34"
 		(at 238.76 72.39 0)
 		(effects
@@
 		)
 	)
-	(label "GPIO_60"
-		(at 50.8 35.56 0)
-		(effects
-			(font
-				(size 1.27 1.27)
-			)
-			(justify left bottom)
-		)
-	)
 	(label "GPIO_76"
-		(at 198.12 29.21 180)
+		(at 198.12 26.67 180)
 		(effects
 			(font
@@
 	)
 	(label "GPIO_74"
-		(at 198.12 26.67 180)
+		(at 198.12 29.21 180)
 		(effects
 			(font
@@
 		)
 	)
-	(label "GPIO_50"
-		(at 50.8 38.1 0)
-		(effects
-			(font
-				(size 1.27 1.27)
-			)
-			(justify left bottom)
-		)
-	)
 	(label "GPIO_62"
 		(at 87.63 49.53 180)
@@
 		)
 	)
-	(label "GPIO_60"
+	(label "GPIO_38"
 		(at 238.76 69.85 0)
 		(effects
@@
 		)
 	)
+	(label "GPIO_34"
+		(at 87.63 29.21 180)
+		(effects
+			(font
+				(size 1.27 1.27)
+			)
+			(justify right bottom)
+		)
+	)
 	(label "UART4_TXD"
 		(at 33.02 38.1 180)
@@
 		(effects
 			(font
+				(size 1.27 1.27)
+			)
+			(justify right bottom)
+		)
+	)
+	(label "GPIO_38"
+		(at 87.63 26.67 180)
+		(effects
+			(font
