File: HAB-terminator/hab-terminator/hab-terminator.kicad_sch (KiCad schematic)
At the start: 35 parts, among them J1 Battery, J2 Burn wire, J3 Actuator, J4 MSD-4-A, Q1 DMN2053UVTQ-7, Q2 DMN2053UVTQ-7, Q3 AO3401A, SW1 SW_Push, SW2 SW_Push_EXT, U1 XIAO-ESP32-C3-SMD, U2 DRV8212P, U3 BMP384

Commit message: terminatotr
Parts:
- removed C3: 100nF, Capacitor_SMD:C_0603_1608Metric_Pad1.08x0.95mm_HandSolder, symbol Device:C
- removed C5: 22uF, Capacitor_SMD:C_0805_2012Metric, symbol Device:C
- removed R6: 330, Resistor_SMD:R_0603_1608Metric_Pad0.98x0.95mm_HandSolder, symbol Device:R_US
- removed R7: 100k, Resistor_SMD:R_0603_1608Metric_Pad0.98x0.95mm_HandSolder, symbol Device:R_US
- removed SW1: SW_Push, Button_Switch_SMD:SW_Push_1P1T_NO_E-Switch_TL3301NxxxxxG, symbol Switch:SW_Push
- removed U3: BMP384, BMP384:LGA10_2.0X2.0X0.95_BOS, symbol BMP384:BMP384
- added C7: 100nF, Capacitor_SMD:C_0603_1608Metric, symbol Device:C
- added D4, D5: LED, LED_SMD:LED_0603_1608Metric, symbol Device:LED
- added J5: Heater, Connector_PinSocket_2.54mm:PinSocket_1x02_P2.54mm_Vertical, symbol Connector:Conn_01x02_Socket
- added Q4: AO3401A, Package_TO_SOT_SMD:SOT-23, symbol Transistor_FET:AO3401A
- added R17: 100k, Resistor_SMD:R_0603_1608Metric, symbol Device:R_US
- added R18: 10k, Resistor_SMD:R_0603_1608Metric, symbol Device:R_US
- added R19: 330, Resistor_SMD:R_0603_1608Metric, symbol Device:R_US
- added R20, R21: 150k, Resistor_SMD:R_0603_1608Metric, symbol Device:R_US
- added U3: 74LVC1G3157, Package_TO_SOT_SMD:SOT-363_SC-70-6, symbol 74xGxx:74LVC1G3157
- added U4: MS5607-02BA, Package_LGA:LGA-8_3x5mm_P1.25mm, symbol Sensor_Pressure:MS5607-02BA
- C2, C4, C6: footprint Capacitor_SMD:C_0603_1608Metric_Pad1.08x0.95mm_HandSolder -> Capacitor_SMD:C_0603_1608Metric
- R10, R11, R12, R13, R15, R3, R4, R5, R8, R9, TH1: footprint Resistor_SMD:R_0603_1608Metric_Pad0.98x0.95mm_HandSolder -> Resistor_SMD:R_0603_1608Metric
- R14: value 10k -> 4.7k; footprint Resistor_SMD:R_0603_1608Metric_Pad0.98x0.95mm_HandSolder -> Resistor_SMD:R_0603_1608Metric
- R16: value 1k -> 330; footprint Resistor_SMD:R_0603_1608Metric_Pad0.98x0.95mm_HandSolder -> Resistor_SMD:R_0603_1608Metric
Connections:
- net +3V3: now also U3.5 (VCC), U4.1 (VDD), U4.2 (PS)
- net +BATT: now also C4.1, J2.2 (Pin_2), Q3.2 (S), U2.1 (VM), J5.1 (Pin_1), R17.1, R19.2, R21.1; no longer J1.1 (Pin_1), J2.1 (Pin_1), Q3.3 (D), R13.1, SW2.1
- net BURN_ARM/PWR_HOLD: now also Q1.3 (G), C7.2; no longer R5.1
- net GND: now also J1.1 (Pin_1), C7.1, D4.1 (K), D5.1 (K), Q4.2 (S), R18.1, R20.1, U3.2 (GND), U4.3 (GND); no longer J1.2 (Pin_2), Q3.2 (S), R11.1
- net I2C_SCL: now also R15.1, U4.8 (SCLK); no longer R14.1
- net I2C_SDA: now also R14.1, U4.7 (SDI/SDA); no longer R15.1
- net HEATER_EN/A_MUX: now reaches R5.2
- net HEATER_EN/A_MUX: now also U1.3 (GPIO4_A2_D2), Q4.1 (G), R17.2, U3.6; no longer Q1.3 (G)
- net BURN_EN/ACT_1: now reaches Q1.1 (G), R8.1
- net BURN_EN/ACT_1: now also R3.2, U1.7 (GPIO21_D6_TX), U2.6 (IN1)
- net CSB/~{SLEEP}: now reaches R10.1, U2.7 (~{SLEEP})
- net CSB/~{SLEEP}: now also U4.4 (CSB), U4.5 (CSB)
- net at Q1.4 (D): now also J2.1 (Pin_1); no longer J2.2 (Pin_2)
- net V_USB: now reaches U1.14 (VBUS)
- net ACT_1 renamed SW_SNS/ACT_2
- net SW_SNS/ACT_2: now also R11.1, U2.5 (IN2), R18.2; no longer U2.6 (IN1)
- removed net ACT_2: U1.7 (GPIO21_D6_TX), U2.5 (IN2)
- removed net BURN_EN: R3.2, U1.3 (GPIO4_A2_D2)
- net NTC_1 renamed NTC
- net NTC: now also U3.1; no longer U1.1 (GPIO2_A0_D0)
- new net: D5.2 (A), R5.1
- new net: J5.2 (Pin_2), Q4.3 (D)
- new net: R20.2, R21.2, U3.3
- new net: D4.2 (A), R19.1
- new net NTC/VBAT_SNS: U1.1 (GPIO2_A0_D0), U3.4
- new net VBAT: J1.2 (Pin_2), Q3.3 (D), R13.1, SW2.1
Other:
- note added: "2:1 MUX between thermistor and battery voltage"
- note added: "Configure ADC attenuation to 11dB"
- note removed: "TODO simulate"
- moved on the sheet: C4, D1, D2, D3, J3, J4, Q1A, Q1B, Q2A, Q2B, Q3, R10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
