File: HAB-terminator/hab-terminator/hab-terminator.kicad_sch (KiCad schematic)
At the start: 41 parts, among them J1 Battery, J2 Burn wire, J3 Actuator, J4 MSD-4-A, J5 Heater, Q1 DMN2053UVTQ-7, Q2 DMN2053UVTQ-7, Q3 AO3401A, Q4 AO3401A, SW2 SW_Push_EXT, U1 XIAO-ESP32-C3-SMD, U2 DRV8212P, U3 74LVC1G3157, U4 MS5607-02BA

Commit message: updating terminator
Parts:
- R14, R15: value 4.7k -> 10k
Connections:
- net +BATT: now also Q3.3 (D); no longer Q3.2 (S)
- net GND: now also Q4.3 (D); no longer Q4.2 (S)
- net VBAT: now also Q3.2 (S); no longer Q3.3 (D)
- net at J5.2 (Pin_2): now also Q4.2 (S); no longer Q4.3 (D)
Changed lines of the file:
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@@
 		(lib_id "Transistor_FET:AO3401A")
 		(at 87.63 171.45 0)
+		(mirror x)
 		(unit 1)
 		(body_style 1)
@@
 		(in_pos_files yes)
 		(dnp no)
-		(fields_autoplaced yes)
 		(property "Reference" "Q4"
-			(at 93.98 170.1799 0)
+			(at 93.98 172.7201 0)
 			(show_name no)
 			(do_not_autoplace no)
@@
 		)
 		(property "Value" "AO3401A"
-			(at 93.98 172.7199 0)
+			(at 93.98 170.1801 0)
 			(show_name no)
 			(do_not_autoplace no)
@@
 		)
 		(property "Footprint" "Package_TO_SOT_SMD:SOT-23"
-			(at 92.71 173.355 0)
+			(at 92.71 169.545 0)
 			(hide yes)
 			(show_name no)
@@
 		)
 		(property "Datasheet" "http://www.aosmd.com/pdfs/datasheet/AO3401A.pdf"
-			(at 92.71 175.26 0)
+			(at 92.71 167.64 0)
 			(hide yes)
 			(show_name no)
@@
 			)
 		)
-		(property "Value" "4.7k"
+		(property "Value" "10k"
 			(at 176.784 82.5501 0)
 			(show_name no)
@@
 			)
 		)
-		(property "Value" "4.7k"
+		(property "Value" "10k"
 			(at 182.626 84.582 0)
 			(show_name no)
@@
 		(lib_id "Transistor_FET:AO3401A")
 		(at 205.74 133.35 0)
+		(mirror x)
 		(unit 1)
 		(body_style 1)
@@
 		(in_pos_files yes)
 		(dnp no)
-		(fields_autoplaced yes)
 		(property "Reference" "Q3"
-			(at 212.09 132.0799 0)
+			(at 212.09 134.6201 0)
 			(show_name no)
 			(do_not_autoplace no)
@@
 		)
 		(property "Value" "AO3401A"
-			(at 212.09 134.6199 0)
+			(at 212.09 132.0801 0)
 			(show_name no)
 			(do_not_autoplace no)
@@
 		)
 		(property "Footprint" "Package_TO_SOT_SMD:SOT-23"
-			(at 210.82 135.255 0)
+			(at 210.82 131.445 0)
 			(hide yes)
 			(show_name no)
@@
 		)
 		(property "Datasheet" "http://www.aosmd.com/pdfs/datasheet/AO3401A.pdf"
-			(at 210.82 137.16 0)
+			(at 210.82 129.54 0)
 			(hide yes)
 			(show_name no)

Commit message: updated terminator layout
Parts:
- removed R15: 10k, Resistor_SMD:R_0603_1608Metric, symbol Device:R_US
- R11, R14, R18: value 10k -> 100k
- R20, R21: value 150k -> 100k
Connections:
- net +3V3: no longer R14.2, U4.2 (PS)
- net GND: now also R14.2, U4.2 (PS)
- net NTC/VBAT_SNS: now also U1.2 (GPIO3_A1_D1); no longer U1.1 (GPIO2_A0_D0)
- net SPI_CLK: now also U4.8 (SCLK)
- net SPI_MISO: now also U4.6 (SDO)
- net SPI_MOSI: now also U4.7 (SDI/SDA)
- net BURN_ARM/PWR_HOLD renamed PWR_HOLD
- net PWR_HOLD: now also U1.4 (GPIO5_A3_D3); no longer Q1.3 (G), R4.2, U1.2 (GPIO3_A1_D1)
- net CSB/~{SLEEP}: no longer names the net of R10.1, U2.7 (~{SLEEP})
- net CSB/~{SLEEP}: no longer U4.4 (CSB), U4.5 (CSB)
- net I2C_SCL renamed MS5607_CS
- net MS5607_CS: now also U4.4 (CSB), U4.5 (CSB); no longer U4.8 (SCLK)
- net I2C_SDA renamed BURN_ARM/ACT_2
- net BURN_ARM/ACT_2: now also Q1.3 (G), R4.2, U2.5 (IN2); no longer U4.7 (SDI/SDA)
- net SW_SNS/ACT_2 renamed SW_SNS
- net SW_SNS: now also U1.1 (GPIO2_A0_D0); no longer U1.4 (GPIO5_A3_D3), U2.5 (IN2)
- no-connect marks 4 -> 3
Other:
- note added: "Sets to SPI mode"
- note removed: "Sets to I2C mode"
- note removed: "addr: 0x76"
- moved on the sheet: R10
