File: HAB-terminator/hab-terminator/hab-terminator.kicad_pcb (KiCad board)
At the start: 2 copper layers, 23.8 x 61 mm, 35 parts, among them J1 Battery, J2 Burn wire, J3 Actuator, J4 MSD-4-A, Q1 DMN2053UVTQ-7, Q2 DMN2053UVTQ-7, Q3 AO3401A, SW1 SW_Push, SW2 SW_Push_EXT, U1 XIAO-ESP32-C3-SMD, U2 DRV8212P, U3 BMP384

Commit message: terminatotr
Parts:
- removed C3: 100nF, Capacitor_SMD:C_0603_1608Metric_Pad1.08x0.95mm_HandSolder
- removed C5: 22uF, Capacitor_SMD:C_0805_2012Metric
- removed R6: 330, Resistor_SMD:R_0603_1608Metric_Pad0.98x0.95mm_HandSolder
- removed R7: 100k, Resistor_SMD:R_0603_1608Metric_Pad0.98x0.95mm_HandSolder
- removed SW1: SW_Push, Button_Switch_SMD:SW_Push_1P1T_NO_E-Switch_TL3301NxxxxxG
- added C7: 100nF, Capacitor_SMD:C_0603_1608Metric, F.Cu at (93.4, 129.2)
- added D4: LED, LED_SMD:LED_0603_1608Metric, F.Cu at (106.6, 120.8)
- added D5: LED, LED_SMD:LED_0603_1608Metric, F.Cu at (106.8, 139.8)
- added J5: Heater, Connector_PinSocket_2.54mm:PinSocket_1x02_P2.54mm_Vertical, F.Cu at (106.5, 136.8)
- added Q4: AO3401A, Package_TO_SOT_SMD:SOT-23, F.Cu at (100.0, 137.2)
- added R17: 100k, Resistor_SMD:R_0603_1608Metric, F.Cu at (100.0, 134.2)
- added R18: 10k, Resistor_SMD:R_0603_1608Metric, F.Cu at (97.6, 132.4)
- added R19: 330, Resistor_SMD:R_0603_1608Metric, F.Cu at (103.2, 120.8)
- added R20: 150k, Resistor_SMD:R_0603_1608Metric, F.Cu at (95.0, 123.2)
- added R21: 150k, Resistor_SMD:R_0603_1608Metric, F.Cu at (99.8, 120.8)
- added U4: MS5607-02BA, Package_LGA:LGA-8_3x5mm_P1.25mm, F.Cu at (90.2, 123.8)
- C2: footprint Capacitor_SMD:C_0603_1608Metric_Pad1.08x0.95mm_HandSolder -> Capacitor_SMD:C_0603_1608Metric; moved to B.Cu
- C4, C6: footprint Capacitor_SMD:C_0603_1608Metric_Pad1.08x0.95mm_HandSolder -> Capacitor_SMD:C_0603_1608Metric
- R10, R11, R12, R13, R15, R3, R4, R5, R8, TH1: footprint Resistor_SMD:R_0603_1608Metric_Pad0.98x0.95mm_HandSolder -> Resistor_SMD:R_0603_1608Metric
- R14: value 10k -> 4.7k; footprint Resistor_SMD:R_0603_1608Metric_Pad0.98x0.95mm_HandSolder -> Resistor_SMD:R_0603_1608Metric
- R16: value 1k -> 330; footprint Resistor_SMD:R_0603_1608Metric_Pad0.98x0.95mm_HandSolder -> Resistor_SMD:R_0603_1608Metric
- R9: footprint Resistor_SMD:R_0603_1608Metric_Pad0.98x0.95mm_HandSolder -> Resistor_SMD:R_0603_1608Metric; moved to B.Cu
- U3: value BMP384 -> 74LVC1G3157; footprint BMP384:LGA10_2.0X2.0X0.95_BOS -> Package_TO_SOT_SMD:SOT-363_SC-70-6
- moved R9 67.5 mm to (97.0, 111.7)
- moved R15 57.6 mm to (88.2, 120.8), turned to 180 degrees
- moved R14 53.6 mm to (92.0, 120.8)
- moved C4 51.3 mm to (86.4, 127.4), turned to 90 degrees
- moved R13 50.9 mm to (94.8, 126.0), turned to -90 degrees
- moved C6 49.9 mm to (86.4, 123.7), turned to -90 degrees
- moved R10 48.9 mm to (92.2, 126.8), turned to 180 degrees
- moved R11 40.4 mm to (100.8, 130.8), turned to 90 degrees
- moved C2 39.0 mm to (97.0, 113.4)
- moved D2 38.0 mm to (87.0, 139.8), turned to 0 degrees
- moved R4 34.8 mm to (90.2, 139.8), turned to 0 degrees
- moved R3 29.0 mm to (90.2, 138.0), turned to 0 degrees
- moved D1 25.2 mm to (87.0, 138.0), turned to 0 degrees
- moved SW2 23.8 mm to (106.5, 133.0), turned to -90 degrees
- moved R16 19.4 mm to (103.4, 130.0)
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Connections:
- net Net-(U2-~{SLEEP}) renamed /CSB/~{SLEEP}
- C2 pad 1: /NTC_1 -> /NTC
- C4 pad 1: Net-(U2-VM) -> +BATT
- J1 pad 1: +BATT -> GND
- J1 pad 2: GND -> /VBAT
- J2 pad 1: +BATT -> Net-(J2-Pin_1)
- J2 pad 2: Net-(J2-Pin_2) -> +BATT
- Q1 pad 1: Net-(Q1A-G) -> /BURN_EN/ACT_1
- Q1 pad 3: Net-(Q1B-G) -> /BURN_ARM/PWR_HOLD
- Q1 pad 4: Net-(J2-Pin_2) -> Net-(J2-Pin_1)
- Q3 pad 2: GND -> +BATT
- Q3 pad 3: +BATT -> /VBAT
- R11 pad 1: GND -> /SW_SNS/ACT_2
- R13 pad 1: +BATT -> /VBAT
- R14 pad 1: /I2C_SCL -> /I2C_SDA
- R15 pad 1: /I2C_SDA -> /I2C_SCL
- R3 pad 2: /BURN_EN -> /BURN_EN/ACT_1
- R5 pad 1: /BURN_ARM/PWR_HOLD -> Net-(D5-A)
- R5 pad 2: Net-(Q1B-G) -> /HEATER_EN/A_MUX
- R8 pad 1: Net-(Q1A-G) -> /BURN_EN/ACT_1
- R9 pad 1: /NTC_1 -> /NTC
- SW2 pad 1: +BATT -> /VBAT
- TH1 pad 1: /NTC_1 -> /NTC
- U1 pad 1: /NTC_1 -> /NTC/VBAT_SNS
- U1 pad 14: unconnected-(U1-VBUS-Pad14) -> /V_USB
- U1 pad 3: /BURN_EN -> /HEATER_EN/A_MUX
- U1 pad 4: /ACT_1 -> /SW_SNS/ACT_2
- U1 pad 7: /ACT_2 -> /BURN_EN/ACT_1
- U2 pad 1: Net-(U2-VM) -> +BATT
- U2 pad 5: /ACT_2 -> /SW_SNS/ACT_2
- U2 pad 6: /ACT_1 -> /BURN_EN/ACT_1
- U3 pad 1: +3V3 -> /NTC
- U3 pad 2: /I2C_SCL -> GND
- U3 pad 3: GND -> Net-(R20-Pad2)
- U3 pad 4: /I2C_SDA -> /NTC/VBAT_SNS
- U3 pad 5: GND -> +3V3
- U3 pad 6: +3V3 -> /HEATER_EN/A_MUX
Routing:
- net +BATT: track 0.00 -> 87.7 mm, vias 0 -> 1
- net +3V3: track 0.00 -> 84.4 mm, vias 0 -> 6
- net /BURN_ARM/PWR_HOLD: track 0.00 -> 53.0 mm, vias 0 -> 5
- net /HEATER_EN/A_MUX: track 0.00 -> 47.1 mm, vias 0 -> 4
- net /SPI_MISO: track 0.00 -> 38.2 mm, vias 0 -> 2
- net /SPI_MOSI: track 0.00 -> 37.7 mm, vias 0 -> 2
- net /SPI_CLK: track 0.00 -> 35.3 mm, vias 0 -> 2
- net /SW_SNS/ACT_2: track 0.00 -> 34.9 mm, vias 0 -> 3
- net /BURN_EN/ACT_1: track 0.00 -> 33.2 mm, vias 0 -> 3
- net /SD_CS: track 0.00 -> 30.2 mm, vias 0 -> 2
- net /NTC/VBAT_SNS: track 0.00 -> 23.5 mm, vias 0 -> 2
- net /VBAT: track 0.00 -> 17.9 mm
- net /I2C_SCL: track 0.00 -> 15.1 mm, vias 0 -> 2
- net /NTC: track 0.00 -> 13.5 mm, vias 0 -> 1
- net /I2C_SDA: track 0.00 -> 10.6 mm
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- added copper zone on B.Cu, net GND
- added copper zone on F.Cu, net GND
Other:
- board size 23.8 x 61 mm -> 25 x 60 mm
- board text added: "ARM"
- board text added: "Ben D'Agnillo - 06/26"
- board text added: "FIRE"
- board text added: "HAB-Deployer V1.0"
- board text added: "HEATER"
- board text added: "POWER"

Commit message: fixing power board
Parts:
- added G***: LOGO, LOGO, B.Cu at (96.9, 149.8)
- moved J4 0.60 mm to (97.2, 150.2)
Other:
- board size 25 x 60 mm -> 25 x 63.3 mm
