File: PMDS-motor-drivers/PMDS-motor-drivers.kicad_pcb (KiCad board)
At the start: 2 copper layers, 51 x 100.4 mm, 34 parts, among them J1 Conn_01x15, J2 Conn_01x15, J3 Conn_01x10, J4 Conn_01x02, J5 Screw_Terminal_01x02, J6 MSD-4-A, J7 Screw_Terminal_01x02, J8 power for motor driver, SW1 SW_Push, SW2 SW_Push, SW3 SW_Push, SW4 SW_DPST_x2, U1 L9110H, U2 5V buck, U3 MS5607-02BA, U4 L9110H

Commit message: fixes
Parts:
- U1, U4: footprint Package_DIP:DIP-8_W8.89mm_SMDSocket_LongPads -> Package_DIP:DIP-8_W7.62mm
- moved U4 5.91 mm to (204.6, 126.5)
- moved U1 5.82 mm to (204.6, 139.1)
- moved C6 1.51 mm to (198.0, 111.4), turned to 90 degrees
- moved D3 1.15 mm to (200.6, 85.2), turned to 180 degrees
Routing:
- net /FWD_1: track 59.1 -> 57.3 mm
- net /REV_1: track 59.1 -> 57.3 mm
- net /REV_2: track 49.4 -> 50.7 mm
- net /FWD_2: track 50.5 -> 51.9 mm
- net +5V: track 103.4 -> 102.3 mm
- net Net-(J7-Pin_1): track 10.1 -> 11.0 mm
- net GND: vias 186 -> 180
Other:
- outline, holes or cut-outs redrawn
