File: PMDS-motor-drivers/PMDS-motor-drivers.kicad_sch (KiCad schematic)
At the start: 30 parts, among them J4 Conn_01x02, J5 Screw_Terminal_01x02, J6 MSD-4-A, J7 Screw_Terminal_01x02, M1 Motor_DC, M2 Motor_DC, SW1 SW_Push, SW2 SW_Push, SW3 SW_Push, SW4 SW_DPST_x2, U1 L9110H, U2 5V buck, U3 MS5607-02BA, U4 L9110H

Commit message: fixes
Parts:
- U1, U4: footprint Package_DIP:DIP-8_W8.89mm_SMDSocket_LongPads -> Package_DIP:DIP-8_W7.62mm
Changed lines of the file:
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@@
 			)
 		)
-		(property "Footprint" "Package_DIP:DIP-8_W8.89mm_SMDSocket_LongPads"
+		(property "Footprint" "Package_DIP:DIP-8_W7.62mm"
 			(at 137.16 100.33 0)
 			(hide yes)
@@
 			)
 		)
-		(property "Footprint" "Package_DIP:DIP-8_W8.89mm_SMDSocket_LongPads"
+		(property "Footprint" "Package_DIP:DIP-8_W7.62mm"
 			(at 66.04 97.79 0)
 			(hide yes)
