File: Photodiode-breakout/Photodiode-breakout.kicad_sch (KiCad schematic)
At the start: 21 parts, among them J1 Conn_01x06_Pin, U1 OPA320AIDBVR, U2 ADS1220xPW

Commit message: post 2nd revision update
Connections:
- net NTC_DIFF+: now also R5.2, TH1.2; no longer R3.1, R4.2
- net NTC_DIFF-: now also R3.1, R4.2; no longer R5.2, TH1.2
Changed lines of the file:
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@@
-		)
-	)
-	(label "NTC_DIFF-"
-		(at 124.46 124.46 0)
-		(effects
-			(font
-				(size 1.27 1.27)
-			)
-			(justify left bottom)
 		)
 	)
@@
 	(label "BIAS_IN+"
 		(at 104.14 73.66 180)
+		(effects
+			(font
+				(size 1.27 1.27)
+			)
+			(justify right bottom)
+		)
+	)
+	(label "NTC_DIFF-"
+		(at 107.95 124.46 180)
 		(effects
 			(font
@@
 	)
 	(label "NTC_DIFF+"
-		(at 107.95 124.46 180)
+		(at 124.46 124.46 0)
 		(effects
 			(font
 				(size 1.27 1.27)
 			)
-			(justify right bottom)
+			(justify left bottom)
 		)
 	)
